File: DQBSC/MPU.kicad_sch (KiCad schematic)
At the start: 167 parts, among them U1 MIMX8MD6DVAJZAB, U11 TLV803EB26RDBZR, U12 SIT1630AI-S4-DCC-32.768G, Y4 ABM3B-25.000MHZ-D4Y-T, Y5 ABM3B-25.000MHZ-D4Y-T

Commit message: Update.
Connections:
- net GPIO2 renamed NWDOG
Other:
- note added: "IMX8 CSI"
- note added: "add capacitive couplig to tx and clk?"
Changed lines of the file:
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@@
     (effects (font (size 1.27 1.27) (color 0 0 255 1)) (justify left bottom))
+  )
+  (text "add capacitive couplig to tx and clk?" (exclude_from_sim no)
+ (at 99.06 180.34 0)
+    (effects (font (size 1.016 1.016)) (justify left bottom))
   )
   (text "IMX8 HDMI" (exclude_from_sim no)
@@
     (effects (font (size 1.27 1.27)) (justify left bottom))
   )
-  (text "IX8 DRAM" (exclude_from_sim no)
+  (text "IMX8 CSI" (exclude_from_sim no)
  (at 237.998 225.552 0)
     (effects (font (size 1.27 1.27) (thickness 0.254) bold (color 255 255 255 1)) (justify right bottom))
@@
     (property "Intersheetrefs" "${INTERSHEET_REFS}" (at 294.64 114.416 90)
       (effects (font (size 1.27 1.27)) (justify right) hide)
-    )
-  )
-  (global_label "GPIO2" (shape bidirectional) (at 213.36 233.68 0) (fields_autoplaced)
-    (effects (font (size 1 1)) (justify left))
-    (property "Intersheetrefs" "${INTERSHEET_REFS}" (at 220.8741 233.68 0)
-      (effects (font (size 1.27 1.27)) (justify left) hide)
     )
   )
@@
     )
   )
+  (global_label "NWDOG" (shape input) (at 213.36 233.68 0) (fields_autoplaced)
+    (effects (font (size 1 1)) (justify left))
+    (property "Intersheetrefs" "${INTERSHEET_REFS}" (at 220.9484 233.68 0)
+      (effects (font (size 1.27 1.27)) (justify left) hide)
+    )
+  )

Commit message: UPDATE, FULL ROUTING!
Parts:
- FB1: footprint (none) -> Inductor_SMD:L_0402_1005Metric
Connections:
- net 3.3V_SW: now also U1.W18 (NVCC_SNVS)
- net NVCC_SNVS_3V3: no longer U1.W18 (NVCC_SNVS)
- net BT_DEV_WAKE: no longer names the net of U1.G21 (NAND_CE1_B)
- net BT_HOST_WAKE: no longer names the net of U1.M20 (NAND_DQS)
- net NAND_DATA4: no longer names the net of U1.L20 (NAND_DATA04)
- net NAND_DATA5: no longer names the net of U1.J22 (NAND_DATA05)
- net NAND_DATA6: no longer names the net of U1.L19 (NAND_DATA06)
- net NAND_DATA7: no longer names the net of U1.M19 (NAND_DATA07)
- net NAND_nCE3: no longer names the net of U1.H20 (NAND_CE3_B)
- net NAND_nREADY: no longer names the net of U1.K20 (NAND_READY_B)
- net NAND_nWE: no longer names the net of U1.K22 (NAND_WE_B)
- net NAND_nWP: no longer names the net of U1.K21 (NAND_WP_B)
- net QSPIA_CLE: no longer names the net of U1.H21 (NAND_CLE)
- net TCPC_nINT: no longer names the net of U1.F21 (NAND_CE2_B)
- net USB1_SS_SEL: no longer names the net of U1.K19 (NAND_RE_B)
- no-connect marks 33 -> 46
