File: DQBSC/MPU.kicad_sch (KiCad schematic)
At the start: 167 parts, among them U1 MIMX8MD6DVAJZAB, U11 TLV803EB26RDBZR, U12 SIT1630AI-S4-DCC-32.768G, Y4 ABM3B-25.000MHZ-D4Y-T, Y5 ABM3B-25.000MHZ-D4Y-T

Commit message: Update.
Connections:
- net GPIO12 renamed USB1_PWR_EN
- net GPIO13 renamed USB1_OC
- net GPIO14 renamed USB2_PWR_EN
- net GPIO15 renamed USB2_OC
Changed lines of the file:
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@@
     (effects (font (size 1.27 1.27)) (justify left bottom))
   )
-  (global_label "GPIO13" (shape bidirectional) (at 213.36 261.62 0) (fields_autoplaced)
-    (effects (font (size 1 1)) (justify left))
-    (property "Intersheetrefs" "${INTERSHEET_REFS}" (at 220.8741 261.62 0)
-      (effects (font (size 1.27 1.27)) (justify left) hide)
-    )
-  )
   (global_label "POR_B" (shape input) (at 347.98 182.88 180) (fields_autoplaced)
     (effects (font (size 1 1)) (justify right))
@@
     )
   )
-  (global_label "GPIO14" (shape bidirectional) (at 213.36 264.16 0) (fields_autoplaced)
+  (global_label "USB2_PWR_EN" (shape bidirectional) (at 213.36 264.16 0) (fields_autoplaced)
     (effects (font (size 1 1)) (justify left))
-    (property "Intersheetrefs" "${INTERSHEET_REFS}" (at 220.8741 264.16 0)
+    (property "Intersheetrefs" "${INTERSHEET_REFS}" (at 227.1568 264.16 0)
       (effects (font (size 1.27 1.27)) (justify left) hide)
     )
@@
     )
   )
+  (global_label "USB1_OC" (shape bidirectional) (at 213.36 261.62 0) (fields_autoplaced)
+    (effects (font (size 1 1)) (justify left))
+    (property "Intersheetrefs" "${INTERSHEET_REFS}" (at 223.3472 261.62 0)
+      (effects (font (size 1.27 1.27)) (justify left) hide)
+    )
+  )
   (global_label "ENET_TD2" (shape output) (at 256.54 160.02 270) (fields_autoplaced)
     (effects (font (size 1 1)) (justify right))
@@
     )
   )
+  (global_label "USB1_PWR_EN" (shape bidirectional) (at 213.36 259.08 0) (fields_autoplaced)
+    (effects (font (size 1 1)) (justify left))
+    (property "Intersheetrefs" "${INTERSHEET_REFS}" (at 227.1568 259.08 0)
+      (effects (font (size 1.27 1.27)) (justify left) hide)
+    )
+  )
   (global_label "ENET_TXC" (shape output) (at 248.92 160.02 270) (fields_autoplaced)
     (effects (font (size 1 1)) (justify right))
@@
     )
   )
-  (global_label "GPIO12" (shape bidirectional) (at 213.36 259.08 0) (fields_autoplaced)
-    (effects (font (size 1 1)) (justify left))
-    (property "Intersheetrefs" "${INTERSHEET_REFS}" (at 220.8741 259.08 0)
-      (effects (font (size 1.27 1.27)) (justify left) hide)
-    )
-  )
   (global_label "ENET_TD1" (shape output) (at 254 160.02 270) (fields_autoplaced)
     (effects (font (size 1 1)) (justify right))
@@
     )
   )
-  (global_label "GPIO15" (shape bidirectional) (at 213.36 266.7 0) (fields_autoplaced)
+  (global_label "USB2_OC" (shape bidirectional) (at 213.36 266.7 0) (fields_autoplaced)
     (effects (font (size 1 1)) (justify left))
-    (property "Intersheetrefs" "${INTERSHEET_REFS}" (at 220.8741 266.7 0)
+    (property "Intersheetrefs" "${INTERSHEET_REFS}" (at 223.3472 266.7 0)
       (effects (font (size 1.27 1.27)) (justify left) hide)
     )
@@
   (symbol (lib_id "DQSBC:R_US") (at 238.76 214.63 0) (unit 1)
     (exclude_from_sim no) (in_bom yes) (on_board yes) (dnp no)
-    (property "Reference" "R41" (at 237.998 218.44 90)
+    (property "Reference" "R41" (at 236.22 215.9 90)
       (effects (font (size 1.27 1.27)))
     )
-    (property "Value" "15K" (at 238.125 210.185 90)
+    (property "Value" "15K" (at 236.22 213.36 90)
       (effects (font (size 1.27 1.27)))
     )

Commit message: Update.
Parts:
- added HS1: HSB07-202009, DQSBC:HSB07-202009, symbol Mechanical:Heatsink
Other:
- moved on the sheet: C196, C367, R5, R69, R70, Y5
