File: DQBSC/DQBSC.kicad_sch (KiCad schematic)
At the start: 0 parts

Commit message: UPDATE TO POWER TREE.
Connections:
- no-connect marks 2 -> 0
Other:
- note added: "DSI"
- note added: "GPIO X"
- note added: "HDMI"
- note added: "I2C X"
- note added: "PCIE X"
- note added: "POWER INPUT 5 ~ 25V DC"
- note added: "RGMII"
- note added: "UART X"
- note added: "USB"
- note removed: "*0.028A/3.3V"
- note removed: "*0.068A/3.3V"
- note removed: "*0.096A/3.3V"
- note removed: "*0.5MA/3.3V"
- note removed: "*0.6A"
- note removed: "*0.6A/3.3V"
- note removed: "*0.7A/3.3V"
- note removed: "*0.85A/3.3V"
- note removed: "*0.91A/3.3V"
- note removed: "*0.9A"
- note removed: "*0.9V/0.1A"
- note removed: "*0.9V/0.25A"
- note removed: "*0.9V/0.35A"
- note removed: "*0.9V/2.5A"
- note removed: "*0.9V/2A"
- note removed: "*1.1V/2.5A"
- note removed: "*1.8V/1A"
- note removed: "*1V/1.5MA"
- note removed: "*1V/3A"
- note removed: "*4A"
- note removed: "0.9V/2A"
- note removed: "0.9V/3A"
- note removed: "3.3VSW/10A"
- note removed: "GEN1"
- note removed: "GEN2"
- note removed: "GEN3"
- note removed: "GEN4"
- note removed: "GEN5"
- note removed: "GEN6"
- note removed: "NVCC_DRAM"
- note removed: "PF4210"
- note removed: "PMIC"
- note removed: "SW1AB"
- note removed: "SW1C"
- note removed: "SW2"
- note removed: "SW3AB"
- note removed: "SW4A"
- note removed: "VDDA_1V8"
- note removed: "VDD_1V8"
- note removed: "VDD_ARM"
- note removed: "VDD_DRAM"
- note removed: "VDD_GPU"
- note removed: "VDD_PHY_0V9"
- note removed: "VDD_PHY_1V8"
- note removed: "VDD_PHY_3V3"
- note removed: "VDD_SOC"
- note removed: "VDD_VPU"
- note removed: "VIN = 4.75 ~ 20V"
- note removed: "VSNVS"

Commit message: Update.
Changed lines of the file:
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@@
     (rev "1.00")
   )
+  (polyline (pts (xy 55.88 198.12) (xy 53.34 195.58))
+    (stroke (width 1) (type default) (color 0 0 0 1))
+  )
   (polyline (pts (xy 139.7 139.7) (xy 195.58 139.7))
     (stroke (width 1) (type default) (color 0 0 0 1))
   )
+  (polyline (pts (xy 76.2 185.42) (xy 78.74 187.96))
+    (stroke (width 1) (type default) (color 0 0 0 1))
+  )
   (polyline (pts (xy 139.7 109.22) (xy 195.58 109.22))
     (stroke (width 1) (type default) (color 0 0 0 1))
@@
     (stroke (width 1) (type default) (color 0 0 0 1))
   )
+  (polyline (pts (xy 58.42 195.58) (xy 55.88 198.12))
+    (stroke (width 1) (type default) (color 0 0 0 1))
+  )
   (polyline (pts (xy 139.7 99.06) (xy 182.88 99.06))
     (stroke (width 1) (type default) (color 0 0 0 1))
@@
     (stroke (width 1) (type default) (color 0 0 0 1))
   )
+  (polyline (pts (xy 104.14 195.58) (xy 101.6 198.12))
+    (stroke (width 1) (type default) (color 0 0 0 1))
+  )
   (polyline (pts (xy 76.2 185.42) (xy 76.2 198.12))
     (stroke (width 1) (type default) (color 0 0 0 1))
@@
     (stroke (width 1) (type default) (color 0 0 0 1))
   )
+  (polyline (pts (xy 73.66 187.96) (xy 76.2 185.42))
+    (stroke (width 1) (type default) (color 0 0 0 1))
+  )
   (polyline (pts (xy 193.04 127) (xy 195.58 129.54))
     (stroke (width 1) (type default) (color 0 0 0 1))
@@
     (stroke (width 1) (type default) (color 0 0 0 1))
   )
+  (polyline (pts (xy 101.6 198.12) (xy 99.06 195.58))
+    (stroke (width 1) (type default) (color 0 0 0 1))
+  )
   (polyline (pts (xy 195.58 149.86) (xy 193.04 152.4))
     (stroke (width 1) (type default) (color 0 0 0 1))
@@
   )
   (polyline (pts (xy 55.88 185.42) (xy 55.88 198.12))
+    (stroke (width 1) (type default) (color 0 0 0 1))
+  )
+  (polyline (pts (xy 101.6 185.42) (xy 104.14 187.96))
     (stroke (width 1) (type default) (color 0 0 0 1))
   )
@@
     (stroke (width 0) (type default) (color 132 0 0 1))
   )
-  (polyline (pts (xy 204.47 241.3) (xy 201.93 243.84))
-    (stroke (width 1) (type default) (color 0 0 0 1))
-  )
   (polyline (pts (xy 193.04 96.52) (xy 195.58 99.06))
     (stroke (width 1) (type default) (color 0 0 0 1))
   )
   (polyline (pts (xy 190.5 99.06) (xy 195.58 99.06))
+    (stroke (width 1) (type default) (color 0 0 0 1))
+  )
+  (polyline (pts (xy 78.74 195.58) (xy 76.2 198.12))
     (stroke (width 1) (type default) (color 0 0 0 1))
   )
@@
     (stroke (width 0) (type default))
   )
+  (polyline (pts (xy 99.06 187.96) (xy 101.6 185.42))
+    (stroke (width 1) (type default) (color 0 0 0 1))
+  )
+  (polyline (pts (xy 55.88 185.42) (xy 58.42 187.96))
+    (stroke (width 1) (type default) (color 0 0 0 1))
+  )
   (polyline (pts (xy 139.7 157.48) (xy 195.58 157.48))
     (stroke (width 1) (type default) (color 0 0 0 1))
   )
-  (polyline (pts (xy 201.93 238.76) (xy 204.47 241.3))
+  (polyline (pts (xy 53.34 187.96) (xy 55.88 185.42))
     (stroke (width 1) (type default) (color 0 0 0 1))
   )
@@
     (stroke (width 1) (type default) (color 0 0 0 1))
   )
+  (polyline (pts (xy 76.2 198.12) (xy 73.66 195.58))
+    (stroke (width 1) (type default) (color 0 0 0 1))
+  )
   (polyline (pts (xy 195.58 139.7) (xy 193.04 142.24))
     (stroke (width 1) (type default) (color 0 0 0 1))
   )
   (polyline (pts (xy 180.34 96.52) (xy 182.88 99.06))
-    (stroke (width 1) (type default) (color 0 0 0 1))
-  )
-  (polyline (pts (xy 148.59 241.3) (xy 204.47 241.3))
     (stroke (width 1) (type default) (color 0 0 0 1))
   )
@@
     (effects (font (size 2 2) (color 0 0 0 1)))
   )
-  (text_box "ENET\nPHY"
+  (text_box "EMMC\n16 GB"
     (exclude_from_sim no) (at 71.12 198.12 0) (size 10.16 10.16)
     (stroke (width 0.5) (type default) (color 0 0 0 1))
@@
     (effects (font (size 1 1) (thickness 0.4) bold (color 0 0 0 1)))
   )
-  (text_box "ENET\nPHY"
+  (text_box "NOR FLASH\n256 Mbit"
     (exclude_from_sim no) (at 96.52 198.12 0) (size 10.16 10.16)
     (stroke (width 0.5) (type default) (color 0 0 0 1))
@@
     (effects (font (size 1 1) (thickness 0.4) bold (color 0 0 0 1)))
   )
-  (text_box "ENET\nPHY"
+  (text_box "LPRRD4 RAM\n4 GB"
     (exclude_from_sim no) (at 50.8 198.12 0) (size 10.16 10.16)
     (stroke (width 0.5) (type default) (color 0 0 0 1))
@@
   (text "HDMI" (exclude_from_sim no)
  (at 154.94 107.95 0)
-    (effects (font (size 2 2) (thickness 0.4) bold (color 0 0 0 1)) (justify left bottom))
-  )
-  (text "HDMI" (exclude_from_sim no)
- (at 163.83 240.03 0)
     (effects (font (size 2 2) (thickness 0.4) bold (color 0 0 0 1)) (justify left bottom))
   )
@@
       (effects (font (size 1.27 1.27)) (justify left bottom))
     )
-    (property "Sheetfile" "MPU.kicad_sch" (at 36.83 223.52 0)
+    (property "Sheetfile" "MPU.kicad_sch" (at 36.195 183.515 0)
       (effects (font (size 1.27 1.27)) (justify left top))
     )
@@
     (stroke (width 0.5) (type solid) (color 0 0 0 1))
     (fill (color 255 255 255 0.5000))
-    (property "Sheetname" "MEMORIES" (at 35.56 197.485 0)
+    (property "Sheetname" "MEMORIES" (at 36.195 198.12 0)
       (effects (font (size 1.27 1.27)) (justify left bottom))
     )
-    (property "Sheetfile" "MEM.kicad_sch" (at 35.56 211.836 0)
+    (property "Sheetfile" "MEM.kicad_sch" (at 36.195 211.455 0)
       (effects (font (size 1.27 1.27)) (justify left top))
     )
