File: DQBSC/IO.kicad_sch (KiCad schematic)
At the start: 54 parts, among them J1 3-1827253-6, J2 Conn_02x05_Odd_Even, U5 VSC8541XMV-02, Y1 Crystal

Commit message: Update.
Parts:
- added C12: 1nF, Capacitor_SMD:C_0603_1608Metric, symbol awg1000:CAP_UNPOL
- added C12: 1UF, Capacitor_SMD:C_0603_1608Metric, symbol awg1000:CAP_UNPOL
- added D5, D7: ~, Diode_SMD:D_SOD-123F, symbol Device:D_Schottky
- added R19: 100, Resistor_SMD:R_0402_1005Metric_Pad0.72x0.64mm_HandSolder, symbol awg1000:R
- added R19 (x3): 1M, Resistor_SMD:R_0402_1005Metric_Pad0.72x0.64mm_HandSolder, symbol awg1000:R
- added SW1: SW_DIP_x02, symbol Switch:SW_DIP_x02
- added SW2, SW3: NANOT160AS, DQSBC:NANOT160AS, symbol Switch:SW_Push
- added U13: APX811-26UG-7, Package_TO_SOT_SMD:SOT-143, symbol DQSBC:APX811-26UG-7
Connections:
- net GND: now also C12.2, R19.2, SW2.1, SW3.1, U13.1 (GND)
- new net: C12.2, D7.1 (K), R19.1
- new net: C12.1, D5.1 (K), R19.1
- new net: R19.2, R19.2, U13.2 (NRST)
- new net 3.3V_SW: U13.4 (VCC)
- new net MNRST: D5.2 (A), D7.2 (A), R19.1, U13.3 (NMR)
- new net NWDOG: C12.1
- new net ONOFF: SW2.2
- new net PMIC_ON_REQ: R19.1
- new net SYS_NRST: R19.2, SW3.2
Other:
- moved on the sheet: J1

Commit message: UPDATE TO POWER TREE.
Parts:
- removed C12: 1nF, Capacitor_SMD:C_0603_1608Metric, symbol awg1000:CAP_UNPOL
- removed C12: 1UF, Capacitor_SMD:C_0603_1608Metric, symbol awg1000:CAP_UNPOL
- removed D5, D7: ~, Diode_SMD:D_SOD-123F, symbol Device:D_Schottky
- removed R19: 100, Resistor_SMD:R_0402_1005Metric_Pad0.72x0.64mm_HandSolder, symbol awg1000:R
- removed R19 (x3): 1M, Resistor_SMD:R_0402_1005Metric_Pad0.72x0.64mm_HandSolder, symbol awg1000:R
- removed U13: APX811-26UG-7, Package_TO_SOT_SMD:SOT-143, symbol DQSBC:APX811-26UG-7
- added D6: LED, LED_SMD:LED_0603_1608Metric, symbol Device:LED
- added D8: LED, symbol Device:LED
- added R16: 10k, Resistor_SMD:R_0402_1005Metric, symbol awg1000:R
- SW1: footprint (none) -> Button_Switch_SMD:SW_DIP_SPSTx02_Slide_KingTek_DSHP02TJ_W5.25mm_P1.27mm_JPin
Connections:
- net 3.3V_SW: now also R16.1
- net GND: now also D6.1 (K)
- net SYS_NRST: now also J1.B95 (DDI0_DDC_AUX_SEL)
- net LDO_EN: now reaches J1.B94 (DDI0_PAIR6-_(*))
- net SYS_NRST_OUT: now reaches J1.B96 (RSVD)
- new net: D6.2 (A), R16.2
- no-connect marks 20 -> 19
Other:
- note added: "USER BUTTONS"
- moved on the sheet: C50, D1, D2, H1, H2, H3, H4, J2, R73, R74, R75, R76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

Commit message: UPDATE, FULL ROUTING!
Parts:
- added Q1 (x3): 2SK3018-TP, Package_TO_SOT_SMD:SOT-323_SC-70, symbol Device:Q_NMOS_DGS
- added R26, R55, R62, R85: 10k, Resistor_SMD:R_0402_1005Metric, symbol awg1000:R
- added R58, R61: 100k, Resistor_SMD:R_0402_1005Metric, symbol awg1000:R
- added R84: 220, Resistor_SMD:R_0402_1005Metric, symbol awg1000:R
- D2: footprint Diode_SMD:D_SOD-323 -> Diode_SMD:D_SOD-123F
- D8: footprint (none) -> LED_SMD:LED_0603_1608Metric; now not fitted
- R16: value 10k -> 220
Connections:
- net 3.3V_SW: now also R84.1, R85.1
- net 3.3V_SW_DELAYED: now also R26.1, R55.1, R62.1
- net GND: now also J1.A73 (eDP_TX1+/LVDS_A1+), J1.A76 (eDP_TX0-/LVDS_A2-), J1.A79 (LVDS_A3-), J1.A97 (TYPE10#), Q1.3 (S), Q1.3 (S), Q1.3 (S), R58.2, R61.2; no longer D6.1 (K), J1.A80 (GND(FIXED)), J1.A96 (TPM_PP_(*))
- net GPIO0: now also Q1.2 (G), R85.2
- net PCIE1_REF_CLKN: now also J1.B42 (USB3-); no longer J1.B48 (EXCD1_CPPE#)
- net PCIE1_REF_CLKP: now also J1.B43 (USB3+); no longer J1.B49 (SYS_RESET#)
- net PCIE1_RXN: now also J1.B49 (SYS_RESET#); no longer J1.B46 (USB1+)
- net PCIE1_RXP: now also J1.B48 (EXCD1_CPPE#); no longer J1.B45 (USB1-)
- net PCIE1_TXN: now also J1.B46 (USB1+); no longer J1.B42 (USB3-)
- net PCIE1_TXP: now also J1.B45 (USB1-); no longer J1.B43 (USB3+)
- net at D8.1 (K): now also Q1.1 (D)
- net at D8.2 (A): now also R84.2
- net BOOT_SEL: now reaches J1.A67 (GPI2)
- net BOOT_SEL: now also Q1.2 (G), R62.2
- net SD2_nRST: now reaches J1.A85 (GPI3)
- net SD2_nCD: now reaches J1.A86 (RSVD)
- net SD2_WP: now reaches J1.A88 (PCIE_CLK_REF+)
- net SD2_D3: now reaches J1.A89 (PCIE_CLK_REF-)
- net SD2_D2: now reaches J1.A91 (SPI_POWER)
- net SD2_D1: now reaches J1.A92 (SPI_MISO_(**))
- net SD2_D0: now reaches J1.A94 (SPI_CLK_(**))
- net SD2_CMD: now reaches J1.A95 (SPI_MOSI_(**))
- net BOOT_MODE1: now reaches SW1.1
- net BOOT_MODE1: now also R61.1
- net BOOT_MODE0: now reaches SW1.2
- net BOOT_MODE0: now also Q1.1 (D), R58.1
- net at SW1.3: now also R26.2
- net at SW1.4: now also R55.2
- net GPIO11: no longer names the net of J1.B69 (PCIE_RX0-)
- net GPIO2: no longer names the net of J1.B82 (DDI0_PAIR3-)
- net LDO_EN renamed VBAT
- new net: D6.1 (K), Q1.1 (D)
- new net PG_VIN: Q1.2 (G)
- new net SD2_CLK: J1.A96 (TPM_PP_(*))
Other:
- note added: "BOOT MODES"
- note added: "LEDS"
- moved on the sheet: D6, R16, SW1

Commit message: Update.
Connections:
- net GND: now also J1.B25 (USB_SSTX1-_(*)), J1.B30 (AC/HDA_SDIN0_(**)); no longer J1.B27 (WDT), J1.B32 (SPKR)
- net GPIO0: now also J1.B82 (DDI0_PAIR3-); no longer J1.B79 (eDP/LVDS_BKLT_EN)
- net GPIO1: now also J1.B81 (DDI0_PAIR3+); no longer J1.B78 (DDI0_PAIR4-_(*))
- net GPIO10: now also J1.B73 (DDI0_PAIR1+); no longer J1.B70 (GND(FIXED))
- net GPIO12: now also J1.B70 (GND(FIXED)); no longer J1.B67 (WAKE1#_(**))
- net GPIO13: now also J1.B69 (PCIE_RX0-); no longer J1.B66 (WAKE0#)
- net GPIO14: now also J1.B67 (WAKE1#_(**)); no longer J1.B64 (PCIE_RX1+)
- net GPIO15: now also J1.B66 (WAKE0#); no longer J1.B63 (GPO3)
- net GPIO3: now also J1.B84 (VCC_5V_SBY); no longer J1.B81 (DDI0_PAIR3+)
- net GPIO4: now also J1.B86 (VCC_5V_SBY); no longer J1.B83 (eDP/LVDS_BKLT_CTRL)
- net GPIO5: now also J1.B79 (eDP/LVDS_BKLT_EN); no longer J1.B76 (DDI0_PAIR2-)
- net GPIO6: now also J1.B78 (DDI0_PAIR4-_(*)); no longer J1.B75 (DDI0_PAIR2+)
- net GPIO8: now also J1.B76 (DDI0_PAIR2-); no longer J1.B73 (DDI0_PAIR1+)
- net GPIO9: now also J1.B75 (DDI0_PAIR2+); no longer J1.B72 (DDI0_PAIR0-)
- net HDMI_AUX_N: now also J1.A59 (PCIE_TX3-); no longer J1.A56 (RSVD)
- net HDMI_AUX_P: now also J1.A58 (PCIE_TX3+); no longer J1.A55 (RSVD)
- net HDMI_CEC: now also J1.A65 (PCIE_TX1-); no longer J1.A62 (PCIE_TX2-)
- net HDMI_HDP: now also J1.A64 (PCIE_TX1+); no longer J1.A61 (PCIE_TX2+)
- net HDMI_REFCLK_N: now also J1.A49 (EXCD0_CPPE#); no longer J1.A46 (USB1_DP)
- net HDMI_REFCLK_P: now also J1.A50 (LPC_SERIRQ_(**)); no longer J1.A47 (VCC_RTC)
- net HDMI_SCL: now also J1.A62 (PCIE_TX2-); no longer J1.A59 (PCIE_TX3-)
- net HDMI_SDA: now also J1.A61 (PCIE_TX2+); no longer J1.A58 (PCIE_TX3+)
- net HDMI_TX0_N: now also J1.A53 (RSVD); no longer J1.A50 (LPC_SERIRQ_(**))
- net HDMI_TX0_P: now also J1.A52 (RSVD); no longer J1.A49 (EXCD0_CPPE#)
- net HDMI_TX1_N: now also J1.A55 (RSVD); no longer J1.A52 (RSVD)
- net HDMI_TX1_P: now also J1.A56 (RSVD); no longer J1.A53 (RSVD)
- net HDMI_TX2_N: now also J1.A47 (VCC_RTC); no longer J1.A44 (GND(FIXED))
- net HDMI_TX2_P: now also J1.A46 (USB1_DP); no longer J1.A43 (USB1_TX_P)
- net HDMI_TX3_N: now also J1.A43 (USB1_TX_P); no longer J1.A40 (USB1_RX_P)
- net HDMI_TX3_P: now also J1.A44 (GND(FIXED)); no longer J1.A41 (GND(FIXED))
- net I2C1_SCL: now also J1.B57 (GPO2); no longer J1.B54 (GPO1)
- net I2C1_SDA: now also J1.B58 (PCIE_RX3+); no longer J1.B55 (RSVD)
- net I2C2_SCL: now also J1.B61 (PCIE_RX2+); no longer J1.B58 (PCIE_RX3+)
- net I2C2_SDA: now also J1.B60 (GND(FIXED)); no longer J1.B57 (GPO2)
- net I2C3_SCL: now also J1.B63 (GPO3); no longer J1.B60 (GND(FIXED))
- net I2C3_SDA: now also J1.B64 (PCIE_RX1+); no longer J1.B61 (PCIE_RX2+)
- net PCIE1_REF_CLKN: now also J1.B45 (USB1-); no longer J1.B42 (USB3-)
- net PCIE1_REF_CLKP: now also J1.B46 (USB1+); no longer J1.B43 (USB3+)
- net PCIE1_RXN: now also J1.B52 (RSVD); no longer J1.B49 (SYS_RESET#)
- net PCIE1_RXP: now also J1.B51 (GND(FIXED)); no longer J1.B48 (EXCD1_CPPE#)
- net PCIE1_TXN: now also J1.B49 (SYS_RESET#); no longer J1.B46 (USB1+)
- net PCIE1_TXP: now also J1.B48 (EXCD1_CPPE#); no longer J1.B45 (USB1-)
- net PCIE2_REF_CLKN: now also J1.B42 (USB3-); no longer J1.B39 (USB5-)
- net PCIE2_REF_CLKP: now also J1.B43 (USB3+); no longer J1.B40 (USB5+)
- net PCIE2_RXN: now also J1.B39 (USB5-); no longer J1.B36 (USB7-_(*))
- net PCIE2_RXP: now also J1.B40 (USB5+); no longer J1.B37 (USB7+_(*))
- net PCIE2_TXN: now also J1.B36 (USB7-_(*)); no longer J1.B33 (I2C_CK)
- net PCIE2_TXP: now also J1.B37 (USB7+_(*)); no longer J1.B34 (I2C_DAT)
- net SPI1_MISO: now also J1.B34 (I2C_DAT); no longer J1.B31 (GND(FIXED))
- net SPI1_MOSI: now also J1.B33 (I2C_CK); no longer J1.B30 (AC/HDA_SDIN0_(**))
- net SPI1_SCLK: now also J1.B31 (GND(FIXED)); no longer J1.B28 (AC/HDA_SDIN2_(*))
- net SPI1_SSO: now also J1.B32 (SPKR); no longer J1.B29 (AC/HDA_SDIN1_(*))
- net SPI2_MISO: now also J1.B29 (AC/HDA_SDIN1_(*)); no longer J1.B26 (USB_SSTX1+_(*))
- net SPI2_MOSI: now also J1.B28 (AC/HDA_SDIN2_(*)); no longer J1.B25 (USB_SSTX1-_(*))
- net SPI2_SCLK: now also J1.B26 (USB_SSTX1+_(*)); no longer J1.B23 (USB_SSTX0+)
- net SPI2_SSO: now also J1.B27 (WDT); no longer J1.B24 (PWR_OK)
- net UART1_RXD: now also J1.B18 (SUS_STAT#); no longer J1.B15 (SMB_ALERT#)
- net UART1_TXD: now also J1.B17 (SATA1_TX-); no longer J1.B14 (SMB_DAT)
- net UART2_RXD: now also J1.B23 (USB_SSTX0+); no longer J1.B20 (SATA1_RX-)
- net UART2_TXD: now also J1.B24 (PWR_OK); no longer J1.B21 (GND(FIXED))
- net UART3_RXD: now also J1.B21 (GND(FIXED)); no longer J1.B18 (SUS_STAT#)
- net UART3_TXD: now also J1.B20 (SATA1_RX-); no longer J1.B17 (SATA1_TX-)
- net UART4_RXD: now also J1.B54 (GPO1); no longer J1.B51 (GND(FIXED))
- net UART4_TXD: now also J1.B55 (RSVD); no longer J1.B52 (RSVD)
- new net USB1_OC: J1.A40 (USB1_RX_P)
- new net USB1_PWR_EN: J1.A41 (GND(FIXED))
- new net USB2_OC: J1.B15 (SMB_ALERT#)
- new net USB2_PWR_EN: J1.B14 (SMB_DAT)

Commit message: Update.
Connections:
- net BOOT_SEL: now also J1.A69 (PCIE_TX0-); no longer J1.A67 (GPI2)
- net GND: now also J1.A43 (USB1_TX_P), J1.A44 (GND(FIXED)), J1.A47 (VCC_RTC), J1.A50 (LPC_SERIRQ_(**)), J1.A53 (RSVD), J1.A56 (RSVD), J1.A59 (PCIE_TX3-), J1.A62 (PCIE_TX2-), J1.A65 (PCIE_TX1-), J1.A68 (PCIE_TX0+), J1.B83 (eDP/LVDS_BKLT_CTRL); no longer J1.A42 (USB1_TX_N), J1.A45 (USB1_DN), J1.A48 (EXCD0_PERST#), J1.A51 (GND(FIXED)), J1.A54 (GPI0), J1.A57 (GND), J1.A60 (GND(FIXED)), J1.A63 (GPI1), J1.A66 (GND), J1.A70 (GND(FIXED))
- net GPIO0: now also J1.B81 (DDI0_PAIR3+); no longer J1.B82 (DDI0_PAIR3-)
- net GPIO1: now also J1.B79 (eDP/LVDS_BKLT_EN); no longer J1.B81 (DDI0_PAIR3+)
- net GPIO10: now also J1.B72 (DDI0_PAIR0-); no longer J1.B73 (DDI0_PAIR1+)
- net GPIO3: now also J1.B82 (DDI0_PAIR3-); no longer J1.B84 (VCC_5V_SBY)
- net GPIO4: now also J1.B84 (VCC_5V_SBY); no longer J1.B86 (VCC_5V_SBY)
- net GPIO5: now also J1.B78 (DDI0_PAIR4-_(*)); no longer J1.B79 (eDP/LVDS_BKLT_EN)
- net GPIO6: now also J1.B76 (DDI0_PAIR2-); no longer J1.B78 (DDI0_PAIR4-_(*))
- net GPIO8: now also J1.B75 (DDI0_PAIR2+); no longer J1.B76 (DDI0_PAIR2-)
- net GPIO9: now also J1.B73 (DDI0_PAIR1+); no longer J1.B75 (DDI0_PAIR2+)
- net HDMI_AUX_N: now also J1.A61 (PCIE_TX2+); no longer J1.A59 (PCIE_TX3-)
- net HDMI_AUX_P: now also J1.A60 (GND(FIXED)); no longer J1.A58 (PCIE_TX3+)
- net HDMI_CEC: now also J1.A67 (GPI2); no longer J1.A65 (PCIE_TX1-)
- net HDMI_HDP: now also J1.A66 (GND); no longer J1.A64 (PCIE_TX1+)
- net HDMI_REFCLK_N: now also J1.A51 (GND(FIXED)); no longer J1.A49 (EXCD0_CPPE#)
- net HDMI_REFCLK_P: now also J1.A52 (RSVD); no longer J1.A50 (LPC_SERIRQ_(**))
- net HDMI_SCL: now also J1.A64 (PCIE_TX1+); no longer J1.A62 (PCIE_TX2-)
- net HDMI_SDA: now also J1.A63 (GPI1); no longer J1.A61 (PCIE_TX2+)
- net HDMI_TX0_N: now also J1.A55 (RSVD); no longer J1.A53 (RSVD)
- net HDMI_TX0_P: now also J1.A54 (GPI0); no longer J1.A52 (RSVD)
- net HDMI_TX1_N: now also J1.A57 (GND); no longer J1.A55 (RSVD)
- net HDMI_TX1_P: now also J1.A58 (PCIE_TX3+); no longer J1.A56 (RSVD)
- net HDMI_TX2_N: now also J1.A49 (EXCD0_CPPE#); no longer J1.A47 (VCC_RTC)
- net HDMI_TX2_P: now also J1.A48 (EXCD0_PERST#); no longer J1.A46 (USB1_DP)
- net HDMI_TX3_N: now also J1.A45 (USB1_DN); no longer J1.A43 (USB1_TX_P)
- net HDMI_TX3_P: now also J1.A46 (USB1_DP); no longer J1.A44 (GND(FIXED))
- new net USB1_ID1: J1.A42 (USB1_TX_N)
- no-connect marks 19 -> 39
Other:
- moved on the sheet: C334, C335
