File: DQBSC/MEM.kicad_sch (KiCad schematic)
At the start: 58 parts, among them U26 W25Q32JWSSIQ, U3 MT53E1G32D2FW-046_WT:A, U4 SDINBDG4-16G-I2, U6 IS25LP256D-JLLE

Commit message: Update.
Parts:
- removed C279, C358: 220nF, awg1000:C0201_L, symbol awg1000:CAP_UNPOL
- removed R16, R17, R19: 0, Resistor_SMD:R_0402_1005Metric, symbol DQSBC:R_US
- removed R61, R62: 49.9, Resistor_SMD:R_0402_1005Metric, symbol awg1000:R
- removed U26: W25Q32JWSSIQ, Package_SO:SOIC-8_3.9x4.9mm_P1.27mm, symbol awg1000:W25Q32JWSSIQ
Connections:
- net QSPIA_IO0 is gone; now on net NAND_DATA3: U6.5 (IO0)
- net QSPIA_IO1 is gone; now on net NAND_DATA0: U6.2 (IO1)
- net QSPIA_IO2 is gone; now on net NAND_DATA1: U6.3 (IO2)
- net QSPIA_IO3 is gone; now on net NAND_DATA2: U6.7 (IO3)
- net NAND_DATA0: no longer R15.1, U4.A3 (D0)
- net NAND_DATA1: no longer U4.A4 (D1)
- net NAND_DATA2: no longer U4.A5 (D2)
- net NAND_DATA3: no longer U4.B2 (D3)
- net SD1_CLK: now also U4.M6 (CLK)
- net SD1_STROBE: now also U4.H5 (RCLK)
- net SD1_nRST: now also R83.1, U4.K5 (NRST)
- net NAND_DATA4 renamed SD1_D4
- net NAND_DATA5 renamed SD1_D5
- net NAND_DATA6 renamed SD1_D6
- net NAND_DATA7 renamed SD1_D7
- new net SD1_D0: R15.1, U4.A3 (D0)
- new net SD1_D1: U4.A4 (D1)
- new net SD1_D2: U4.A5 (D2)
- new net SD1_D3: U4.B2 (D3)
Other:
- note removed: "MPU NOR FLASH"
- moved on the sheet: C354, C357

Commit message: UPDATE, FULL ROUTING!
Connections:
- net DRAMREF: now also R67.2; no longer R67.1
- net DRAM_VREF: now also R67.1; no longer R67.2
- net QSPIA_SCK renamed QSPIA_SCLK
Other:
- moved on the sheet: R67
Changed lines of the file:
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@@
   (junction (at 175.26 111.76) (diameter 0) (color 0 0 0 0)
   )
-  (junction (at 93.98 248.92) (diameter 0) (color 0 0 0 0)
+  (junction (at 99.06 248.92) (diameter 0) (color 0 0 0 0)
   )
   (junction (at 175.26 185.42) (diameter 0) (color 0 0 0 0)
@@
     (stroke (width 0) (type default))
   )
-  (wire (pts (xy 86.36 248.92) (xy 93.98 248.92))
-    (stroke (width 0) (type default))
-  )
   (wire (pts (xy 322.58 223.52) (xy 325.12 223.52))
     (stroke (width 0) (type default))
@@
     (stroke (width 0) (type default))
   )
-  (wire (pts (xy 93.98 246.38) (xy 93.98 248.92))
+  (wire (pts (xy 99.06 246.38) (xy 99.06 248.92))
     (stroke (width 0) (type default))
   )
@@
     (stroke (width 0) (type default))
   )
-  (wire (pts (xy 93.98 236.22) (xy 93.98 238.76))
+  (wire (pts (xy 99.06 236.22) (xy 99.06 238.76))
     (stroke (width 0) (type default))
   )
@@
     (stroke (width 0) (type default))
   )
-  (wire (pts (xy 93.98 248.92) (xy 93.98 255.27))
+  (wire (pts (xy 99.06 248.92) (xy 99.06 255.27))
     (stroke (width 0) (type default))
   )
@@
     (stroke (width 0) (type default))
   )
+  (wire (pts (xy 86.36 248.92) (xy 99.06 248.92))
+    (stroke (width 0) (type default))
+  )
   (wire (pts (xy 45.72 104.14) (xy 50.8 104.14))
     (stroke (width 0) (type default))
@@
     (effects (font (size 1.27 1.27)) (justify left bottom))
   )
-  (label "DRAMREF" (at 83.82 248.92 0) (fields_autoplaced)
+  (label "DRAMREF" (at 87.63 248.92 0) (fields_autoplaced)
     (effects (font (size 1.27 1.27)) (justify left bottom))
   )
@@
     )
   )
+  (global_label "QSPIA_SCLK" (shape output) (at 317.5 83.82 0) (fields_autoplaced)
+    (effects (font (size 1 1)) (justify left))
+    (property "Intersheetrefs" "${INTERSHEET_REFS}" (at 328.7074 83.82 0)
+      (effects (font (size 1.27 1.27)) (justify left) hide)
+    )
+  )
   (global_label "DRAM_CA0_A" (shape output) (at 45.72 76.2 180) (fields_autoplaced)
     (effects (font (size 1 1)) (justify right))
@@
     )
   )
-  (global_label "DRAMREF" (shape bidirectional) (at 93.98 255.27 270) (fields_autoplaced)
+  (global_label "DRAMREF" (shape bidirectional) (at 99.06 255.27 270) (fields_autoplaced)
     (effects (font (size 1.27 1.27)) (justify right))
-    (property "Intersheetrefs" "${INTERSHEET_REFS}" (at 93.98 267.7159 90)
+    (property "Intersheetrefs" "${INTERSHEET_REFS}" (at 99.06 267.7159 90)
       (effects (font (size 1.27 1.27)) (justify right) hide)
     )
@@
     )
   )
-  (global_label "QSPIA_SCK" (shape output) (at 317.5 83.82 0) (fields_autoplaced)
-    (effects (font (size 1 1)) (justify left))
-    (property "Intersheetrefs" "${INTERSHEET_REFS}" (at 327.7105 83.82 0)
-      (effects (font (size 1.27 1.27)) (justify left) hide)
-    )
-  )
   (global_label "DRAM_CKE0_B" (shape output) (at 45.72 111.76 180) (fields_autoplaced)
     (effects (font (size 1 1)) (justify right))
@@
   (symbol (lib_id "DQSBC:C") (at 86.36 254 0) (unit 1)
     (exclude_from_sim no) (in_bom yes) (on_board yes) (dnp no)
-    (property "Reference" "C318" (at 88.265 252.095 0)
+    (property "Reference" "C318" (at 88.265 251.46 0)
       (effects (font (size 1.27 1.27) (color 132 0 0 1)) (justify left))
     )
@@
   (symbol (lib_id "DQSBC:C") (at 86.36 241.3 0) (unit 1)
     (exclude_from_sim no) (in_bom yes) (on_board yes) (dnp no)
-    (property "Reference" "C317" (at 88.265 239.395 0)
+    (property "Reference" "C317" (at 88.265 238.76 0)
       (effects (font (size 1.27 1.27) (color 132 0 0 1)) (justify left))
     )
@@
     )
   )
-  (symbol (lib_id "awg1000:DRAM_VREF") (at 93.98 236.22 0) (unit 1)
+  (symbol (lib_id "awg1000:DRAM_VREF") (at 99.06 236.22 0) (unit 1)
     (exclude_from_sim no) (in_bom yes) (on_board yes) (dnp no)
-    (property "Reference" "#PWR0189" (at 93.98 238.76 0)
+    (property "Reference" "#PWR0189" (at 99.06 238.76 0)
       (effects (font (size 1.27 1.27)) hide)
     )
-    (property "Value" "DRAM_VREF" (at 93.98 227.965 90)
+    (property "Value" "DRAM_VREF" (at 99.06 232.41 0)
       (effects (font (size 1.27 1.27)))
     )
-    (property "Footprint" "" (at 93.98 236.22 0)
+    (property "Footprint" "" (at 99.06 236.22 0)
       (effects (font (size 1.27 1.27)) hide)
     )
-    (property "Datasheet" "" (at 93.98 236.22 0)
+    (property "Datasheet" "" (at 99.06 236.22 0)
       (effects (font (size 1.27 1.27)) hide)
     )
-    (property "Description" "" (at 93.98 236.22 0)
+    (property "Description" "" (at 99.06 236.22 0)
       (effects (font (size 1.27 1.27)) hide)
     )
@@
     )
   )
-  (symbol (lib_id "DQSBC:R_US") (at 93.98 242.57 180) (unit 1)
+  (symbol (lib_id "DQSBC:R_US") (at 99.06 242.57 0) (mirror y) (unit 1)
     (exclude_from_sim no) (in_bom yes) (on_board yes) (dnp no)
-    (property "Reference" "R67" (at 94.742 238.76 90)
+    (property "Reference" "R67" (at 101.6 244.475 90)
       (effects (font (size 1.27 1.27)))
     )
-    (property "Value" "0" (at 94.742 246.634 90)
+    (property "Value" "0" (at 101.6 239.395 90)
       (effects (font (size 1.27 1.27)))
     )
-    (property "Footprint" "Resistor_SMD:R_0402_1005Metric" (at 92.964 242.316 90)
+    (property "Footprint" "Resistor_SMD:R_0402_1005Metric" (at 98.044 242.824 90)
       (effects (font (size 1.27 1.27)) hide)
     )
-    (property "Datasheet" "~" (at 93.98 242.57 0)
+    (property "Datasheet" "~" (at 99.06 242.57 0)
       (effects (font (size 1.27 1.27)) hide)
     )
-    (property "Description" "" (at 93.98 242.57 0)
+    (property "Description" "" (at 99.06 242.57 0)
       (effects (font (size 1.27 1.27)) hide)
     )

Commit message: Update.
Other:
- moved on the sheet: C354, C357
Changed lines of the file:
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@@
   (junction (at 327.66 208.28) (diameter 0) (color 0 0 0 0)
   )
-  (junction (at 284.48 55.88) (diameter 0.9144) (color 0 0 0 0)
+  (junction (at 284.48 53.34) (diameter 0.9144) (color 0 0 0 0)
   )
   (junction (at 129.54 236.22) (diameter 0) (color 0 0 0 0)
@@
   (junction (at 175.26 116.84) (diameter 0) (color 0 0 0 0)
   )
+  (junction (at 284.48 60.96) (diameter 0) (color 0 0 0 0)
+  )
   (junction (at 175.26 124.46) (diameter 0) (color 0 0 0 0)
   )
@@
   (junction (at 167.64 236.22) (diameter 0) (color 0 0 0 0)
   )
-  (junction (at 284.48 66.04) (diameter 0.9144) (color 0 0 0 0)
-  )
   (junction (at 137.16 256.54) (diameter 0) (color 0 0 0 0)
   )
@@
     (stroke (width 0) (type default))
   )
-  (wire (pts (xy 284.48 66.04) (xy 294.64 66.04))
+  (wire (pts (xy 284.48 60.96) (xy 294.64 60.96))
     (stroke (width 0) (type solid))
   )
@@
     (stroke (width 0) (type default))
   )
-  (wire (pts (xy 284.48 54.61) (xy 284.48 55.88))
+  (wire (pts (xy 284.48 50.8) (xy 284.48 53.34))
     (stroke (width 0) (type solid))
   )
@@
     (stroke (width 0) (type default))
   )
-  (wire (pts (xy 284.48 55.88) (xy 284.48 57.15))
-    (stroke (width 0) (type solid))
-  )
   (wire (pts (xy 172.72 167.64) (xy 175.26 167.64))
     (stroke (width 0) (type default))
@@
     (stroke (width 0) (type default))
   )
-  (wire (pts (xy 284.48 55.88) (xy 294.64 55.88))
+  (wire (pts (xy 284.48 53.34) (xy 294.64 53.34))
     (stroke (width 0) (type solid))
   )
@@
     (stroke (width 0) (type default))
   )
-  (wire (pts (xy 284.48 64.77) (xy 284.48 66.04))
-    (stroke (width 0) (type solid))
-  )
   (wire (pts (xy 347.98 190.5) (xy 347.98 193.04))
     (stroke (width 0) (type default))
@@
     (stroke (width 0) (type default))
   )
-  (wire (pts (xy 294.64 55.88) (xy 294.64 57.15))
-    (stroke (width 0) (type solid))
-  )
   (wire (pts (xy 134.62 60.96) (xy 134.62 63.5))
     (stroke (width 0) (type default))
@@
     (stroke (width 0) (type default))
   )
-  (wire (pts (xy 284.48 66.04) (xy 284.48 67.31))
-    (stroke (width 0) (type solid))
-  )
   (wire (pts (xy 81.28 233.68) (xy 81.28 236.22))
     (stroke (width 0) (type default))
@@
     (stroke (width 0) (type default))
   )
-  (wire (pts (xy 99.06 248.92) (xy 99.06 255.27))
+  (wire (pts (xy 99.06 248.92) (xy 99.06 254))
     (stroke (width 0) (type default))
   )
@@
     (stroke (width 0) (type default))
   )
-  (wire (pts (xy 294.64 66.04) (xy 294.64 64.77))
-    (stroke (width 0) (type solid))
+  (wire (pts (xy 284.48 63.5) (xy 284.48 60.96))
+    (stroke (width 0) (type default))
   )
   (wire (pts (xy 175.26 71.12) (xy 175.26 73.66))
@@
     )
   )
-  (global_label "DRAMREF" (shape bidirectional) (at 99.06 255.27 270) (fields_autoplaced)
+  (global_label "DRAMREF" (shape bidirectional) (at 99.06 254 270) (fields_autoplaced)
     (effects (font (size 1.27 1.27)) (justify right))
-    (property "Intersheetrefs" "${INTERSHEET_REFS}" (at 99.06 267.7159 90)
+    (property "Intersheetrefs" "${INTERSHEET_REFS}" (at 99.06 266.4459 90)
       (effects (font (size 1.27 1.27)) (justify right) hide)
     )
@@
   (symbol (lib_id "DQSBC:SDINBDG4-16G-I2") (at 281.94 190.5 0) (unit 1)
     (exclude_from_sim no) (in_bom yes) (on_board yes) (dnp no)
-    (property "Reference" "U4" (at 282.448 188.214 0)
+    (property "Reference" "U4" (at 283.21 187.96 0)
       (effects (font (size 1.27 1.27)))
     )
@@
     )
   )
-  (symbol (lib_name "awg1000:CAP_UNPOL_70") (lib_id "awg1000:CAP_UNPOL") (at 294.64 60.96 0) (unit 1)
+  (symbol (lib_name "awg1000:CAP_UNPOL_70") (lib_id "awg1000:CAP_UNPOL") (at 294.64 57.15 0) (unit 1)
     (exclude_from_sim no) (in_bom yes) (on_board yes) (dnp no)
-    (property "Reference" "C357" (at 296.926 59.436 0)
+    (property "Reference" "C357" (at 296.926 55.626 0)
       (effects (font (size 1.27 1.27)) (justify left))
     )
-    (property "Value" "220nF" (at 296.926 60.96 0)
+    (property "Value" "220nF" (at 296.926 57.15 0)
       (effects (font (size 1.27 1.27)) (justify left))
     )
-    (property "Footprint" "awg1000:C0201_L" (at 295.6052 64.77 0)
+    (property "Footprint" "awg1000:C0201_L" (at 295.6052 60.96 0)
       (effects (font (size 1.27 1.27)) hide)
     )
-    (property "Datasheet" "~" (at 295.402 59.944 0)
+    (property "Datasheet" "~" (at 295.402 56.134 0)
       (effects (font (size 1.27 1.27)) hide)
     )
-    (property "Description" "" (at 294.64 60.96 0)
+    (property "Description" "" (at 294.64 57.15 0)
       (effects (font (size 1.27 1.27)) hide)
     )
-    (property "VOLTAGE" "16V" (at 297.053 62.484 0)
+    (property "VOLTAGE" "16V" (at 297.053 58.674 0)
       (effects (font (size 1.27 1.27)) (justify left))
     )
@@
     )
   )
-  (symbol (lib_id "DQSBC:3.3V_SW_DELAYED") (at 284.48 54.61 0) (unit 1)
+  (symbol (lib_id "DQSBC:3.3V_SW_DELAYED") (at 284.48 50.8 0) (unit 1)
     (exclude_from_sim no) (in_bom yes) (on_board yes) (dnp no)
-    (property "Reference" "#PWR0254" (at 284.48 55.88 0)
+    (property "Reference" "#PWR0254" (at 284.48 52.07 0)
       (effects (font (size 1.27 1.27)) hide)
     )
-    (property "Value" "3.3V_SW_DELAYED" (at 284.48 51.054 0)
+    (property "Value" "3.3V_SW_DELAYED" (at 284.48 47.244 0)
       (effects (font (size 1.27 1.27)))
     )
-    (property "Footprint" "" (at 284.48 54.61 0)
+    (property "Footprint" "" (at 284.48 50.8 0)
       (effects (font (size 1.27 1.27)) hide)
     )
-    (property "Datasheet" "" (at 284.48 54.61 0)
+    (property "Datasheet" "" (at 284.48 50.8 0)
       (effects (font (size 1.27 1.27)) hide)
     )
-    (property "Description" "" (at 284.48 54.61 0)
+    (property "Description" "" (at 284.48 50.8 0)
       (effects (font (size 1.27 1.27)) hide)
     )
@@
     )
   )
-  (symbol (lib_id "DQSBC:GND") (at 284.48 67.31 0) (unit 1)
+  (symbol (lib_id "DQSBC:GND") (at 284.48 63.5 0) (unit 1)
     (exclude_from_sim no) (in_bom yes) (on_board yes) (dnp no)
-    (property "Reference" "#PWR0362" (at 283.845 73.025 0)
+    (property "Reference" "#PWR0362" (at 283.845 69.215 0)
       (effects (font (size 1.27 1.27)) hide)
     )
-    (property "Value" "GND" (at 284.48 71.12 0)
+    (property "Value" "GND" (at 284.48 67.31 0)
       (effects (font (size 1.27 1.27) (color 255 0 0 1)))
     )
-    (property "Footprint" "" (at 284.48 67.31 0)
+    (property "Footprint" "" (at 284.48 63.5 0)
       (effects (font (size 1.27 1.27)) hide)
     )
-    (property "Datasheet" "" (at 284.48 67.31 0)
+    (property "Datasheet" "" (at 284.48 63.5 0)
       (effects (font (size 1.27 1.27)) hide)
     )
-    (property "Description" "" (at 284.48 67.31 0)
+    (property "Description" "" (at 284.48 63.5 0)
       (effects (font (size 1.27 1.27)) hide)
     )
@@
     )
   )
-  (symbol (lib_name "awg1000:CAP_UNPOL_68") (lib_id "awg1000:CAP_UNPOL") (at 284.48 60.96 0) (unit 1)
+  (symbol (lib_name "awg1000:CAP_UNPOL_68") (lib_id "awg1000:CAP_UNPOL") (at 284.48 57.15 0) (unit 1)
     (exclude_from_sim no) (in_bom yes) (on_board yes) (dnp no)
-    (property "Reference" "C354" (at 286.766 59.436 0)
+    (property "Reference" "C354" (at 286.766 55.626 0)
       (effects (font (size 1.27 1.27)) (justify left))
     )
-    (property "Value" "22uF" (at 286.766 60.96 0)
+    (property "Value" "22uF" (at 286.766 57.15 0)
       (effects (font (size 1.27 1.27)) (justify left))
     )
-    (property "Footprint" "Resistor_SMD:R_0402_1005Metric_Pad0.72x0.64mm_HandSolder" (at 285.4452 64.77 0)
+    (property "Footprint" "Resistor_SMD:R_0402_1005Metric_Pad0.72x0.64mm_HandSolder" (at 285.4452 60.96 0)
       (effects (font (size 1.27 1.27)) hide)
     )
-    (property "Datasheet" "~" (at 285.242 59.944 0)
+    (property "Datasheet" "~" (at 285.242 56.134 0)
       (effects (font (size 1.27 1.27)) hide)
     )
-    (property "Description" "" (at 284.48 60.96 0)
+    (property "Description" "" (at 284.48 57.15 0)
       (effects (font (size 1.27 1.27)) hide)
     )
-    (property "VOLTAGE" "10V" (at 286.893 62.484 0)
+    (property "VOLTAGE" "10V" (at 286.893 58.674 0)
       (effects (font (size 1.27 1.27)) (justify left))
     )
