File: DQBSC/PWR.kicad_sch (KiCad schematic)
At the start: 132 parts, among them Q2 2SK3018-TP, Q3 SI7309DN-T1-E3, U10 TPS54531DDA, U13 APX811-26UG-7, U14 TPS62840, U2 SIC402ACD-T1-GE3, U7 TPS78412QDBVRQ1, U8 MC34PF4210A1ES, U9 TPS54531DDA

Commit message: Update.
Parts:
- removed U13: APX811-26UG-7, Package_TO_SOT_SMD:SOT-143, symbol DQSBC:APX811-26UG-7
Connections:
- net 3.3V_SW_DELAYED: no longer U10.3 (EN)
- new net SOC_0V9_EN: U10.3 (EN)
Other:
- moved on the sheet: L11
Changed lines of the file:
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@@
   (junction (at 33.02 175.26) (diameter 0) (color 0 0 0 0)
   )
-  (junction (at 259.08 50.8) (diameter 0) (color 0 0 0 0)
-  )
   (junction (at 358.14 40.64) (diameter 0) (color 0 0 0 0)
   )
@@
     (stroke (width 0) (type solid))
   )
-  (wire (pts (xy 294.64 48.26) (xy 297.18 48.26))
+  (wire (pts (xy 293.37 48.26) (xy 297.18 48.26))
     (stroke (width 0) (type solid))
   )
@@
     (stroke (width 0) (type default))
   )
-  (wire (pts (xy 254 190.5) (xy 254 193.04))
-    (stroke (width 0) (type default))
-  )
-  (wire (pts (xy 264.16 53.34) (xy 259.08 53.34))
+  (wire (pts (xy 254 53.34) (xy 264.16 53.34))
     (stroke (width 0) (type solid))
   )
@@
     (stroke (width 0) (type solid))
   )
-  (wire (pts (xy 259.08 53.34) (xy 259.08 50.8))
-    (stroke (width 0) (type solid))
-  )
   (wire (pts (xy 157.48 127) (xy 160.02 127))
     (stroke (width 0) (type default))
@@
     (stroke (width 0) (type default))
   )
-  (wire (pts (xy 251.46 198.12) (xy 259.08 198.12))
-    (stroke (width 0) (type default))
-  )
   (wire (pts (xy 231.14 152.4) (xy 231.14 154.94))
     (stroke (width 0) (type default))
@@
     (stroke (width 0) (type default))
   )
-  (wire (pts (xy 254 193.04) (xy 251.46 193.04))
-    (stroke (width 0) (type default))
-  )
   (wire (pts (xy 50.8 35.56) (xy 50.8 30.48))
     (stroke (width 0) (type default))
@@
     (stroke (width 0) (type solid))
   )
+  (wire (pts (xy 254 50.8) (xy 254 53.34))
+    (stroke (width 0) (type solid))
+  )
   (wire (pts (xy 119.38 152.4) (xy 119.38 154.94))
     (stroke (width 0) (type default))
@@
     (stroke (width 0) (type default))
   )
-  (wire (pts (xy 281.94 48.26) (xy 287.02 48.26))
+  (wire (pts (xy 281.94 48.26) (xy 285.75 48.26))
     (stroke (width 0) (type solid))
   )
@@
     (stroke (width 0) (type solid))
   )
-  (wire (pts (xy 231.14 193.04) (xy 233.68 193.04))
-    (stroke (width 0) (type default))
-  )
   (polyline (pts (xy 271.78 99.06) (xy 271.78 275.971))
     (stroke (width 0) (type default) (color 132 0 0 1))
@@
     )
   )
+  (global_label "SOC_0V9_EN" (shape input) (at 254 50.8 90) (fields_autoplaced)
+    (effects (font (size 1.016 1.016)) (justify left))
+    (property "Intersheetrefs" "${INTERSHEET_REFS}" (at 254 39.0262 90)
+      (effects (font (size 1.27 1.27)) (justify left) hide)
+    )
+  )
   (symbol (lib_id "DQSBC:MC32PF4210A3ES") (at 121.92 124.46 0) (unit 3)
     (exclude_from_sim no) (in_bom yes) (on_board yes) (dnp no)
@@
     )
   )
-  (symbol (lib_id "Device:L") (at 290.83 48.26 90) (unit 1)
+  (symbol (lib_id "Device:L") (at 289.56 48.26 90) (unit 1)
     (exclude_from_sim no) (in_bom yes) (on_board yes) (dnp no)
-    (property "Reference" "L11" (at 286.512 47.244 90)
+    (property "Reference" "L11" (at 285.242 47.244 90)
       (effects (font (size 1.27 1.27)))
     )
-    (property "Value" "47uH" (at 295.656 47.117 90)
+    (property "Value" "47uH" (at 294.386 47.117 90)
       (effects (font (size 1.27 1.27)))
     )
-    (property "Footprint" "Inductor_SMD:L_Bourns_SRR1260" (at 290.83 48.26 0)
+    (property "Footprint" "Inductor_SMD:L_Bourns_SRR1260" (at 289.56 48.26 0)
       (effects (font (size 1.27 1.27)) hide)
     )
-    (property "Datasheet" "~" (at 290.83 48.26 0)
+    (property "Datasheet" "~" (at 289.56 48.26 0)
       (effects (font (size 1.27 1.27)) hide)
     )
-    (property "Description" "" (at 290.83 48.26 0)
+    (property "Description" "" (at 289.56 48.26 0)
       (effects (font (size 1.27 1.27)) hide)
     )
-    (property "Part Number" "SRR1280-470M" (at 293.116 46.736 90)
+    (property "Part Number" "SRR1280-470M" (at 291.846 46.736 90)
       (effects (font (size 1.27 1.27)) hide)
     )
@@
     )
   )
-  (symbol (lib_id "DQSBC:GND") (at 231.14 193.04 270) (unit 1)
-    (exclude_from_sim no) (in_bom yes) (on_board yes) (dnp no)
-    (property "Reference" "#PWR0181" (at 224.79 193.04 0)
-      (effects (font (size 1.27 1.27)) hide)
-    )
-    (property "Value" "GND" (at 227.33 193.04 0)
-      (effects (font (size 1.27 1.27) (color 255 0 0 1)))
-    )
-    (property "Footprint" "" (at 231.14 193.04 0)
-      (effects (font (size 1.27 1.27)) hide)
-    )
-    (property "Datasheet" "" (at 231.14 193.04 0)
-      (effects (font (size 1.27 1.27)) hide)
-    )
-    (property "Description" "" (at 231.14 193.04 0)
-      (effects (font (size 1.27 1.27)) hide)
-    )
-    (pin "1")
-    (instances
-      (project "DQBSC"
-        (path "/8aaed6d1-6388-4dfb-8015-aa095e997bfa/bd4d4a4a-feba-4969-9481-b8d6f4eb80d3"
-          (reference "#PWR0181") (unit 1)
-        )
-      )
-    )
-  )
   (symbol (lib_id "DQSBC:3.3V_SW") (at 96.52 40.64 0) (unit 1)
     (exclude_from_sim no) (in_bom yes) (on_board yes) (dnp no)
@@
     )
   )
-  (symbol (lib_name "awg1000:R_12") (lib_id "awg1000:R") (at 297.18 54.61 0) (unit 1)
+  (symbol (lib_name "awg1000:R_12") (lib_id "awg1000:R") (at 297.18 54.61 0) (mirror y) (unit 1)
     (exclude_from_sim no) (in_bom yes) (on_board yes) (dnp no)
-    (property "Reference" "R34" (at 296.418 56.896 90)
+    (property "Reference" "R34" (at 299.72 55.88 90)
       (effects (font (size 1.27 1.27)) (justify right))
     )
-    (property "Value" "7.15k" (at 296.418 52.578 90)
+    (property "Value" "7.15k" (at 299.72 53.34 90)
       (effects (font (size 1.27 1.27)) (justify left))
     )
-    (property "Footprint" "Resistor_SMD:R_0402_1005Metric_Pad0.72x0.64mm_HandSolder" (at 298.196 54.864 90)
+    (property "Footprint" "Resistor_SMD:R_0402_1005Metric_Pad0.72x0.64mm_HandSolder" (at 296.164 54.864 90)
       (effects (font (size 1.27 1.27)) hide)
     )
@@
     )
   )
-  (symbol (lib_id "DQSBC:3.3V_SW") (at 254 190.5 0) (unit 1)
-    (exclude_from_sim no) (in_bom yes) (on_board yes) (dnp no)
-    (property "Reference" "#PWR0102" (at 254 191.77 0)
-      (effects (font (size 1.27 1.27)) hide)
-    )
-    (property "Value" "3.3V_SW" (at 254 186.944 0)
-      (effects (font (size 1.27 1.27)))
-    )
-    (property "Footprint" "" (at 254 190.5 0)
-      (effects (font (size 1.27 1.27)) hide)
-    )
-    (property "Datasheet" "" (at 254 190.5 0)
-      (effects (font (size 1.27 1.27)) hide)
-    )
-    (property "Description" "" (at 254 190.5 0)
-      (effects (font (size 1.27 1.27)) hide)
-    )
-    (pin "1")
-    (instances
-      (project "DQBSC"
-        (path "/8aaed6d1-6388-4dfb-8015-aa095e997bfa/bd4d4a4a-feba-4969-9481-b8d6f4eb80d3"
-          (reference "#PWR0102") (unit 1)
-        )
-      )
-    )
-  )
   (symbol (lib_id "DQSBC:C") (at 121.92 218.44 0) (unit 1)
     (exclude_from_sim no) (in_bom yes) (on_board yes) (dnp no)
@@
     )
   )
-  (symbol (lib_name "awg1000:R_14") (lib_id "awg1000:R") (at 297.18 67.31 0) (unit 1)
+  (symbol (lib_name "awg1000:R_14") (lib_id "awg1000:R") (at 297.18 67.31 0) (mirror y) (unit 1)
     (exclude_from_sim no) (in_bom yes) (on_board yes) (dnp no)
-    (property "Reference" "R35" (at 296.418 69.596 90)
+    (property "Reference" "R35" (at 299.72 68.58 90)
       (effects (font (size 1.27 1.27)) (justify right))
     )
-    (property "Value" "7.15k" (at 296.418 65.278 90)
+    (property "Value" "7.15k" (at 299.72 66.04 90)
       (effects (font (size 1.27 1.27)) (justify left))
     )
-    (property "Footprint" "Resistor_SMD:R_0402_1005Metric_Pad0.72x0.64mm_HandSolder" (at 298.196 67.564 90)
+    (property "Footprint" "Resistor_SMD:R_0402_1005Metric_Pad0.72x0.64mm_HandSolder" (at 296.164 67.564 90)
       (effects (font (size 1.27 1.27)) hide)
     )
@@
         )
       )
-    )
-  )
-  (symbol (lib_id "DQSBC:APX811-26UG-7") (at 236.22 190.5 0) (unit 1)
-    (exclude_from_sim no) (in_bom yes) (on_board yes) (dnp no)
-    (property "Reference" "U13" (at 236.855 189.865 0)
-      (effects (font (size 1.27 1.27)))
-    )
-    (property "Value" "APX811-26UG-7" (at 244.475 201.93 0)
-      (effects (font (size 1.27 1.27)))
-    )
-    (property "Footprint" "Package_TO_SOT_SMD:SOT-143" (at 236.22 190.5 0)
-      (effects (font (size 1.27 1.27)) hide)
-    )
-    (property "Datasheet" "" (at 236.22 190.5 0)
-      (effects (font (size 1.27 1.27)) hide)
-    )
-    (property "Description" "" (at 236.22 190.5 0)
-      (effects (font (size 1.27 1.27)) hide)
-    )
-    (pin "1")
-    (pin "2")
-    (pin "3")
-    (pin "4")
-    (instances
-      (project "DQBSC"
-        (path "/8aaed6d1-6388-4dfb-8015-aa095e997bfa/bd4d4a4a-feba-4969-9481-b8d6f4eb80d3"
-          (reference "U13") (unit 1)
-        )
-      )

Commit message: UPDATE TO POWER TREE.
Parts:
- removed C57, C61: 4.7uF, Capacitor_SMD:C_0402_1005Metric_Pad0.74x0.62mm_HandSolder, symbol awg1000:CAP_UNPOL
- removed C58, C62: 0.47uF, Resistor_SMD:R_0402_1005Metric_Pad0.72x0.64mm_HandSolder, symbol awg1000:CAP_UNPOL
- removed C59, C60, C63, C64: 0.47u, Resistor_SMD:R_0402_1005Metric_Pad0.72x0.64mm_HandSolder, symbol awg1000:CAP_UNPOL
- removed C66, C67: 33uF, Capacitor_SMD:CP_Elec_6.3x7.7, symbol awg1000:CAP_POL
- removed C71, C73, C74, C76, C77, C79: 10uF, Capacitor_SMD:C_1206_3216Metric, symbol awg1000:CAP_UNPOL
- removed C75, C78: 220nF, awg1000:C0201_L, symbol awg1000:CAP_UNPOL
- removed D1 (x2): RSX501LAM20TR, Diode_SMD:D_SOD-128, symbol Device:D_Schottky
- removed L10, L11: 47uH, Inductor_SMD:L_Bourns_SRR1260, symbol Device:L
- removed R26: 7.15k, Resistor_SMD:R_0402_1005Metric, symbol awg1000:R
- removed U10, U9: TPS54531DDA, Package_SO:SOIC-8-1EP_3.9x4.9mm_P1.27mm_EP2.29x3mm_ThermalVias, symbol awg1000:TPS54531DDA
- added C12: 1UF, Capacitor_SMD:C_0603_1608Metric, symbol awg1000:CAP_UNPOL
- added C13: 1nF, Capacitor_SMD:C_0603_1608Metric, symbol awg1000:CAP_UNPOL
- added C18, C19, C24, C25, C26, C27, C29: 100nF, Capacitor_SMD:C_0201_0603Metric, symbol awg1000:CAP_UNPOL
- added C20, C21, C22, C23, C28, C30: 22uF, Capacitor_SMD:C_0603_1608Metric, symbol awg1000:CAP_UNPOL
- added D1: RSX501LAM20TR, Diode_SMD:D_0603_1608Metric, symbol Device:D_Schottky
- added D3: D_TVS, symbol Device:D_TVS
- added D5, D7: ~, Diode_SMD:D_0603_1608Metric, symbol Device:D_Schottky
- added L2, L3: 0.47uH, Inductor_SMD:L_1008_2520Metric, symbol Device:L
- added Q1: 2SK3018-TP, Package_TO_SOT_SMD:SOT-323_SC-70, symbol Device:Q_NMOS_DGS
- added R17: 100, Resistor_SMD:R_0402_1005Metric_Pad0.72x0.64mm_HandSolder, symbol awg1000:R
- added R19, R45: 10K, Resistor_SMD:R_0402_1005Metric_Pad0.72x0.64mm_HandSolder, symbol awg1000:R
- added R43, R46: 7.15k, Resistor_SMD:R_0402_1005Metric, symbol awg1000:R
- added R44: 1M, Resistor_SMD:R_0402_1005Metric_Pad0.72x0.64mm_HandSolder, symbol awg1000:R
- added R50: 6.98K, Resistor_SMD:R_0402_1005Metric_Pad0.72x0.64mm_HandSolder, symbol awg1000:R
- added R51: 56K, Resistor_SMD:R_0402_1005Metric_Pad0.72x0.64mm_HandSolder, symbol awg1000:R
- added R52: 100K, Resistor_SMD:R_0402_1005Metric_Pad0.72x0.64mm_HandSolder, symbol awg1000:R
- added R53: 0, Resistor_SMD:R_0402_1005Metric_Pad0.72x0.64mm_HandSolder, symbol awg1000:R
- added SH1, SH2: ~, Resistor_SMD:R_0805_2012Metric, symbol DQSBC:SHORT_STRING
- added TP1: ~, symbol DQSBC:TP
- added U10, U9: MP2147GD-Z, DQSBC:MP2147GD-Z, symbol DQSBC:MP2147GD-Z
- added U13: APX811-26UG-7, Package_TO_SOT_SMD:SOT-143, symbol DQSBC:APX811-26UG-7
- added U15: LDCL015, Package_TO_SOT_SMD:SOT-23-5, symbol DQSBC:LDCL015MR
- C11, C72: value 10uF -> 22uF; footprint Capacitor_SMD:C_1206_3216Metric -> Capacitor_SMD:C_0603_1608Metric; VOLTAGE 16V -> 10V
- C312: value 22uF -> 1uF
- C321: value 22uF -> 0.022UF
- C322: value 22uF -> 0.1uF; Voltage V -> 50V
- R20: value 0 -> 180K
- R21: value 7.15k -> 180K
- R22: value 7.15k -> 360K
- R33: value 0 -> 360K
- R34, R35, R36, R37: value 7.15k -> 10K
- R82: value 7.15k -> 44.2K
Connections:
- net 3.3V_SW: now also C26.1, R19.1, U13.4 (VCC)
- net 3.3V_SW_DELAYED: now also C19.2, C21.2, C25.2, C29.1, C30.1, R52.2, U10.11 (VIN2), U10.8 (VIN1), U15.1 (IN), U9.11 (VIN2), U9.8 (VIN1); no longer C11.2
- net GND: now also C11.2, R33.2, C13.1, C18.2, C19.1, C20.2, C21.1, C22.2, C23.2, C24.2, C25.1, C26.2, C27.2, C28.2, C29.2, C30.2, D3.2 (A2), Q1.3 (S), R44.2, R51.1, U10.10 (GND), U13.1 (GND), U15.2 (GND), U9.10 (GND); no longer C11.1, R35.2
- net PMIC_ON: now also R34.1, D1.2 (A)
- net PMIC_ON_REQ: now also R35.1
- net PMIC_STBY_REQ: now also Q1.2 (G)
- net VDD_ARM_0V9: now also SH1.2; no longer R21.1
- net VDD_SNVS_0V9: now also C27.1, C28.1, R50.1, U15.5 (OUT)
- net VDD_SOC_0V9: now also SH2.2; no longer R34.1
- net VIN: now also D3.1 (A1), R43.1, R46.1
- net at R21.2, R22.1: now also U9.3 (FB)
- net at R33.1: now also R20.2, U10.3 (FB)
- net at R29.1: now also U2.30 (AGND); no longer U2.31 (TON)
- net at R29.2: now also U2.31 (TON); no longer U2.30 (AGND)
- net at R34.2: now also U9.5 (EN); no longer R35.1
- net PG_VIN: now reaches U2.26 (PGOOD)
- net PG_VIN: now also R53.2
- net at R20.1: now also C22.1, C23.1, C24.1, L2.2, SH2.1, U10.2 (OUT)
- net LDO_EN: no longer names the net of U2.32 (ENL)
- net LDO_EN: now also R46.2; no longer U2.29 (EN/PSV)
- new net: R52.1, R53.1, U15.3 (EN)
- new net: C12.2, D7.1 (K), R44.1
- new net: C13.2, D5.1 (K), R17.1
- new net: R50.2, R51.2, U15.4 (ADJ)
- new net: TP1.1, U9.7 (PG)
- new net: L2.1, U10.1 (SW), U10.9 (SW)
- new net: C11.1, C18.1, C20.1, L3.2, R21.1, SH1.1, U9.2 (OUT)
- new net: L3.1, U9.1 (SW), U9.9 (SW)
- new net: R43.2, U2.29 (EN/PSV)
- new net: D1.1 (K), U10.7 (PG)
- new net MNRST: D5.2 (A), D7.2 (A), R45.1, U13.3 (NMR)
- new net NWDOG: C12.1
- new net P_MODE: Q1.1 (D), R19.2, U10.6 (MODE), U9.6 (MODE)
- new net SOC_EN: R35.2, R45.2, U10.5 (EN), U13.2 (NRST)
- new net SYS_NRST: R17.2
- no-connect marks 10 -> 14
Other:
- note added: "(0.9 V, 4.0 A)"
- note added: "*0.028A/3.3V"
- note added: "*0.068A/3.3V"
- note added: "*0.096A/3.3V"
- note added: "*0.5MA/3.3V"
- note added: "*0.6A/3.3V"
- note added: "*0.7A/3.3V"
- note added: "*0.85A/3.3V"
- note added: "*0.91A/3.3V"
- note added: "*0.9V/0.25A"
- note added: "*0.9V/2.5A"
- note added: "*0.9V/2A"
- note added: "*0.9V/4A"
- note added: "*1.1V/2.5A"
- note added: "*1.8V,0.35A"
- note added: "*1.8V/0.1A"
- note added: "*1.8V/1A"
- note added: "*1V/1.5MA"
- note added: "*1V/3A"
- note added: "*3.3V/0.1A"
- note added: "*3.3V/10A"
- note added: "*4A"
- note added: "0.9V/4A CORTEX A53 SMPS"
- note added: "0.9V/4A SOC SMPS"
- note added: "1.8V GPIO PIO"
- note added: "3.3 V GPIO PAO"
- note added: "3.3V SWITCH"
- note added: "CORTEX A53 PLATFORM"
- note added: "DRAM CONT., DRAM PYH"
- note added: "DRAM PHY"
- note added: "ENABLE"
- note added: "GEN1"
- note added: "GEN2"
- note added: "GEN3"
- note added: "GEN4"
- note added: "GEN5"
- note added: "GEN6"
- note added: "GPU"
- note added: "LPDDR4"
- note added: "PCIE, HDMI, MIPI"
- note added: "PCIE, HDMI, MIPI, USB1, 2"
- note added: "PF4210"
- note added: "PLL, XTAL, TEMP. SENS."
- note added: "PROCESSOR"
- note added: "SMPS"
- note added: "SNVS 0.9V LDO"
- note added: "SNVS_LP"
- note added: "SOC, 3.3V, 1.8 GPIO PAO"
- note added: "SW1AB"
- note added: "SW1C"
- note added: "SW2"
- note added: "SW3AB"
- note added: "SW4A"
- note added: "USB1, 2"
- note added: "VIN = 4.75 ~ 20V"
- note added: "VPU"
- note added: "VSNVS"
- note added: "i.MX 8M"
- note removed: "0.9V 3A PERIPHERALS SMPS"
- note removed: "3.3V 5A PERIPHERALS SMPS"
- moved on the sheet: C14, C15, C16, C17, C312, C313, C314, C321, C322, C72, L1, Q2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

Commit message: UPDATE, FULL ROUTING!
Parts:
- C12, D7, R44: now not fitted
Changed lines of the file:
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@@
     )
   )
+  (global_label "PG_VIN" (shape input) (at 81.28 30.48 0) (fields_autoplaced)
+    (effects (font (size 1 1)) (justify left))
+    (property "Intersheetrefs" "${INTERSHEET_REFS}" (at 88.7731 30.48 0)
+      (effects (font (size 1.27 1.27)) (justify left) hide)
+    )
+  )
   (global_label "NWDOG" (shape input) (at 364.49 91.44 180) (fields_autoplaced)
     (effects (font (size 1 1)) (justify right))
@@
   )
   (symbol (lib_name "awg1000:R_14") (lib_id "awg1000:R") (at 373.38 96.52 270) (mirror x) (unit 1)
-    (exclude_from_sim no) (in_bom yes) (on_board yes) (dnp no)
+    (exclude_from_sim no) (in_bom yes) (on_board yes) (dnp yes)
     (property "Reference" "R44" (at 372.11 93.98 90)
       (effects (font (size 1.27 1.27)) (justify right))
@@
   )
   (symbol (lib_id "Device:D_Schottky") (at 388.62 91.44 0) (unit 1)
-    (exclude_from_sim no) (in_bom yes) (on_board yes) (dnp no)
+    (exclude_from_sim no) (in_bom yes) (on_board yes) (dnp yes)
     (property "Reference" "D7" (at 384.81 90.17 0)
       (effects (font (size 1.27 1.27)))
@@
   )
   (symbol (lib_name "awg1000:CAP_UNPOL_69") (lib_id "awg1000:CAP_UNPOL") (at 373.38 91.44 90) (unit 1)
-    (exclude_from_sim no) (in_bom yes) (on_board yes) (dnp no)
+    (exclude_from_sim no) (in_bom yes) (on_board yes) (dnp yes)
     (property "Reference" "C12" (at 371.856 89.154 0)
       (effects (font (size 1.27 1.27)) (justify left))

Commit message: Update.
Connections:
- no-connect marks 14 -> 12
Other:
- moved on the sheet: C12, C13, C14, C15, C16, C17, C313, C314, D5, D7, R17, R34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
