File: 02_ECAD/MEM.kicad_sch (KiCad schematic)
At the start: 50 parts, among them U12 MT53E1G32D2FW-046_WT:A, U13 SDINBDG4-16G-I2, U14 IS25LP256D-JLLE

Commit message: Update.
Parts:
- renumbered C226 to C244, C227 to C245, C228 to C246, C229 to C247, C230 to C248, C231 to C249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
Other:
- note added: "Z DQ, DMI -> 42 Ohms, Z DQS/CLK -> 85 Ohms."

Commit message: Update.
Parts:
- renumbered C244 to C252, C245 to C253, C246 to C254, C247 to C255, C248 to C256, C249 to C257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
Other:
- note added: "LPRRD4 4GB RAM"
- note removed: "LPRRD4 RAM"
