File: 02_ECAD/MEM.kicad_sch (KiCad schematic)
At the start: 50 parts, among them U12 MT53E1G32D2FW-046_WT:A, U13 SDINBDG4-16G-I2, U14 IS25LP256D-JLLE

Commit message: Skew Check.
Other:
- note added: "EMMC 5.1"
- note removed: "EMMC"
Changed lines of the file:
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@@
 	(rectangle
 		(start 195.58 137.16)
-		(end 201.93 139.7)
+		(end 205.74 139.7)
 		(stroke
 			(width -0.0001)
@@
 		)
 	)
-	(text "EMMC"
+	(text "EMMC 5.1"
 		(exclude_from_sim no)
-		(at 201.422 139.192 0)
+		(at 205.74 139.7 0)
 		(effects
 			(font

Commit message: Update.
Parts:
- C252, C257, C258, C259, C260, C261, C262, C263, C264, C265, C266, C268, C269, C270, C271, C272, C273: MPN (none) -> CM05X5R475M16AH; Voltage V -> 16V
- C253, C254: MPN (none) -> GRM033Z71C104KE14D; Voltage V -> 16V
- C255, C256, C267: MPN (none) -> CL10A226MO7JZNC; Voltage V -> 16V
- C274: footprint Resistor_SMD:R_0402_1005Metric_Pad0.72x0.64mm_HandSolder -> Capacitor_SMD:C_0402_1005Metric; MPN (none) -> GRM158R61A226ME15D; Voltage (none) -> 10V
- C275: MPN (none) -> GRM033R61C224KE14D; Voltage (none) -> 16V
- C276, C277, C278, C279, C280, C281, C282, C283, C284, C285, C286: MPN (none) -> CC0402JRX7R7BB472; Voltage V -> 16V
- R63, R64: MPN (none) -> RC1005F151CS
- R65, R66: value 10K -> 10k; MPN (none) -> NRC04F1002TRF
- R67, R68: MPN (none) -> CR0402FC240RS1
- R69, R70: MPN (none) -> WR04X1501FTL
- R71: MPN (none) -> CR0402PC0RS001
- R72, R73, R74: MPN (none) -> RN73R1ETTP4701F50
- U12: MPN (none) -> MT53E1G32D2FW-046_WT:A
- U13: MPN (none) -> SDINBDG4-16G-I2
- U14: MPN (none) -> IS25LP256D-JLLE

Commit message: Update.
Parts:
- C275: renamed from C274; symbol awg1000:CAP_UNPOL -> SBC:C; Voltage 10V -> (none)
- C276: renamed from C275; symbol awg1000:CAP_UNPOL -> SBC:C; Voltage 16V -> (none)
- U14: footprint DQSBC:WSON-8-1EP_8x6mm_P1.27mm_E4.7X4.6mm -> SBC:WSON-8-1EP_8x6mm_P1.27mm_E4.7X4.6mm
- renumbered C252 to C253, C253 to C254, C254 to C255, C255 to C256, C256 to C257, C257 to C258, C258 to C259, C259 to C260, C260 to C261, C261 to C262, C262 to C263, C263 to C264, C264 to C265, C265 to C266, C266 to C267, C267 to C268, C268 to C269, C269 to C270, C270 to C271, C271 to C272, C272 to C273, C273 to C274, C276 to C277, C277 to C278, C278 to C279, C279 to C280, C280 to C281, C281 to C282, C282 to C283, C283 to C284, C284 to C285, C285 to C286, C286 to C287, R63 to R64, R64 to R65, R65 to R66, R66 to R67, R67 to R68, R68 to R69, R69 to R70, R70 to R71, R71 to R72, R72 to R73, R73 to R74, R74 to R75
Other:
- moved on the sheet: C278, C280, C282, C284, C286, R66
