File: 02_ECAD/MPU.kicad_sch (KiCad schematic)
At the start: 165 parts, among them U10 SIT1630AI-S4-DCC-32.768G, U11 TLV803EB26RDBZR, U9 MIMX8MD6DVAJZAB, Y1 ABM3B-25.000MHZ-D4Y-T, Y2 ABM3B-25.000MHZ-D4Y-T

Commit message: Update.
Parts:
- added C100, C101, C102, C103, C88, C89, C90, C91, C92, C93, C94, C95, C96, C97, C98, C99: 0.1uF, Capacitor_SMD:C_0201_0603Metric, symbol DQSBC:C
- added C184, C217: 100nF, Capacitor_SMD:C_0201_0603Metric, symbol DQSBC:C
- added Q4: NMOS, symbol Simulation_SPICE:NMOS
- added R41, R42, R43, R44, R45, R46, R47, R48, R49, R50, R51, R52: 1M, Resistor_SMD:R_0402_1005Metric, symbol DQSBC:R_US
- C123: renamed from C107; value 1uF -> 0.1uF
- C126: renamed from C110; value 1uF -> 0.1uF
- C127: renamed from C111; value 1uF -> 0.1uF
- C128: renamed from C112; value 1uF -> 100nF
- C129: renamed from C113; value 1uF -> 100nF
- C130: renamed from C114; value 1uF -> 100nF
- C131: renamed from C115; value 1uF -> 100nF
- C132: renamed from C116; value 22uF -> 100nF
- C134: renamed from C118; value 1uF -> 100nF
- C135: renamed from C119; value 1uF -> 100nF
- C136: renamed from C120; value 1uF -> 100nF
- C137: renamed from C121; value 1uF -> 100nF
- C138: renamed from C122; value 1uF -> 100nF
- C139: renamed from C123; value 1uF -> 100nF
- C141: renamed from C125; value 1uF -> 100nF
- C143: renamed from C127; value 1uF -> 0.1uF
- C144: renamed from C128; value 1uF -> 0.1uF
- C152: renamed from C136; value 1uF -> 100nF
- C155: renamed from C139; value 1uF -> 0.1uF
- C159: renamed from C143; value 1uF -> 10nF
- C167: renamed from C151; value 1uF -> 10nF
- C173: renamed from C156; value 1uF -> 100nF
- C177: renamed from C161; value 1uF -> 4.7nF
- C178: renamed from C162; value 1uF -> 100nF
- C189: renamed from C172; value 1uF -> 4.7nF
- C198: renamed from C181; value 1uF -> 4.7nF
- C207: renamed from C190; value 1uF -> 4.7nF
- C208: renamed from C191; value 1uF -> 4.7nF
- C214: renamed from C197; value 1uF -> 100nF
- C219: renamed from C201; value 1uF -> 4.7nF
- C220: renamed from C202; value 1uF -> 4.7nF
- C229: renamed from C211; value 1uF -> 4.7nF
- C230: renamed from C212; value 1uF -> 4.7nF
- C238: renamed from C220; value 1uF -> 4.7nF
- C239: renamed from C221; value 1uF -> 4.7nF
- FB1: value FerriteBead_Small -> 120 Ohms @ 100MHz
- FB2: value FerriteBead_Small -> 240 Ohms @ 100MHz
- R35, R37: value R_US -> 200
- R61: renamed from R49; value 0 -> 100K
- renumbered C88 to C104, C89 to C105, C90 to C106, C91 to C107, C92 to C108, C93 to C109, C94 to C110, C95 to C111, C96 to C112, C97 to C113, C98 to C114, C99 to C115, C100 to C116, C101 to C117, C102 to C118, C103 to C119, C104 to C120, C105 to C121, C106 to C122, C108 to C124, C109 to C125, C117 to C133, C124 to C140, C126 to C142, C129 to C145, C130 to C146, C131 to C147, C132 to C148, C133 to C149, C134 to C150, C135 to C151, C137 to C153, C138 to C154, C140 to C156, C141 to C157, C142 to C158, C144 to C160, C145 to C161, C146 to C162, C147 to C163, C148 to C164, C149 to C165, C150 to C166, C152 to C168, C153 to C169, C154 to C170, C155 to C171, C158 to C172, C157 to C174, C159 to C175, C160 to C176, C163 to C179, C164 to C180, C165 to C181, C166 to C182, C167 to C183, C168 to C185, C169 to C186, C170 to C187, C171 to C188, C173 to C190, C174 to C191, C175 to C192, C176 to C193, C177 to C194, C178 to C195, C179 to C196, C180 to C197, C182 to C199, C183 to C200, C184 to C201, C185 to C202, C186 to C203, C187 to C204, C188 to C205, C189 to C206, C192 to C209, C193 to C210, C194 to C211, C195 to C212, C196 to C213, C198 to C215, C199 to C216, C200 to C218, C203 to C221, C204 to C222, C205 to C223, C206 to C224, C207 to C225, C208 to C226, C209 to C227, C210 to C228, C213 to C231, C214 to C232, C215 to C233, C216 to C234, C217 to C235, C218 to C236, C219 to C237, C222 to C240, C223 to C241, C224 to C242, C225 to C243, R41 to R53, R42 to R54, R43 to R55, R44 to R56, R45 to R57, R46 to R58, R47 to R59, R48 to R60, R50 to R62
Connections:
- net GND: now also C184.2, C217.2, Q4.3 (S)
- net HDMI_AUX_N: now also C93.2, R49.1; no longer U9.V2 (HDMI_AUX_N)
- net HDMI_AUX_P: now also C92.2, R51.1; no longer U9.V1 (HDMI_AUX_P)
- net HDMI_REFCLK_N: now also C103.2, R42.1; no longer U9.R1 (HDMI_REFCLK_N)
- net HDMI_REFCLK_P: now also C102.2, R41.1; no longer U9.R2 (HDMI_REFCLK_P)
- net HDMI_TX0_N: now also C101.2, R44.1; no longer U9.T2 (HDMI_TX_M_LN_0)
- net HDMI_TX0_P: now also C100.2, R43.1; no longer U9.T1 (HDMI_TX_P_LN_0)
- net HDMI_TX1_N: now also C99.2, R52.1; no longer U9.U1 (HDMI_TX_M_LN_1)
- net HDMI_TX1_P: now also C98.2, R50.1; no longer U9.U2 (HDMI_TX_P_LN_1)
- net HDMI_TX2_N: now also C97.2, R45.1; no longer U9.N1 (HDMI_TX_M_LN_2)
- net HDMI_TX2_P: now also C96.2, R47.1; no longer U9.N2 (HDMI_TX_P_LN_2)
- net HDMI_TX3_N: now also C95.2, R48.1; no longer U9.M2 (HDMI_TX_M_LN_3)
- net HDMI_TX3_P: now also C94.2, R46.1; no longer U9.M1 (HDMI_TX_P_LN_3)
- net PCIE1_TXN: now also C88.2; no longer U9.J24 (PCIE1_TXN_N)
- net PCIE1_TXP: now also C89.2; no longer U9.J25 (PCIE1_TXN_P)
- net PCIE2_TXN: now also C91.2; no longer U9.E25 (PCIE2_TXN_P)
- net PCIE2_TXP: now also C90.2; no longer U9.E24 (PCIE2_TXN_N)
- net VDD_PHY_1V8: now also Q4.2 (G)
- net VDD_PHY_3V3: now also C184.1, C217.1
- new net: C88.1, U9.J24 (PCIE1_TXN_N)
- new net: C91.1, U9.E25 (PCIE2_TXN_P)
- new net: C89.1, U9.J25 (PCIE1_TXN_P)
- new net: C90.1, U9.E24 (PCIE2_TXN_N)
- new net H0_N: C103.1, U9.R1 (HDMI_REFCLK_N)
- new net H0_P: C102.1, U9.R2 (HDMI_REFCLK_P)
- new net H1_N: C101.1, U9.T2 (HDMI_TX_M_LN_0)
- new net H1_P: C100.1, U9.T1 (HDMI_TX_P_LN_0)
- new net H2_N: C99.1, U9.U1 (HDMI_TX_M_LN_1)
- new net H2_P: C98.1, U9.U2 (HDMI_TX_P_LN_1)
- new net H3_N: C93.1, U9.V2 (HDMI_AUX_N)
- new net H3_P: C92.1, U9.V1 (HDMI_AUX_P)
- new net H4_N: C97.1, U9.N1 (HDMI_TX_M_LN_2)
- new net H4_P: C96.1, U9.N2 (HDMI_TX_P_LN_2)
- new net H5_N: C95.1, U9.M2 (HDMI_TX_M_LN_3)
- new net H5_P: C94.1, U9.M1 (HDMI_TX_P_LN_3)
- new net R_GND: Q4.1 (D), R41.2, R42.2, R43.2, R44.2, R45.2, R46.2, R47.2, R48.2, R49.2, R50.2, R51.2, R52.2
Other:
- note added: "IX8 PCIE 2.0"
- note added: "Z DSI -> 100 Ohms."
- note added: "Z HDMI -> 100 Ohms."
- note added: "Z PCIe TX/RX -> 85 Ohms, Z PCIe Clk -> 100 Ohms."
- note added: "Z USB -> 90 Ohm.s"
- note removed: "IX8 PCIE"
- note removed: "add capacitive couplig to tx and clk?"
- moved on the sheet: C172, R39, U9J

Commit message: Update.
Parts:
- removed Q4: NMOS, symbol Simulation_SPICE:NMOS
- removed unit 9 of U9
- added C90, C91, C92, C93, C96, C97, C98, C99: 0.1uF, Capacitor_SMD:C_0201_0603Metric, symbol DQSBC:C
- added Q4: NX3020NAKS, Package_TO_SOT_SMD:SOT-23-3, symbol Device:Q_NMOS_GSD
- R41: renamed from R45; value 1M -> 604; footprint Resistor_SMD:R_0402_1005Metric -> Resistor_SMD:R_0201_0603Metric_Pad0.64x0.40mm_HandSolder
- R42: renamed from R47; value 1M -> 604; footprint Resistor_SMD:R_0402_1005Metric -> Resistor_SMD:R_0201_0603Metric_Pad0.64x0.40mm_HandSolder
- R43: renamed from R49; value 1M -> 604; footprint Resistor_SMD:R_0402_1005Metric -> Resistor_SMD:R_0201_0603Metric_Pad0.64x0.40mm_HandSolder
- R44: renamed from R51; value 1M -> 604; footprint Resistor_SMD:R_0402_1005Metric -> Resistor_SMD:R_0201_0603Metric_Pad0.64x0.40mm_HandSolder
- R45: renamed from R41; value 1M -> 604; footprint Resistor_SMD:R_0402_1005Metric -> Resistor_SMD:R_0201_0603Metric_Pad0.64x0.40mm_HandSolder
- R46: renamed from R42; value 1M -> 604; footprint Resistor_SMD:R_0402_1005Metric -> Resistor_SMD:R_0201_0603Metric_Pad0.64x0.40mm_HandSolder
- R47: renamed from R43; value 1M -> 604; footprint Resistor_SMD:R_0402_1005Metric -> Resistor_SMD:R_0201_0603Metric_Pad0.64x0.40mm_HandSolder
- R48: renamed from R44; value 1M -> 604; footprint Resistor_SMD:R_0402_1005Metric -> Resistor_SMD:R_0201_0603Metric_Pad0.64x0.40mm_HandSolder
- R49: renamed from R46; value 1M -> 604; footprint Resistor_SMD:R_0402_1005Metric -> Resistor_SMD:R_0201_0603Metric_Pad0.64x0.40mm_HandSolder
- R50: renamed from R48; value 1M -> 604; footprint Resistor_SMD:R_0402_1005Metric -> Resistor_SMD:R_0201_0603Metric_Pad0.64x0.40mm_HandSolder
- R51: renamed from R50; value 1M -> 604; footprint Resistor_SMD:R_0402_1005Metric -> Resistor_SMD:R_0201_0603Metric_Pad0.64x0.40mm_HandSolder
- R52: value 1M -> 604; footprint Resistor_SMD:R_0402_1005Metric -> Resistor_SMD:R_0201_0603Metric_Pad0.64x0.40mm_HandSolder
- renumbered C92 to C100, C94 to C101, C96 to C102, C98 to C103, C100 to C104, C102 to C105, C93 to C106, C95 to C107, C97 to C108, C99 to C109, C101 to C110, C103 to C111, C105 to C112, C111 to C113, C117 to C114, C109 to C115, C115 to C116, C120 to C117, C104 to C118, C110 to C119, C116 to C120, C108 to C121, C114 to C122, C119 to C123, C107 to C124, C113 to C125, C118 to C126, C106 to C127, C112 to C128, C121 to C129, C122 to C130, C123 to C131, C124 to C132, C125 to C133, C126 to C134, C127 to C135, C128 to C136, C129 to C137, C130 to C138, C131 to C139, C132 to C140, C133 to C141, C134 to C142, C135 to C143, C136 to C144, C137 to C145, C138 to C146, C139 to C147, C140 to C148, C156 to C149, C141 to C150, C142 to C151, C143 to C152, C144 to C153, C145 to C154, C146 to C155, C147 to C156, C148 to C157, C149 to C158, C150 to C159, C151 to C160, C152 to C161, C153 to C162, C154 to C163, C155 to C164, C157 to C165, C158 to C166, C159 to C167, C160 to C168, C161 to C169, C162 to C170, C163 to C171, C164 to C172, C165 to C173, C166 to C174, C167 to C175, C168 to C176, C169 to C177, C170 to C178, C171 to C179, C172 to C180, C173 to C181, C174 to C182, C175 to C183, C176 to C184, C177 to C185, C178 to C186, C179 to C187, C180 to C188, C181 to C189, C182 to C190, C183 to C191, C184 to C192, C185 to C193, C186 to C194, C187 to C195, C188 to C196, C189 to C197, C190 to C198, C191 to C199, C192 to C200, C193 to C201, C194 to C202, C195 to C203, C196 to C204, C197 to C205, C198 to C206, C199 to C207, C200 to C208, C201 to C209, C202 to C210, C203 to C211, C204 to C212, C205 to C213, C206 to C214, C207 to C215, C208 to C216, C209 to C217, C210 to C218, C211 to C219, C212 to C220, C213 to C221, C214 to C222, C215 to C223, C216 to C224, C217 to C225, C218 to C226, C219 to C227, C220 to C228, C221 to C229, C222 to C230, C223 to C231, C224 to C232, C225 to C233, C226 to C234, C227 to C235, C228 to C236, C229 to C237, C230 to C238, C231 to C239, C232 to C240, C233 to C241, C234 to C242, C235 to C243, C236 to C244, C237 to C245, C238 to C246, C239 to C247, C240 to C248, C241 to C249, C242 to C250, C243 to C251, C90 to C94, C91 to C95, R40 to R39, R39 to R40
Connections:
- net GND: now also Q4.2 (S)
- net HDMI_REFCLK_N: now also R46.2; no longer R46.1
- net HDMI_REFCLK_P: now also R45.2; no longer R45.1
- net HDMI_TX0_N: now also R48.2; no longer R48.1
- net HDMI_TX0_P: now also R47.2; no longer R47.1
- net HDMI_TX1_N: now also R52.2; no longer R52.1
- net HDMI_TX1_P: now also R51.2; no longer R51.1
- net HDMI_TX3_N: now also R50.2; no longer R50.1
- net HDMI_TX3_P: now also R49.2; no longer R49.1
- net R_GND: now also R45.1, R46.1, R47.1, R48.1, R49.1, R50.1, R51.1, R52.1, Q4.3 (D); no longer R45.2, R46.2, R47.2, R48.2, R49.2, R50.2, R51.2, R52.2
- net USB1_RX_N: now also C93.2; no longer U9.B12 (USB1_RX_N)
- net USB1_RX_P: now also C92.2; no longer U9.A12 (USB1_RX_P)
- net USB1_TX_N: now also C91.2; no longer U9.B13 (USB1_TX_N)
- net USB1_TX_P: now also C90.2; no longer U9.A13 (USB1_TX_P)
- net USB2_RX_N: now also C99.2; no longer U9.B8 (USB2_RX_N)
- net USB2_RX_P: now also C98.2; no longer U9.A8 (USB2_RX_P)
- net USB2_TX_N: now also C97.2; no longer U9.B9 (USB2_TX_N)
- net USB2_TX_P: now also C96.2; no longer U9.A9 (USB2_TX_P7)
- net VDD_PHY_1V8: now also Q4.1 (G)
- net pi_P: now reaches C88.1, U9.J24 (PCIE1_TXN_N)
- net pi2_N: now reaches C95.1, U9.E25 (PCIE2_TXN_P)
- net pi_N: now reaches C89.1, U9.J25 (PCIE1_TXN_P)
- net pi2_P: now reaches C94.1, U9.E24 (PCIE2_TXN_N)
- net GPIO0 renamed PCIE2_nCLKREQ
- net GPIO1 renamed PCIE1_nCLKREQ
- net PCIE1_REF_CLKN renamed IX8_PCIE1_CLK_N
- net PCIE1_REF_CLKP renamed IX8_PCIE1_CLK_P
- net PCIE2_REF_CLKN renamed IX8_PCIE2_CLK_P
- net PCIE2_REF_CLKP renamed IX8_PCIE2_CLK_N
- new net U1_RX_N: C93.1, U9.B12 (USB1_RX_N)
- new net U1_RX_P: C92.1, U9.A12 (USB1_RX_P)
- new net U1_TX_N: C91.1, U9.B13 (USB1_TX_N)
- new net U1_TX_P: C90.1, U9.A13 (USB1_TX_P)
- new net U2_RX_N: C99.1, U9.B8 (USB2_RX_N)
- new net U2_RX_P: C98.1, U9.A8 (USB2_RX_P)
- new net U2_TX_N: C97.1, U9.B9 (USB2_TX_N)
- new net U2_TX_P: C96.1, U9.A9 (USB2_TX_P7)
- no-connect marks 48 -> 28
Other:
- note added: "IMX8 HDMI 2.0A"
- note removed: "IMX8 CSI"
- note removed: "IMX8 HDMI"
- moved on the sheet: C100, C101, C102, C103, C104, C105, C106, C107, C108, C109, C110, C111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

Commit message: Update.
Parts:
- C100, C101, C102, C103, C104, C105, C106, C107, C108, C109, C110, C111, C131, C134, C135, C152, C153, C164, C88, C89, C90, C91, C92, C93, C94, C95, C96, C97, C98, C99: MPN (none) -> GRM033Z71C104KE14D; Voltage 6.3V -> 16V
- C112, C113, C114, C115, C116, C117, C118, C119, C120, C121, C122, C123, C124, C125, C126, C127, C128, C160, C163, C171, C172, C174, C176, C177, C179, C180, C182, C183, C184, C187, C188, C189, C191, C194, C195, C196, C198, C199, C200, C201, C203, C204, C205, C207, C208, C209, C210, C213, C214, C217, C218, C219, C220, C221, C223, C224, C226, C229, C230, C231, C232, C233, C234, C235, C236, C239, C240, C241, C242, C243, C244, C245, C248, C249, C250, C251, C87: MPN (none) -> JMK063ABJ105KP-F
- C129, C130, C133, C141, C151, C154, C155, C156, C157, C158, C165, C166, C168, C169, C170, C173, C178, C190, C193, C202, C212: MPN (none) -> GRM158R61A226ME15D; Voltage 6.3V -> 10V
- C132, C148, C159, C162: value C -> 27pF; MPN (none) -> KGM03ACG1E270KH; Voltage V -> 16V
- C136, C137, C138, C139, C142, C143, C144, C145, C146, C147, C150, C161, C181, C186, C192, C222, C225: value 100nF -> 0.1uF; MPN (none) -> GRM033Z71C104KE14D; Voltage 6.3V -> 16V
- C140: value 100nF -> 0.1uF; MPN (none) -> CC0402JRX7R7BB472; Voltage 6.3V -> 16V
- C149, C211: MPN (none) -> GRM033Z71C104KE14D; Voltage V -> 16V
- C167, C175: MPN (none) -> GRM033R71C103KE14D
- C185, C197, C206, C215, C216, C227, C228, C237, C238, C246, C247: MPN (none) -> GRM033R71C472KE14D
- FB1: MPN (none) -> BLM15PD121SN1D
- FB2: MPN (none) -> MMZ0603S241HT000
- HS1: MPN (none) -> HSB07-202009
- Q4: MPN (none) -> NX3020NAKS
- R33, R62: MPN (none) -> NRC04F1002TRF
- R34: MPN (none) -> CR0402FC240RS1
- R35, R36, R37, R38: MPN (none) -> RK73G1ETTP2000F
- R39: MPN (none) -> CR0402FC15KS01
- R40: MPN (none) -> ERJ-2RKF4990X
- R41, R42, R43, R44, R45, R46, R47, R48, R49, R50, R51, R52: footprint Resistor_SMD:R_0201_0603Metric_Pad0.64x0.40mm_HandSolder -> Resistor_SMD:R_0201_0603Metric; MPN (none) -> RC0201FR-07604RL
- R53, R54: MPN (none) -> CR0402FC1MS001
- R55, R56: MPN (none) -> RC0201FR-07100RL
- R57: MPN (none) -> RN73R1ETTP4701F50
- R58, R60, R61: MPN (none) -> CR0402FC100KS1
- R59: MPN (none) -> WR04X1501FTL
- U10: MPN (none) -> SIT1630AI-S4-DCC-32.768G
- U11: MPN (none) -> TLV803EB26RDBZR
- U9: MPN (none) -> MIMX8MD6DVAJZAB
- Y1: MPN (none) -> ABM3B-25.000MHZ-D4Y-T
- Y2: value ABM3B-25.000MHZ-D4Y-T -> ABM3B-27.000MHZ-D3Y-T; MPN (none) -> ABM3B-27.000MHZ-D3Y-T
