File: 02_ECAD/MPU.kicad_sch (KiCad schematic)
At the start: 204 parts, among them Q4 NX3020NAKS, U10 SIT1630AI-S4-DCC-32.768G, U11 TLV803EB26RDBZR, U9 MIMX8MD6DVAJZAB, Y1 ABM3B-25.000MHZ-D4Y-T, Y2 ABM3B-27.000MHZ-D3Y-T

Commit message: Regular Update.
Changed lines of the file:
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@@
 	(text_box "A 100 Ω typical ESR and 8 pF CL crystal rated for\na maximum drive level of 200 μW is acceptable.\nConsult crystal vendor and do matching test for\ndesigning external compensation capacitors is\npreferred. Use short traces between the crystal\nand the processor, with a ground plane under the\ncrystal, load capacitors, and associated traces."
 		(exclude_from_sim no)
-		(at 386.08 157.734 0)
+		(at 393.446 158.242 0)
 		(size 21.844 17.526)
 		(stroke

Commit message: Update.
Parts:
- HS1: value HSB07-202009 -> HSB07-202009
- renumbered C99 to C100, C100 to C101, C101 to C102, C102 to C103, C103 to C104, C104 to C105, C105 to C106, C106 to C107, C107 to C108, C108 to C109, C109 to C110, C110 to C111, C111 to C112, C112 to C113, C113 to C114, C114 to C115, C115 to C116, C116 to C117, C117 to C118, C118 to C119, C119 to C120, C120 to C121, C121 to C122, C122 to C123, C123 to C124, C124 to C125, C125 to C126, C126 to C127, C127 to C128, C128 to C129, C129 to C130, C130 to C131, C131 to C132, C132 to C133, C133 to C134, C134 to C135, C135 to C136, C136 to C137, C137 to C138, C138 to C139, C139 to C140, C140 to C141, C141 to C142, C142 to C143, C143 to C144, C144 to C145, C145 to C146, C146 to C147, C147 to C148, C148 to C149, C149 to C150, C150 to C151, C151 to C152, C152 to C153, C153 to C154, C154 to C155, C155 to C156, C156 to C157, C157 to C158, C158 to C159, C159 to C160, C160 to C161, C161 to C162, C162 to C163, C163 to C164, C164 to C165, C165 to C166, C166 to C167, C167 to C168, C168 to C169, C169 to C170, C170 to C171, C171 to C172, C172 to C173, C173 to C174, C174 to C175, C175 to C176, C176 to C177, C177 to C178, C178 to C179, C179 to C180, C180 to C181, C181 to C182, C182 to C183, C183 to C184, C184 to C185, C185 to C186, C186 to C187, C187 to C188, C188 to C189, C189 to C190, C190 to C191, C191 to C192, C192 to C193, C193 to C194, C194 to C195, C195 to C196, C196 to C197, C197 to C198, C198 to C199, C199 to C200, C200 to C201, C201 to C202, C202 to C203, C203 to C204, C204 to C205, C205 to C206, C206 to C207, C207 to C208, C208 to C209, C209 to C210, C210 to C211, C211 to C212, C212 to C213, C213 to C214, C214 to C215, C215 to C216, C216 to C217, C217 to C218, C218 to C219, C219 to C220, C220 to C221, C221 to C222, C222 to C223, C223 to C224, C224 to C225, C225 to C226, C226 to C227, C227 to C228, C228 to C229, C229 to C230, C230 to C231, C231 to C232, C232 to C233, C233 to C234, C234 to C235, C235 to C236, C236 to C237, C237 to C238, C238 to C239, C239 to C240, C240 to C241, C241 to C242, C242 to C243, C243 to C244, C244 to C245, C245 to C246, C246 to C247, C247 to C248, C248 to C249, C249 to C250, C250 to C251, C251 to C252, C87 to C88, C88 to C89, C89 to C90, C90 to C91, C91 to C92, C92 to C93, C93 to C94, C94 to C95, C95 to C96, C96 to C97, C97 to C98, C98 to C99, R33 to R34, R34 to R35, R35 to R36, R36 to R37, R37 to R38, R38 to R39, R39 to R40, R40 to R41, R41 to R42, R42 to R43, R43 to R44, R44 to R45, R45 to R46, R46 to R47, R47 to R48, R48 to R49, R49 to R50, R50 to R51, R51 to R52, R52 to R53, R53 to R54, R54 to R55, R55 to R56, R56 to R57, R57 to R58, R58 to R59, R59 to R60, R60 to R61, R61 to R62, R62 to R63
Other:
- note removed: "MIMX8MD6DVAJZAB"
- moved on the sheet: C100, C101, C102, C103, C104, C105, C106, C107, C108, C109, C110, C111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
