File: 02_ECAD/IO.kicad_sch (KiCad schematic)
At the start: 75 parts, among them J1 3-1827253-6, J2 Conn_02x05_Odd_Even, J3 Conn_Coaxial, SW1 NANOT160AS, SW2 NANOT160AS, SW3 SW_DIP_x02, U15 VSC8541XMV-02, U16 ESP32-PICO-D4, Y3 Crystal

Commit message: UPDATE.
Parts:
- added C290: 10uF, Capacitor_SMD:C_0402_1005Metric, symbol DQSBC:C
- added C291, C292, C293, C294: 0.1uF, Capacitor_SMD:C_0402_1005Metric, symbol DQSBC:C
- added J4: RFShield_OnePiece, SBC:Laird_Technologies_BMI-S-101_13.66x12.70mm, symbol Device:RFShield_OnePiece
- added U17: ESP-PSRAM32, Package_SO:SOIC-8_3.9x4.9mm_P1.27mm, symbol Memory_RAM:ESP-PSRAM32
- J2: value Conn_02x05_Odd_Even -> B10B-PHDSS; Quantity (none) -> B10B-PHDSS
Connections:
- net 3.3V_SW_DELAYED: now also C290.1, C291.1, C292.1, C293.1, C294.1, U17.8 (VCC)
- net GND: now also C290.2, C291.2, C292.2, C293.2, C294.2, J4.1 (Shield), U17.4 (VSS)
- net SIO1: now reaches U16.27 (IO17)
- net SIO1: now also U17.2 (SO/SIO)
- net SIO3: now reaches U16.30 (CMD)
- net SIO3: now also U17.7 (SIO3)
- net SCLK: now reaches U16.31 (CLK)
- net SCLK: now also U17.6 (SCLK)
- net SIO2: now reaches U16.32 (SD0)
- net SIO2: now also U17.3 (SIO2)
- net SIO0: now reaches U16.33 (SD1)
- net SIO0: now also U17.5 (SI/SIO)
- net ESP32_RX: now reaches U16.40 (U0RXD/IO3)
- net ESP32_TX: now reaches U16.41 (U0TXD/IO1)
- new net RAM_CS: U17.1 (~{CE})
Other:
- note added: "WIFI+BLUETOOTH ( OPTIONAL )"
- moved on the sheet: C288, C289, J3, L8, U16

Commit message: Update.
Parts:
- removed R72, R73: 10k, Resistor_SMD:R_0402_1005Metric, symbol awg1000:R
- renumbered C265 to C283, C266 to C284, C294 to C285, C290 to C286, C288 to C287, C291 to C288, C292 to C290, C293 to C291, C267 to C292, C268 to C293, C269 to C294, C270 to C295, C271 to C296, C272 to C297, C273 to C298, C274 to C299, C275 to C300, C276 to C301, C277 to C302, C278 to C303, C279 to C304, C280 to C305, C281 to C306, C282 to C307, C283 to C308, C284 to C309, C285 to C310, C286 to C311, C287 to C312, J4 to J2, J2 to J3, J3 to J4, R63 to R75, R64 to R76, R65 to R77, R66 to R78, R67 to R79, R68 to R80, R69 to R81, R70 to R82, R71 to R83, R74 to R84, R75 to R85, R76 to R86, R77 to R87, R78 to R88, R79 to R89, R80 to R90, R81 to R91, R82 to R92, R83 to R93, R84 to R94, R85 to R95, U17 to U16, U16 to U17

Commit message: Update.
Parts:
- added C291, C292, C300, C301: C, Capacitor_SMD:C_0201_0603Metric, symbol DQSBC:C
- added C293, C294, C295, C296, C297, C298, C299, C302, C303, C304, C305, C306, C307, C308: 1uF, Capacitor_SMD:C_0201_0603Metric, symbol DQSBC:C
- added D11, D12, D7, D8: RSX501LAM20TR, Diode_SMD:D_0603_1608Metric, symbol Device:D_Schottky
- added FB3, FB4, FB5, FB6: 120 Ohms @ 100MHz, Inductor_SMD:L_0402_1005Metric, symbol Device:FerriteBead_Small
- added Q8, Q9: NX3020NAKS, Package_TO_SOT_SMD:SOT-23-3, symbol Device:Q_NMOS_GSD
- added R82, R89: 0, Resistor_SMD:R_0402_1005Metric, symbol awg1000:R
- added R84, R85, R86, R94: 10k, Resistor_SMD:R_0402_1005Metric, symbol awg1000:R
- added U15, U16: 9FGV0241AKLF, Package_DFN_QFN:VQFN-24-1EP_4x4mm_P0.5mm_EP2.5x2.5mm, symbol SBC:9FGV0241AKLF
- added Y3, Y4: ABM3B-25.000MHZ-D4Y-T, SBC:Crystal_SMD_Abracon_ABM3B-4Pin_5.0x3.2mm, symbol Device:Crystal_GND24
- gave numbers to parts that had none: 7
- renumbered C283 to C309, C285 to C310, C286 to C311, C287 to C312, C288 to C313, C289 to C314, C290 to C315, C291 to C316, C284 to C317, C301 to C318, C292 to C319, C298 to C320, C299 to C321, C300 to C322, C305 to C323, C302 to C324, C303 to C325, C304 to C326, C297 to C327, C309 to C328, C294 to C329, C306 to C330, C307 to C331, C308 to C332, C293 to C333, C310 to C334, C311 to C335, C312 to C336, C295 to C337, C296 to C338, D8 to D10, D7 to D9, FB3 to FB7, FB4 to FB8, L8 to L10, R94 to R100, R95 to R101, R82 to R87, R84 to R88, R85 to R90, R86 to R91, R87 to R92, R88 to R93, R89 to R95, R90 to R96, R91 to R97, R92 to R98, R93 to R99, U15 to U17, U16 to U18, U17 to U19, Y3 to Y5
Connections:
- net 3.3V_SW_DELAYED: now also R85.1, R86.1
- net GND: now also J1.B54 (GPO1), J1.B55 (RSVD), C291.2, C292.2, C293.2, C294.2, C295.2, C296.2, C297.2, C298.2, C299.2, C300.2, C301.2, C302.2, C303.2, C304.2, C305.2, C306.2, C307.2, C308.2, Q8.2 (S), Q9.2 (S), U15. (SS_EN_TRI), U15.10 (GND_1), U15.15 (GND_A), U15.21 (GND_2), U15.24 (GND_XTAL), U15.25 (EPAD), U15.6 (GND_DIG), U16. (SS_EN_TRI), U16.10 (GND_1), U16.15 (GND_A), U16.21 (GND_2), U16.24 (GND_XTAL), U16.25 (EPAD), U16.6 (GND_DIG), Y3.2, Y3.4, Y4.2, Y4.4
- net I2C1_SCL: now also J1.B63 (GPO3); no longer J1.B57 (GPO2)
- net I2C1_SDA: now also J1.B64 (PCIE_RX1+); no longer J1.B58 (PCIE_RX3+)
- net I2C2_SCL: now also J1.B67 (WAKE1#_(**)), R85.2, U15.8 (SCLK_3.3), U16.8 (SCLK_3.3); no longer J1.B61 (PCIE_RX2+)
- net I2C2_SDA: now also J1.B66 (WAKE0#), R86.2, U15.9 (SDATA_3.3), U16.9 (SDATA_3.3); no longer J1.B60 (GND(FIXED))
- net I2C3_SCL: now also J1.B69 (PCIE_RX0-); no longer J1.B63 (GPO3)
- net I2C3_SDA: now also J1.B70 (GND(FIXED)); no longer J1.B64 (PCIE_RX1+)
- net UART4_RXD: now also J1.B60 (GND(FIXED)); no longer J1.B54 (GPO1)
- net UART4_TXD: now also J1.B61 (PCIE_RX2+); no longer J1.B55 (RSVD)
- net PCIE1_REF_CLKN renamed HOST_PCIE1_CLK_N
- net HOST_PCIE1_CLK_N: now also U15.14 (NDIF0)
- net PCIE1_REF_CLKP renamed HOST_PCIE1_CLK_P
- net HOST_PCIE1_CLK_P: now also U15.13 (DIF0)
- net PCIE2_REF_CLKN renamed HOST_PCIE2_CLK_N
- net HOST_PCIE2_CLK_N: now also U16.14 (NDIF0)
- net PCIE2_REF_CLKP renamed HOST_PCIE2_CLK_P
- net HOST_PCIE2_CLK_P: now also U16.13 (DIF0)
- new net: C293.1, C294.1, FB3.2, U15.11 (VDD1.8_1), U15.20 (VDD1.8_2)
- new net: C305.1, C307.1, C308.1, FB6.2, U16.16 (VDDA1.8), U16.3 (VDDXTAL1.8)
- new net: D11.2 (A), D12.2 (A), Q9.1 (G), R94.2
- new net: C296.1, C298.1, C299.1, FB4.2, U15.16 (VDDA1.8), U15.3 (VDDXTAL1.8)
- new net: D7.2 (A), D8.2 (A), Q8.1 (G), R84.2
- new net: C302.1, C303.1, FB5.2, U16.11 (VDD1.8_1), U16.20 (VDD1.8_2)
- new net 25MHZ_P1I: C291.1, U15.1 (X1_25), Y3.3
- new net 25MHZ_P1O: C292.1, U15.2 (X2), Y3.1
- new net 25MHZ_P2I: C300.1, U16.1 (X1_25), Y4.3
- new net 25MHZ_P2O: C301.1, U16.2 (X2), Y4.1
- new net IX8_PCIE1_CLK_N: U15.18 (NDIF1)
- new net IX8_PCIE1_CLK_P: U15.17 (DIF1)
- new net IX8_PCIE2_CLK_N: U16.18 (NDIF1)
- new net IX8_PCIE2_CLK_P: U16.17 (DIF1)
- new net PCIE1_NCLKREQ: D7.1 (K), R82.1
- new net PCIE1_REQ: Q8.3 (D), U15.22 (NCKPWRGD_PD)
- new net PCIE1_nCLKREQ: D8.1 (K), R82.2
- new net PCIE2_NCLKREQ: D11.1 (K), R89.1
- new net PCIE2_REQ: Q9.3 (D), U16.22 (NCKPWRGD_PD)
- new net PCIE2_nCLKREQ: D12.1 (K), R89.2
- new net VDD_1V8: C295.1, C297.1, C304.1, C306.1, FB3.1, FB4.1, FB5.1, FB6.1, R84.1, R94.1, U15.7 (VDDDIG1.8), U16.7 (VDDDIG1.8)
- no-connect marks 43 -> 41
Other:
- note added: "PCIE 2.0 X 2"
- note added: "PCIE CLK GEN."
- moved on the sheet: C309, C317, C318, C319, C320, C321, C322, C323, C324, C325, C326, C327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

Commit message: Skew Check.
Parts:
- added R100, R101, R102, R103, R104, R105, R98, R99: 39, Resistor_SMD:R_0201_0603Metric_Pad0.64x0.40mm_HandSolder, symbol awg1000:R
- renumbered R98 to R106, R99 to R107, R100 to R108, R101 to R109
Connections:
- net ENET_RD0: now also R102.1; no longer U17.29 (RXD0)
- net ENET_RD1: now also R103.1; no longer U17.27 (RXD1)
- net ENET_RD2: now also R104.1; no longer U17.26 (RXD2)
- net ENET_RD3: now also R105.1; no longer U17.25 (RXD3)
- net ENET_RXC: now also R100.1; no longer U17.32 (RX_CLK)
- net ENET_RX_CTL: now also R101.1; no longer U17.30 (RX_DV/RX_CTL)
- net ESP32_RX: now also R99.1
- net ESP32_TX: now also R98.1
- net GND: now also U15.12 (NOE0), U15.19 (NOE1), U15.23 (SS_EN_TRI), U16.12 (NOE0), U16.19 (NOE1), U16.23 (SS_EN_TRI); no longer U15. (SS_EN_TRI), U16. (SS_EN_TRI)
- net RAM_CS: now also U19.30 (CMD)
- net SIO3: now also U19.25 (IO16); no longer U19.30 (CMD)
- net UART1_RXD: now also R98.2
- net UART1_TXD: now also R99.2
- net GPIO1: no longer names the net of J1.B79 (eDP/LVDS_BKLT_EN)
- new net: R102.2, U17.29 (RXD0)
- new net: R105.2, U17.25 (RXD3)
- new net: R101.2, U17.30 (RX_DV/RX_CTL)
- new net: R103.2, U17.27 (RXD1)
- new net: R104.2, U17.26 (RXD2)
- new net: R100.2, U17.32 (RX_CLK)
Other:
- note added: "Length Match"
- note added: "needs reveiw"

Commit message: Update.
Parts:
- C287, C288, C289, C290: MPN (none) -> GCJ188R72A223KA01D
- C291, C292, C300, C301: value C -> 27pF; MPN (none) -> KGM03ACG1E270KH; Voltage V -> 16V
- C293, C294, C295, C296, C297, C298, C299, C302, C303, C304, C305, C306, C307, C308: MPN (none) -> JMK063ABJ105KP-F
- C309: MPN (none) -> KGM05AR71C103KH
- C310, C318, C323, C324, C325, C326, C329, C330, C331, C332, C334, C335, C336, C337: MPN (none) -> CC0402JRX7R7BB472; Voltage V -> 16V
- C311: MPN (none) -> GRM155R61A106ME11D; Voltage V -> 10V; now not fitted
- C312, C314: MPN (none) -> GRM033Z71C104KE14D; Voltage V -> 16V; now not fitted
- C313, C315, C316: MPN (none) -> CC0402JRX7R7BB472; Voltage V -> 16V; now not fitted
- C317: value C -> 0.1uF; MPN (none) -> CC0402JRX7R7BB472; Voltage V -> 16V
- C319, C327: value C -> 26pF; MPN (none) -> KGM03ACG1E270KH; Voltage V -> 16V
- C320, C321, C322, C328, C333, C338: MPN (none) -> GRM155R61A106ME11D; Voltage V -> 10V
- D10, D9: value D_Schottky -> SD0603S040S0R2; MPN (none) -> SD0603S040S0R2
- D11, D12, D7, D8: MPN (none) -> SD0603S040S0R2
- D5, D6: value LED -> BQ-0603G027-H3YYD0N-E0; MPN (none) -> BQ-0603G027-H3YYD0N-E0
- FB3, FB4, FB5, FB6: MPN (none) -> BLM15PD121SN1D
- FB7, FB8: value FerriteBead_Small -> 240 Ohms @ 100MHz; MPN (none) -> BMC1JY0240AN
- H1, H2, H3, H4: now not fitted; now left out of the parts list
- J1: MPN (none) -> 3-1827253-6
- J2: MPN (none) -> BMI-S-101_13; now not fitted
- J3: MPN (none) -> B10B-PHDSS
- J4, L10: now not fitted
- Q5, Q6, Q7: MPN (none) -> 2SK3018-TP
- Q8, Q9: MPN (none) -> NX3020NAKS
- R100, R101, R102, R103, R104, R105: footprint Resistor_SMD:R_0201_0603Metric_Pad0.64x0.40mm_HandSolder -> Resistor_SMD:R_0201_0603Metric; MPN (none) -> CR0201JM39RS01
- R106, R77, R78, R80, R83, R84, R85, R86, R87, R94: MPN (none) -> NRC04F1002TRF
- R107, R82, R89, R91, R92, R93, R96, R97: MPN (none) -> CR0402PC0RS001
- R108: MPN (none) -> CR0402FC1MS001
- R109, R88: footprint Resistor_SMD:R_0402_1005Metric -> Resistor_SMD:R_0201_0603Metric; MPN (none) -> CR0201JM39RS01
- R75, R76: MPN (none) -> RK73G1ETTP2200F
- R79, R81: MPN (none) -> CR0402FC100KS1
- R90: MPN (none) -> RC0402FR-07100RL
- R95: MPN (none) -> ERJ-2RKF2001X
- R98, R99: footprint Resistor_SMD:R_0201_0603Metric_Pad0.64x0.40mm_HandSolder -> Resistor_SMD:R_0201_0603Metric; MPN (none) -> CR0201JM39RS01; now not fitted
- SW1, SW2: MPN (none) -> NANOT160AS
- SW3: value SW_DIP_x02 -> 74404024010; MPN (none) -> 74404024010
- U15, U16: MPN (none) -> 9FGV0241AKLF
- U17: MPN (none) -> VSC8541XMV-02
- U18: MPN (none) -> ESP-PSRAM32; now not fitted
- U19: MPN (none) -> ESP32-PICO-D4; now not fitted
- Y3, Y4: MPN (none) -> ABM3B-25.000MHZ-D4Y-T
- Y5: value Crystal -> ABM3B-25.000MHZ-D4Y-T; MPN (none) -> ABM3B-25.000MHZ-D4Y-T
Connections:
- net RAM_CS: now also U19.29 (SD3/IO10); no longer U19.30 (CMD)
- net SIO3: now also U19.30 (CMD); no longer U19.25 (IO16)
Other:
- note removed: "needs reveiw"
- moved on the sheet: C310

Commit message: Regular Update.
Changed lines of the file:
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@@
 	(polyline
 		(pts
-			(xy 307.34 12.7) (xy 307.34 119.38)
+			(xy 307.34 12.065) (xy 307.34 119.38)
 		)
 		(stroke
@@
 	)
 	(rectangle
-		(start 307.34 12.7)
-		(end 340.36 15.24)
+		(start 307.34 12.065)
+		(end 340.36 14.605)
 		(stroke
 			(width -0.0001)
@@
 	(text "WIFI+BLUETOOTH ( OPTIONAL )"
 		(exclude_from_sim no)
-		(at 337.82 15.24 0)
+		(at 340.36 14.224 0)
 		(effects
 			(font
@@
 	(text "JTAG DEBUG"
 		(exclude_from_sim no)
-		(at 199.517 200.152 0)
+		(at 200.152 200.66 0)
 		(effects
 			(font
@@
 		(shape bidirectional)
 		(at 233.68 30.48 90)
-		(fields_autoplaced yes)
 		(effects
 			(font
@@
 		)
 		(property "Intersheetrefs" "${INTERSHEET_REFS}"
-			(at 235.54 30.48 90)
+			(at 233.68 24.384 90)
 			(effects
 				(font

Commit message: Update.
Parts:
- C288: renamed from C287; symbol awg1000:CAP_UNPOL -> SBC:C
- C289: renamed from C288; symbol awg1000:CAP_UNPOL -> SBC:C
- C290: renamed from C289; symbol awg1000:CAP_UNPOL -> SBC:C
- C291: renamed from C290; symbol awg1000:CAP_UNPOL -> SBC:C
- J1: symbol DQSBC:3-1827253-6 -> SBC:3-1827253-6
- J2: renamed from J3; value B10B-PHDSS -> B10B-PHDSS
- Q5, Q6, Q7: symbol Device:Q_NMOS_DGS -> Device:Q_NMOS_GSD
- renumbered C291 to C292, C292 to C293, C293 to C294, C294 to C295, C295 to C296, C296 to C297, C297 to C298, C298 to C299, C299 to C300, C300 to C301, C301 to C302, C302 to C303, C303 to C304, C304 to C305, C305 to C306, C306 to C307, C307 to C308, C308 to C309, C309 to C310, C310 to C311, C311 to C312, C312 to C313, C313 to C315, C315 to C316, C316 to C317, C317 to C318, C318 to C319, C319 to C320, C320 to C321, C321 to C322, C322 to C323, C323 to C324, C324 to C325, C325 to C326, C326 to C327, C327 to C328, C328 to C329, C329 to C330, C330 to C331, C331 to C332, C332 to C333, C333 to C334, C334 to C335, C335 to C336, C336 to C337, C337 to C338, C338 to C339, J4 to J3, J2 to J4, R99 to R100, R100 to R101, R101 to R102, R102 to R103, R103 to R104, R104 to R105, R105 to R106, R106 to R107, R107 to R108, R108 to R109, R109 to R110, R75 to R76, R76 to R77, R77 to R78, R78 to R79, R79 to R80, R80 to R81, R81 to R82, R82 to R83, R83 to R84, R84 to R85, R85 to R86, R86 to R87, R87 to R88, R88 to R89, R89 to R90, R90 to R91, R91 to R92, R92 to R93, R93 to R94, R94 to R95, R95 to R96, R96 to R97, R97 to R98, R98 to R99
Connections:
- net 3.3V_SW: no longer R76.1
- net BOOT_MODE0: now also Q7.3 (D); no longer Q7.1 (D)
- net BOOT_SEL: now also Q7.1 (G); no longer Q7.2 (G)
- net GND: now also Q5.2 (S), Q6.2 (S), Q7.2 (S); no longer Q5.3 (S), Q6.3 (S), Q7.3 (S)
- net GPIO0: now also Q6.1 (G); no longer Q6.2 (G)
- net PG_VIN: now also Q5.1 (G); no longer Q5.2 (G)
- net VIN: now also R76.1
- net at D5.1 (K): now also Q5.3 (D); no longer Q5.1 (D)
- net at D6.1 (K): now also Q6.3 (D); no longer Q6.1 (D)
Other:
- moved on the sheet: C293, C294, C295, C296, C297, C298, C299, C300, C302, C303, C304, C305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
