File: 02_ECAD/PWR.kicad_sch (KiCad schematic)
At the start: 144 parts, among them Q1 2SK3018-TP, Q2 SI7309DN-T1-E3, Q3 2SK3018-TP, U1 MC34PF4210A1ES, U2 SIC402ACD-T1-GE3, U3 TPS78412QDBVRQ1, U4 LDCL015, U5 MP2147GD-Z, U6 TPS62840, U7 MP2147GD-Z, U8 APX811-26UG-7

Commit message: Update.
Changed lines of the file:
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@@
   (global_label "PMIC_STBY_REQ" (shape input) (at 154.94 137.16 0) (fields_autoplaced)
     (effects (font (size 1 1)) (justify left))
-    (property "Intersheetrefs" "${INTERSHEET_REFS}" (at 168.7696 137.16 0)
+    (property "Intersheetrefs" "${INTERSHEET_REFS}" (at 168.957 137.16 0)
       (effects (font (size 1.27 1.27)) (justify left) hide)
     )
@@
     )
   )
-  (global_label "POR_B" (shape input) (at 154.94 132.08 0) (fields_autoplaced)
+  (global_label "POR_B" (shape output) (at 154.94 132.08 0) (fields_autoplaced)
     (effects (font (size 1 1)) (justify left))
-    (property "Intersheetrefs" "${INTERSHEET_REFS}" (at 161.9124 132.08 0)
+    (property "Intersheetrefs" "${INTERSHEET_REFS}" (at 162.0998 132.08 0)
       (effects (font (size 1.27 1.27)) (justify left) hide)
     )

Commit message: Update.
Parts:
- gave numbers to parts that had none: 3

Commit message: Update.
Parts:
- C1: value 22uF -> 2.2nF; MPN (none) -> KGM05AR71A222JH; Voltage V -> 10V
- C10, C11, C12, C13, C14, C15, C16, C18, C19, C2, C24, C25, C26, C3, C4, C48, C5, C6, C60, C7, C8, C9: MPN (none) -> CM05X5R475M16AH; Voltage V -> 16V
- C17: value 2.2uF -> 0.1uF; MPN (none) -> CC0402JRX7R7BB472; Voltage V -> 16V
- C20, C27, C28: MPN (none) -> GYC1H330MCW1GS
- C21, C22, C23, C29, C30, C31, C32, C33, C34, C37, C38, C39, C44, C45, C49, C50, C51, C52, C53, C54, C55, C58, C59, C61, C62, C64, C69: MPN (none) -> GRM158R61A226ME15D; Voltage V -> 10V
- C35, C40, C42, C46, C66, C67, C70: MPN (none) -> CL31A106KOHNNNE; Voltage (none) -> 16V
- C36, C41, C43: MPN (none) -> CL31A106KOHNNNE; VOLTAGE 16V -> 50V; Voltage (none) -> 16V
- C47: MPN (none) -> GRM033R61C224KE14D; VOLTAGE 16V -> 50V; Voltage (none) -> 16V
- C56: MPN (none) -> GRM155R61H105ME05D; Voltage V -> 50V
- C57: MPN (none) -> CC0402JRX7R7BB472; Voltage 50V -> 16V
- C63: MPN (none) -> GCM155R71E223KA55J; Voltage V -> 25V
- C65, C72, C74, C78, C79, C82, C86: value 100nF -> 0.1uF; MPN (none) -> GRM033Z71C104KE14D; Voltage (none) -> 16V
- C68, C73, C75, C76, C77, C83, C84, C85: MPN (none) -> CL10A226MO7JZNC; Voltage (none) -> 16V
- C71: MPN (none) -> GRM033R61C224KE14D; Voltage (none) -> 16V
- C80: MPN (none) -> 0603B102K500SD
- C81: value 1UF -> 1uF; MPN (none) -> 0603X105K500CT; Voltage (none) -> 50V
- D1: value D_TVS -> P4SMA30CA; MPN (none) -> P4SMA30CA
- D2: MPN (none) -> SD0603S040S0R2
- D3, D4: value ~ -> SD0603S040S0R2; MPN (none) -> SD0603S040S0R2
- L1, L2, L3, L4, L5: MPN (none) -> 74404024010
- L6: value 47uH -> 4.7uH; MPN (none) -> IHLP4040DZER4R7MA1
- L7: MPN (none) -> DFE201612E-2R2M=P2
- L8, L9: MPN (none) -> DFE252012F-R47M=P2
- Q1, Q3: MPN (none) -> 2SK3018-TP
- Q2: MPN (none) -> SI7309DN-T1-E3
- R1: value 7.15k -> 169k; MPN (none) -> CR0402-FX-1693GLF
- R10: MPN (none) -> CR0402FC100KS1
- R11: MPN (none) -> CR0402PC0RS001
- R12, R9: value 10K -> 10k; MPN (none) -> NRC04F1002TRF
- R13, R14: value 4.7K -> 4.7k; MPN (none) -> RN73R1ETTP4701F50
- R15: footprint Resistor_SMD:R_0402_1005Metric_Pad0.72x0.64mm_HandSolder -> Resistor_SMD:R_0402_1005Metric; MPN (none) -> CR0402-FX-4422GLF
- R16, R17, R21, R24, R27, R28: value 10K -> 10k; footprint Resistor_SMD:R_0402_1005Metric_Pad0.72x0.64mm_HandSolder -> Resistor_SMD:R_0402_1005Metric; MPN (none) -> NRC04F1002TRF
- R18: footprint Resistor_SMD:R_0402_1005Metric_Pad0.72x0.64mm_HandSolder -> Resistor_SMD:R_0402_1005Metric; MPN (none) -> CR0402FC100KS1
- R19: footprint Resistor_SMD:R_0402_1005Metric_Pad0.72x0.64mm_HandSolder -> Resistor_SMD:R_0402_1005Metric; MPN (none) -> CR0402PC0RS001
- R2: value 7.15k -> 30k; MPN (none) -> CR0402-FX-3002GLF
- R20: footprint Resistor_SMD:R_0402_1005Metric_Pad0.72x0.64mm_HandSolder -> Resistor_SMD:R_0402_1005Metric; MPN (none) -> RC0402FR-077K15L
- R22: footprint Resistor_SMD:R_0402_1005Metric_Pad0.72x0.64mm_HandSolder -> Resistor_SMD:R_0402_1005Metric; MPN (none) -> RC0402FR-076K98L
- R23: footprint Resistor_SMD:R_0402_1005Metric_Pad0.72x0.64mm_HandSolder -> Resistor_SMD:R_0402_1005Metric; MPN (none) -> CR0402-FX-5602GLF
- R25, R29: footprint Resistor_SMD:R_0402_1005Metric_Pad0.72x0.64mm_HandSolder -> Resistor_SMD:R_0402_1005Metric; MPN (none) -> CR0402-FX-1803GLF
- R26, R30: footprint Resistor_SMD:R_0402_1005Metric_Pad0.72x0.64mm_HandSolder -> Resistor_SMD:R_0402_1005Metric; MPN (none) -> CR0402FC360KS1
- R3: value 7.15k -> 1k; MPN (none) -> WR04X8251FTL; Part Number (none) -> WR04X8251FTL
- R31: footprint Resistor_SMD:R_0402_1005Metric_Pad0.72x0.64mm_HandSolder -> Resistor_SMD:R_0402_1005Metric; MPN (none) -> RC0402FR-07100RL
- R32: footprint Resistor_SMD:R_0402_1005Metric_Pad0.72x0.64mm_HandSolder -> Resistor_SMD:R_0402_1005Metric; MPN (none) -> CR0402FC1MS001
- R4: value 7.15k -> 4.53k; MPN (none) -> CR0402-FX-4531GLF
- R5: value 7.15k -> 100k; MPN (none) -> CR0402FC100KS1
- R6: value 7.15k -> 100; MPN (none) -> RC0402FR-07100RL
- R7: value 7.15k -> 10k; MPN (none) -> NRC04F1002TRF
- R8: value 7.15k -> 3.12k; MPN (none) -> RN73R1ETTP3121F25
- SH1, SH2: value ~ -> 0; MPN (none) -> RMCF0805ZT0R00
- U1: MPN (none) -> MC34PF4210A1ES
- U2: MPN (none) -> SIC402ACD-T1-GE3
- U3: MPN (none) -> TPS78412QDBVRQ1
- U4: MPN (none) -> LDCL015
- U5, U7: MPN (none) -> MP2147GD-Z
- U6: MPN (none) -> TPS62840
- U8: MPN (none) -> APX811-26UG-7
Connections:
- net GND: now also C36.2, C41.2, C43.2, C47.2; no longer C36.1, C41.1, C43.1, C47.1
- net VIN: now also C36.1, C41.1, C43.1, C47.1; no longer C36.2, C41.2, C43.2, C47.2
Other:
- note added: "Wrong connection,missing cap"
- moved on the sheet: C36, C41, C43, C47

Commit message: Regular Update.
Parts:
- C1: MPN KGM05AR71A222JH -> C0402C222J3GAC7867
- C21, C22, C23, C29, C30, C31, C32, C33, C34, C37, C38, C39, C44, C45, C49, C50, C51, C52, C53, C54, C55, C58, C59, C61, C62, C64, C69: MPN GRM158R61A226ME15D -> KGM05DR50J226MH; VOLTAGE (none) -> 6.3V
- C80: MPN 0603B102K500SD -> CL10B102KB8NNNC
- R10, R18, R5: MPN CR0402FC100KS1 -> RC0402FR-07100KL
- R11, R19: MPN CR0402PC0RS001 -> RC0402FR-070RL
- R12, R16, R17, R21, R24, R27, R28, R7, R9: MPN NRC04F1002TRF -> CR0402-FX-1002GLF
- R13, R14: MPN RN73R1ETTP4701F50 -> RC0402FR-074K7L
- R3: MPN WR04X8251FTL -> RC0402FR-071KL
- R32: MPN CR0402FC1MS001 -> RC0402FR-071ML
- R6: value 100 -> 100k
- R8: value 3.12k -> 3.16k; MPN RN73R1ETTP3121F25 -> RC0402FR-073K16L
- U4: value LDCL015 -> LDCL015MR; MPN LDCL015 -> LDCL015MR
- U6: value TPS62840 -> TPS62841DGRR

Commit message: Regular update.
Parts:
- Q2: value SI7309DN-T1-E3 -> SQS405CENW-T1_GE3

Commit message: Update.
Parts:
- added C29: 22uF, Capacitor_SMD:C_0603_1608Metric, symbol SBC:C
- added R9: 10k, Resistor_SMD:R_0402_1005Metric, symbol awg1000:R
- C36: renamed from C35; symbol awg1000:CAP_UNPOL -> SBC:C; Voltage 16V -> (none)
- C37: renamed from C36; symbol awg1000:CAP_UNPOL -> SBC:C; Voltage 16V -> (none)
- C41: renamed from C40; symbol awg1000:CAP_UNPOL -> SBC:C; Voltage 16V -> (none)
- C42: renamed from C41; symbol awg1000:CAP_UNPOL -> SBC:C; Voltage 16V -> (none)
- C43: renamed from C42; symbol awg1000:CAP_UNPOL -> SBC:C; Voltage 16V -> (none)
- C44: renamed from C43; symbol awg1000:CAP_UNPOL -> SBC:C; Voltage 16V -> (none)
- C47: renamed from C46; symbol awg1000:CAP_UNPOL -> SBC:C; Voltage 16V -> (none)
- C48: renamed from C47; symbol awg1000:CAP_UNPOL -> SBC:C; Voltage 16V -> (none)
- C66: renamed from C65; symbol awg1000:CAP_UNPOL -> SBC:C; Voltage 16V -> (none)
- C67: renamed from C66; symbol awg1000:CAP_UNPOL -> SBC:C; Voltage 16V -> (none)
- C68: renamed from C67; symbol awg1000:CAP_UNPOL -> SBC:C; Voltage 16V -> (none)
- C69: renamed from C68; symbol awg1000:CAP_UNPOL -> SBC:C; Voltage 16V -> (none)
- C71: renamed from C70; symbol awg1000:CAP_UNPOL -> SBC:C; Voltage 16V -> (none)
- C72: renamed from C71; symbol awg1000:CAP_UNPOL -> SBC:C; Voltage 16V -> (none)
- C73: renamed from C72; symbol awg1000:CAP_UNPOL -> SBC:C; Voltage 16V -> (none)
- C74: renamed from C73; symbol awg1000:CAP_UNPOL -> SBC:C; Voltage 16V -> (none)
- C75: renamed from C74; symbol awg1000:CAP_UNPOL -> SBC:C; Voltage 16V -> (none)
- C76: renamed from C75; symbol awg1000:CAP_UNPOL -> SBC:C; Voltage 16V -> (none)
- C77: renamed from C76; symbol awg1000:CAP_UNPOL -> SBC:C; Voltage 16V -> (none)
- C78: renamed from C77; symbol awg1000:CAP_UNPOL -> SBC:C; Voltage 16V -> (none)
- C79: renamed from C78; symbol awg1000:CAP_UNPOL -> SBC:C; Voltage 16V -> (none)
- C80: renamed from C79; symbol awg1000:CAP_UNPOL -> SBC:C; Voltage 16V -> (none)
- C81: renamed from C80; symbol awg1000:CAP_UNPOL -> SBC:C
- C82: renamed from C81; symbol awg1000:CAP_UNPOL -> SBC:C; Voltage 50V -> (none)
- C83: renamed from C82; symbol awg1000:CAP_UNPOL -> SBC:C; Voltage 16V -> (none)
- C84: renamed from C83; symbol awg1000:CAP_UNPOL -> SBC:C; Voltage 16V -> (none)
- C85: renamed from C84; symbol awg1000:CAP_UNPOL -> SBC:C; Voltage 16V -> (none)
- C86: renamed from C85; symbol awg1000:CAP_UNPOL -> SBC:C; Voltage 16V -> (none)
- C87: renamed from C86; symbol awg1000:CAP_UNPOL -> SBC:C; Voltage 16V -> (none)
- Q1, Q3: symbol Device:Q_NMOS_DGS -> Device:Q_NMOS_GSD
- R20: renamed from R19; now not fitted
- R21: renamed from R20; value 7.15k -> 4.32k; MPN RC0402FR-077K15L -> RC0402FR-074K32L
- U1: footprint DQSBC:QFN-56-1EP_8x8mm_P0.5mm_EP4.5x5.2mm_ThermalVias -> SBC:QFN-56-1EP_8x8mm_P0.5mm_EP4.5x5.2mm_ThermalVias
- U3: value TPS78412QDBVRQ1 -> TLV74310PDBVR; MPN TPS78412QDBVRQ1 -> TLV74310PDBVR
- U6: value TPS62841DGRR -> TPS62842DGR; MPN TPS62840 -> TPS62842DGR
- renumbered C29 to C30, C30 to C31, C31 to C32, C32 to C33, C33 to C34, C34 to C35, C37 to C38, C38 to C39, C39 to C40, C44 to C45, C45 to C46, C48 to C49, C49 to C50, C50 to C51, C51 to C52, C52 to C53, C53 to C54, C54 to C55, C55 to C56, C56 to C57, C57 to C58, C58 to C59, C59 to C60, C60 to C61, C61 to C62, C62 to C63, C63 to C64, C64 to C65, C69 to C70, R9 to R10, R10 to R11, R11 to R12, R12 to R13, R13 to R14, R14 to R15, R15 to R16, R16 to R17, R17 to R18, R18 to R19, R21 to R22, R22 to R23, R23 to R24, R24 to R25, R25 to R26, R26 to R27, R27 to R28, R28 to R29, R29 to R30, R30 to R31, R31 to R32, R32 to R33
Connections:
- net 3.3V_SW: now also C14.2, U1.40 (VIN3)
- net GND: now also Q1.2 (S), Q3.2 (S), R2.2, C29.2; no longer Q1.3 (S), Q3.3 (S)
- net NVCC_ENET_2V5: now also L7.2, U6.1 (VOS); no longer L7.1, U6.2 (SW)
- net PG_VIN: now also R9.2
- net PMIC_STBY_REQ: now also Q3.1 (G); no longer Q3.2 (G)
- net P_MODE: now also Q3.3 (D); no longer Q3.1 (D)
- net VIN: no longer R7.1
- net at Q1.1 (G): now also C58.1, R17.2; no longer R18.2
- net SIC4020A_VDD: now reaches R1.2, U2.3 (VDD)
- net SIC4020A_VDD: now also R7.1, C29.1, R9.1; no longer R2.2
- new net: Q1.3 (D), R18.2
- new net: L7.1, U6.2 (SW)
Other:
- note added: "3.3V 10A VIN SMPS"
- note removed: "3.3V 5A PMIC_VIN"
- note removed: "Wrong connection,missing cap"
- moved on the sheet: L7
