File: 02_ECAD/SBC.kicad_sch (KiCad schematic)
At the start: 0 parts

Commit message: Update.
Other:
- note added: "GPIOS"
- note added: "I2CS"
- note added: "PCIE 0.2 X 2"
- note added: "UARTS"
- note removed: "GPIO X"
- note removed: "I2C X"
- note removed: "PCIE X"
- note removed: "UART X"

Commit message: Skew Check.
Other:
- note added: "x32bits"
- note added: "x8bits"
Changed lines of the file:
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@@
 		)
 	)
-	(text_box "EMMC\n16 GB"
+	(text_box "EMMC 5.1\n16 GB"
 		(exclude_from_sim no)
 		(at 71.12 198.12 0)
@@
 		)
 	)
+	(text "x32bits"
+		(exclude_from_sim no)
+		(at 57.15 191.77 90)
+		(effects
+			(font
+				(size 1.016 1.016)
+			)
+		)
+	)
+	(text "x8bits"
+		(exclude_from_sim no)
+		(at 77.47 191.77 90)
+		(effects
+			(font
+				(size 1.016 1.016)
+			)
+		)
+	)

Commit message: Update.
Other:
- note added: "28.12.2023"
- note added: "INIT."
Changed lines of the file:
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@@
 	(title_block
 		(title "DQSBC")
-		(date "2023-05-13")
+		(date "2023-12-28")
 		(rev "1.00")
 	)
@@
 		)
 	)
+	(text "INIT."
+		(exclude_from_sim no)
+		(at 323.85 34.29 0)
+		(effects
+			(font
+				(size 2 2)
+				(color 132 0 0 1)
+			)
+			(justify right bottom)
+		)
+	)
 	(text "DSI"
 		(exclude_from_sim no)
@@
 			(font
 				(size 2 2)
+				(color 132 0 0 1)
 			)
 			(justify right bottom)
+		)
+	)
+	(text "28.12.2023"
+		(exclude_from_sim no)
+		(at 284.48 34.29 0)
+		(effects
+			(font
+				(size 2 2)
+				(color 132 0 0 1)
+			)
+			(justify right bottom)
