File: 03_TestingBaseboard/BB.kicad_sch (KiCad schematic)
At the start: 55 parts, among them J1 3-1827253-6, J10 HDMI_A, J12 USB_C_Receptacle, J13 Conn_02x05_Odd_Even, J14 Conn_02x05_Odd_Even, J2 B4P-VH(LF)(SN), J2 Conn_02x05_Odd_Even, J4 RJ45_RB1-125B8G1A, J4 USB3_A, J5 Micro_SD_Card_Det, J7 Conn_02x05_Odd_Even, J8 Conn_02x05_Odd_Even, J9 Bus_M.2_Socket_E, SW1 SW_Push, U1 PCMF3USB3S, U2 PTN36043ABX, U3 PCMF3USB3S, U4 PCMF3USB3S

Commit message: Update.
Parts:
- removed C4: 220uF, awg1000:EEE-FK1H221GP, symbol awg1000:CAP_POL
- removed D3: D, symbol Device:D
- removed J13, J14, J8: Conn_02x05_Odd_Even, Connector_PinHeader_1.00mm:PinHeader_2x05_P1.00mm_Vertical, symbol Connector_Generic:Conn_02x05_Odd_Even
- added C18, C21, C6: 10uF, Capacitor_SMD:C_1206_3216Metric, symbol awg1000:CAP_UNPOL
- added C19, C20, C7: 220nF, Capacitor_SMD:C_0603_1608Metric, symbol awg1000:CAP_UNPOL
- added D1, D13: SD0603S040S0R2, Diode_SMD:D_SOD-323, symbol Device:D_Schottky
- added D10, D5, D6, D7, D8, D9: ESD9B3.3ST5G, Diode_SMD:D_SOD-923, symbol Diode:ESD9B3.3ST5G
- added D12: SM6T24A, Diode_SMD:D_SMB, symbol Diode:SM6T24A
- added D4: ESD5Zxx, Diode_SMD:D_SOD-523, symbol Diode:ESD5Zxx
- added FB1: FerriteBead_Small, Inductor_SMD:L_0402_1005Metric, symbol Device:FerriteBead_Small
- added H1, H2, H3, H4: MountingHole_Pad, MountingHole:MountingHole_2.7mm_M2.5_DIN965_Pad_TopBottom, symbol Mechanical:MountingHole_Pad
- added J10, J11: Conn_01x09_Pin, Connector_PinSocket_1.00mm:PinSocket_1x09_P1.00mm_Vertical, symbol Connector:Conn_01x09_Pin
- added J8: Conn_01x15_Pin, Connector_PinSocket_1.00mm:PinSocket_1x15_P1.00mm_Vertical, symbol Connector:Conn_01x15_Pin
- added R1: 10K, Resistor_SMD:R_0402_1005Metric, symbol awg1000:R
- added R13, R15, R16, R17, R18, R19, R20: 49.9, Resistor_SMD:R_0402_1005Metric_Pad0.72x0.64mm_HandSolder, symbol awg1000:R
- added R2, R3, R4: 24.3K, Resistor_SMD:R_0402_1005Metric, symbol awg1000:R
- added R21: 1M, Resistor_SMD:R_0402_1005Metric_Pad0.72x0.64mm_HandSolder, symbol awg1000:R
- added TH1: Thermistor_PTC_US, Fuse:Fuse_0603_1608Metric_Pad1.05x0.95mm_HandSolder, symbol Device:Thermistor_PTC_US
- added U1: NX5P3090, SBC:WLCSP12_1.65X1.35, symbol SBC:NX5P3090UKZ
- added U6: LM397, Package_TO_SOT_SMD:SOT-23-5, symbol Comparator:LM397
- added U7, U8: PCMF3USB3S, Package_CSP:Nexperia_WLCSP-15_6-3-6_2.37x1.17mm_Layout6x3_P0.4mm, symbol Power_Protection:PCMF3USB3S
- C? (x8): footprint Capacitor_SMD:C_0603_1608Metric -> Capacitor_SMD:C_0402_1005Metric
- R85: footprint Resistor_SMD:R_0402_1005Metric_Pad0.72x0.64mm_HandSolder -> Resistor_SMD:R_0402_1005Metric
- U3: renamed from U2; footprint (none) -> SBC:DHX2QFN18
- renumbered D4 to D11, J9 to J14, J4 to J3, J2 to J5, J7 to J6, J12 to J7, U1 to U2, U3 to U4, U4 to U5
Connections:
- net GPIO1 is gone; now on net SPI1_SSO: J1.A79 (LVDS_A3-)
- net PCIE1_REF_CLKN is gone; now on net I2C2_SDA: J1.A45 (USB1_DN)
- net PCIE1_REF_CLKP is gone; now on net GND: J1.A46 (USB1_DP)
- net PCIE2_REF_CLKN is gone; now on net I2C3_SCL: J1.A42 (USB1_TX_N)
- net PCIE2_REF_CLKP is gone; now on net GND: J1.A43 (USB1_TX_P)
- net +5V: now also C20.1, C21.1, R1.2, R13.2, R15.2, R3.1, TH1.1, U1.B1 (VIN1), U1.B2 (VIN2), U1.C1 (VIN3), U6.5 (V+)
- net BOOT_SEL: now also J1.B42 (USB3-); no longer J1.B69 (PCIE_RX0-)
- net DSI_CLK_N: now also J1.B83 (eDP/LVDS_BKLT_CTRL), J8.3 (Pin_3); no longer J1.B28 (AC/HDA_SDIN2_(*))
- net DSI_CLK_P: now also J1.B82 (DDI0_PAIR3-), J8.2 (Pin_2); no longer J1.B29 (AC/HDA_SDIN1_(*))
- net DSI_D0_N: now also J1.B92 (DDI0_PAIR5-_(*)), J8.12 (Pin_12); no longer J1.B19 (SATA1_RX+)
- net DSI_D0_P: now also J1.B91 (DDI0_PAIR5+_(*)), J8.11 (Pin_11); no longer J1.B20 (SATA1_RX-)
- net DSI_D1_N: now also J1.B89 (DD0_HPD), J8.9 (Pin_9); no longer J1.B22 (USB_SSTX0-)
- net DSI_D1_P: now also J1.B88 (BIOS_DIS1#), J8.8 (Pin_8); no longer J1.B23 (USB_SSTX0+)
- net DSI_D2_N: now also J1.B95 (DDI0_DDC_AUX_SEL), J8.15 (Pin_15); no longer J1.B16 (SATA1_TX+)
- net DSI_D2_P: now also J1.B94 (DDI0_PAIR6-_(*)), J8.14 (Pin_14); no longer J1.B17 (SATA1_TX-)
- net DSI_D3_N: now also J1.B86 (VCC_5V_SBY), J8.6 (Pin_6); no longer J1.B25 (USB_SSTX1-_(*))
- net DSI_D3_P: now also J1.B85 (VCC_5V_SBY), J8.5 (Pin_5); no longer J1.B26 (USB_SSTX1+_(*))
- net GBE0_MDI0_N: now also J1.B100 (GND(FIXED)); no longer J1.B11 (GND(FIXED))
- net GBE0_MDI0_P: now also J1.B99 (DDI0_CTRLDATA_AUX-); no longer J1.B12 (PWRBTN#)
- net GBE0_MDI1_N: now also J1.B103 (SLEEP#); no longer J1.B8 (LPC_DRQ0#_(*))
- net GBE0_MDI1_P: now also J1.B102 (FAN_TACHIN); no longer J1.B9 (LPC_DRQ1#_(*))
- net GBE0_MDI2_N: now also J1.B106 (VCC_12V); no longer J1.B5 (SPI0_IO1)
- net GBE0_MDI2_P: now also J1.B105 (VCC_12V); no longer J1.B6 (SPI0_IO2)
- net GBE0_MDI3_N: now also J1.B109 (VCC_12V); no longer J1.B2 (GBE0_ACT#)
- net GBE0_MDI3_P: now also J1.B108 (VCC_12V); no longer J1.B3 (SPI0_NCS0)
- net GND: now also J1.A104 (VCC_12V), J1.A107 (VCC_12V), J1.A11 (GND(FIXED)), J1.A12 (GBE0_MDI0-), J1.A21 (GND(FIXED)), J1.A28 ((S)ATA_ACT#), J1.A31 (GND(FIXED)), J1.A34 (BIOS_DIS0#), J1.A37 (USB6+), J1.A40 (USB1_RX_P), J1.A49 (EXCD0_CPPE#), J1.A52 (RSVD), J1.A55 (RSVD), J1.A57 (GND), J1.A58 (PCIE_TX3+), J1.A61 (PCIE_TX2+), J1.A64 (PCIE_TX1+), J1.A67 (GPI2), J1.A70 (GND(FIXED)), J1.A73 (eDP_TX1+/LVDS_A1+), J1.A76 (eDP_TX0-/LVDS_A2-), J1.A8 (GBE0_LINK#), J1.A81 (eDP_TX3+/LVDS_A_CK+), J1.A86 (RSVD), J1.A89 (PCIE_CLK_REF-), J1.A9 (GBE0_MDI1-), J1.A92 (SPI_MISO_(**)), J1.A95 (SPI_MOSI_(**)), J1.B104 (VCC_12V), J1.B107 (VCC_12V), J1.B11 (GND(FIXED)), J1.B12 (PWRBTN#), J1.B14 (SMB_DAT), J1.B32 (SPKR), J1.B35 (THRM#), J1.B38 (USB_4_5_OC#), J1.B43 (USB3+), J1.B46 (USB1+), J1.B49 (SYS_RESET#), J1.B52 (RSVD), J1.B55 (RSVD), J1.B58 (PCIE_RX3+), J1.B61 (PCIE_RX2+), J1.B64 (PCIE_RX1+), J1.B67 (WAKE1#_(**)), J1.B72 (DDI0_PAIR0-), J1.B75 (DDI0_PAIR2+), J1.B78 (DDI0_PAIR4-_(*)), J1.B8 (LPC_DRQ0#_(*)), J1.B81 (DDI0_PAIR3+), J1.B9 (LPC_DRQ1#_(*)), J10.11 (CKS), J10.17 (GND), J10.2 (D2S), J10.5 (D1S), J10.8 (D0S), U5.B3 (GND_CH3), C18.2, C19.2, C20.2, C21.2, C6.2, C7.2, D10.1 (A1), D12.2 (A2), D4.2 (A), D5.1 (A1), D6.1 (A1), D7.1 (A1), D8.1 (A1), D9.1 (A1), J10.3 (Pin_3), J10.6 (Pin_6), J10.9 (Pin_9), J11.3 (Pin_3), J11.6 (Pin_6), J11.9 (Pin_9), J8.1 (Pin_1), J8.10 (Pin_10), J8.13 (Pin_13), J8.4 (Pin_4), J8.7 (Pin_7), R16.1, R18.1, R2.1, R21.2, R4.1, U1.B3 (GND1), U1.C3 (GND2), U1.D3 (GND3), U6.2 (V-), U7.B1 (GND_CH1), U7.B2 (GND_CH2), U7.B3 (GND_CH3), U8.B1 (GND_CH1), U8.B2 (GND_CH2), U8.B3 (GND_CH3); no longer J1.A100 (GND(FIXED)), J1.A102 (SER1_RX_(**)), J1.A103 (LID#), J1.A16 (SATA0_TX+), J1.A19 (SATA0_RX+), J1.A22 (USB_SSRX0-), J1.A25 (USB_SSRX1-_(*)), J1.A30 (AC/HDA_RST#_), J1.A35 (THRMTRIP#), J1.A38 (USB1_VBUS), J1.A4 (GBE0_LINK100#), J1.A41 (GND(FIXED)), J1.A44 (GND(FIXED)), J1.A47 (VCC_RTC), J1.A50 (LPC_SERIRQ_(**)), J1.A53 (RSVD), J1.A59 (PCIE_TX3-), J1.A62 (PCIE_TX2-), J1.A65 (PCIE_TX1-), J1.A68 (PCIE_TX0+), J1.A7 (GBE0_MDI2+), J1.A71 (eDP_TX2+/LVDS_A0+), J1.A74 (eDP_TX1-/LVDS_A1-), J1.A77 (eDP/LVDS_VDD_EN), J1.A80 (GND(FIXED)), J1.A83 (eDP_AUX+/LVDS_I2C_CK), J1.A90 (GND(FIXED)), J1.A99 (SER0_RX_(**)), J1.B100 (GND(FIXED)), J1.B102 (FAN_TACHIN), J1.B103 (SLEEP#), J1.B30 (AC/HDA_SDIN0_(**)), J1.B33 (I2C_CK), J1.B36 (USB7-_(*)), J1.B39 (USB5-), J1.B4 (SPI0_IO0), J1.B44 (USB_0_1_OC#), J1.B47 (EXCD1_PERST#), J1.B50 (CB_RESET#), J1.B53 (RSVD), J1.B56 (RSVD), J1.B59 (PCIE_RX3-), J1.B62 (PCIE_RX2-), J1.B65 (PCIE_RX1-), J1.B68 (PCIE_RX0+), J1.B7 (SPI0_IO3), J1.B73 (DDI0_PAIR1+), J1.B76 (DDI0_PAIR2-), J1.B79 (eDP/LVDS_BKLT_EN), J1.B97 (SPI_CS#_(**)), J1.B99 (DDI0_CTRLDATA_AUX-)
- net GPIO0: now also J1.A30 (AC/HDA_RST#_); no longer J1.A81 (eDP_TX3+/LVDS_A_CK+)
- net GPIO10: now also J1.A39 (USB1_RX_N); no longer J1.A72 (eDP_TX2-/LVDS_A0-)
- net GPIO3: now also J1.A29 (AC/HDA_SYNC_(**)); no longer J1.A82 (eDP_TX3-/LVDS_A_CK-)
- net GPIO4: now also J1.A27 (BATLOW#); no longer J1.A84 (eDP_AUX-/LVDS_I2C_DAT)
- net GPIO5: now also J1.A33 (AC/HDA_SDOUT_(**)); no longer J1.A78 (LVDS_A3+)
- net GPIO6: now also J1.A35 (THRMTRIP#); no longer J1.A76 (eDP_TX0-/LVDS_A2-)
- net GPIO8: now also J1.A36 (USB6-); no longer J1.A75 (eDP_TX0+/LVDS_A2+)
- net GPIO9: now also J1.A38 (USB1_VBUS); no longer J1.A73 (eDP_TX1+/LVDS_A1+)
- net HDMI_AUX_N: now also J1.B50 (CB_RESET#), R19.1, U7.C6 (CH3_OUT-); no longer J1.B61 (PCIE_RX2+)
- net HDMI_AUX_P: now also J1.B51 (GND(FIXED)), U7.C5 (CH3_OUT+); no longer J1.B60 (GND(FIXED))
- net HDMI_CEC: now also J1.B44 (USB_0_1_OC#); no longer J1.B67 (WAKE1#_(**))
- net HDMI_HDP: now also J1.B45 (USB1-), R19.2; no longer J1.B66 (WAKE0#), J10.19 (HPD)
- net HDMI_REFCLK_N: now also J1.B60 (GND(FIXED)); no longer J1.B51 (GND(FIXED)), J10.12 (CK-)
- net HDMI_REFCLK_P: now also J1.B59 (PCIE_RX3-); no longer J1.B52 (RSVD), J10.10 (CK+)
- net HDMI_SCL: now also J1.B47 (EXCD1_PERST#), U7.C4 (CH2_OUT-); no longer J1.B64 (PCIE_RX1+), J10.15 (SCL)
- net HDMI_SDA: now also J1.B48 (EXCD1_CPPE#), U7.C3 (CH2_OUT+); no longer J1.B63 (GPO3), J10.16 (SDA)
- net HDMI_TX0_N: now also J1.B56 (RSVD), U8.C6 (CH3_OUT-); no longer J1.B55 (RSVD), J10.9 (D0-)
- net HDMI_TX0_P: now also J1.B57 (GPO2), U8.C5 (CH3_OUT+); no longer J1.B54 (GPO1), J10.7 (D0+)
- net HDMI_TX1_N: now also J1.B54 (GPO1), U8.C4 (CH2_OUT-); no longer J1.B57 (GPO2), J10.6 (D1-)
- net HDMI_TX1_P: now also J1.B53 (RSVD), U8.C3 (CH2_OUT+); no longer J1.B58 (PCIE_RX3+), J10.4 (D1+)
- net HDMI_TX2_N: now also J1.B62 (PCIE_RX2-), U8.C2 (CH1_OUT-); no longer J1.B49 (SYS_RESET#), J10.3 (D2-)
- net HDMI_TX2_P: now also J1.B63 (GPO3), U8.C1 (CH1_OUT+); no longer J1.B48 (EXCD1_CPPE#), J10.1 (D2+)
- net HDMI_TX3_N: now also J1.B66 (WAKE0#), U7.C2 (CH1_OUT-); no longer J1.B45 (USB1-)
- net HDMI_TX3_P: now also J1.B65 (PCIE_RX1-), U7.C1 (CH1_OUT+); no longer J1.B46 (USB1+)
- net I2C1_SCL: now also J1.A48 (EXCD0_PERST#); no longer J1.A57 (GND)
- net I2C1_SDA: now also J1.A47 (VCC_RTC); no longer J1.A58 (PCIE_TX3+)
- net I2C2_SCL: now also J1.A44 (GND(FIXED)); no longer J1.A61 (PCIE_TX2+)
- net I2C2_SDA: no longer J1.A60 (GND(FIXED))
- net I2C3_SCL: no longer J1.A63 (GPI1)
- net I2C3_SDA: now also J1.A41 (GND(FIXED)); no longer J1.A64 (PCIE_TX1+)
- net LED0: now also J1.B97 (SPI_CS#_(**)); no longer J1.B14 (SMB_DAT)
- net LED1: now also J1.B96 (RSVD); no longer J1.B15 (SMB_ALERT#)
- net PCIE1_RXN: now also J1.A59 (PCIE_TX3-), J10.8 (Pin_8); no longer J1.A52 (RSVD)
- net PCIE1_RXP: now also J1.A60 (GND(FIXED)), J10.7 (Pin_7); no longer J1.A51 (GND(FIXED))
- net PCIE1_TXN: now also J1.A62 (PCIE_TX2-), J10.5 (Pin_5); no longer J1.A49 (EXCD0_CPPE#)
- net PCIE1_TXP: now also J1.A63 (GPI1), J10.4 (Pin_4); no longer J1.A48 (EXCD0_PERST#)
- net PCIE2_RXN: now also J1.A72 (eDP_TX2-/LVDS_A0-), J11.4 (Pin_4); no longer J1.A39 (USB1_RX_N)
- net PCIE2_RXP: now also J1.A71 (eDP_TX2+/LVDS_A0+), J11.5 (Pin_5); no longer J1.A40 (USB1_RX_P)
- net PCIE2_TXN: now also J1.A75 (eDP_TX0+/LVDS_A2+), J11.1 (Pin_1); no longer J1.A36 (USB6-)
- net PCIE2_TXP: now also J1.A74 (eDP_TX1-/LVDS_A1-), J11.2 (Pin_2); no longer J1.A37 (USB6+)
- net SD2_CLK: now also J1.B15 (SMB_ALERT#), D8.2 (A2); no longer J1.B96 (RSVD)
- net SD2_CMD: now also J1.B16 (SATA1_TX+), D7.2 (A2); no longer J1.B95 (DDI0_DDC_AUX_SEL)
- net SD2_D0: now also J1.B17 (SATA1_TX-), D9.2 (A2); no longer J1.B94 (DDI0_PAIR6-_(*))
- net SD2_D1: now also J1.B19 (SATA1_RX+), D10.2 (A2); no longer J1.B92 (DDI0_PAIR5-_(*))
- net SD2_D2: now also J1.B20 (SATA1_RX-), D5.2 (A2); no longer J1.B91 (DDI0_PAIR5+_(*))
- net SD2_D3: now also J1.B22 (USB_SSTX0-), D6.2 (A2); no longer J1.B89 (DD0_HPD)
- net SD2_WP: now also J1.B23 (USB_SSTX0+); no longer J1.B88 (BIOS_DIS1#)
- net SD2_nCD: now also J1.B25 (USB_SSTX1-_(*)); no longer J1.B86 (VCC_5V_SBY)
- net SD2_nRST: now also J1.B26 (USB_SSTX1+_(*)); no longer J1.B85 (VCC_5V_SBY)
- net SPI1_MISO: now also J1.A77 (eDP/LVDS_VDD_EN), J6.4 (Pin_4); no longer J1.A34 (BIOS_DIS0#), J6.8 (Pin_8)
- net SPI1_MOSI: now also J1.A78 (LVDS_A3+); no longer J1.A33 (AC/HDA_SDOUT_(**))
- net SPI1_SCLK: now also J1.A80 (GND(FIXED)), J6.10 (Pin_10); no longer J1.A31 (GND(FIXED)), J6.2 (Pin_2)
- net SPI1_SSO: now also J6.8 (Pin_8); no longer J1.A32 (AC/HDA_BITCLK_(**)), J6.4 (Pin_4)
- net SPI2_MISO: now also J1.A82 (eDP_TX3-/LVDS_A_CK-), J5.2 (Pin_2); no longer J1.A29 (AC/HDA_SYNC_(**)), J5.10 (Pin_10)
- net SPI2_MOSI: now also J1.A83 (eDP_AUX+/LVDS_I2C_CK), J5.4 (Pin_4); no longer J1.A28 ((S)ATA_ACT#), J5.8 (Pin_8)
- net SPI2_SCLK: now also J1.A85 (GPI3), J5.8 (Pin_8); no longer J1.A26 (USB_SSRX1+_(*)), J5.4 (Pin_4)
- net SPI2_SSO: now also J1.A84 (eDP_AUX-/LVDS_I2C_DAT); no longer J1.A27 (BATLOW#)
- net SYS_NRST: now also J1.A16 (SATA0_TX+); no longer J1.A95 (SPI_MOSI_(**))
- net SYS_NRST_OUT: now also J1.A15 (SUS_S3#); no longer J1.A96 (TPM_PP_(*))
- net UART1_RXD: now also J1.A93 (GPO0), J5.3 (Pin_3); no longer J1.A18 (SUS_S4#), J5.7 (Pin_7)
- net UART1_TXD: now also J1.A94 (SPI_CLK_(**)), J5.1 (Pin_1); no longer J1.A17 (SATA0_TX-), J5.9 (Pin_9)
- net UART2_RXD: now also J1.A88 (PCIE_CLK_REF+), J5.9 (Pin_9); no longer J1.A23 (USB_SSRX0+), J5.1 (Pin_1)
- net UART2_TXD: now also J1.A87 (eDP_HPD), J5.10 (Pin_10); no longer J1.A24 (SUS_S5#), J5.2 (Pin_2)
- net UART3_RXD: now also J1.A90 (GND(FIXED)), J5.7 (Pin_7); no longer J1.A21 (GND(FIXED)), J5.3 (Pin_3)
- net UART3_TXD: now also J1.A91 (SPI_POWER); no longer J1.A20 (SATA0_RX-)
- net UART4_RXD: now also J1.A51 (GND(FIXED)); no longer J1.A54 (GPI0)
- net UART4_TXD: now also J1.A50 (LPC_SERIRQ_(**)); no longer J1.A55 (RSVD)
- net USB1_DN: now also J1.B79 (eDP/LVDS_BKLT_EN), U2.C4 (CH2_OUT-); no longer J1.B32 (SPKR), U2.C1 (CH1_OUT+)
- net USB1_DP: now also J1.B80 (GND(FIXED)), U2.C3 (CH2_OUT+); no longer J1.B31 (GND(FIXED)), U2.C2 (CH1_OUT-)
- net USB1_ID1: now also J1.B69 (PCIE_RX0-); no longer J1.B42 (USB3-)
- net USB1_OC: now also J1.B71 (DDI0_PAIR0+); no longer J1.B40 (USB5+)
- net USB1_PWR_EN: now also J1.B68 (PCIE_RX0+); no longer J1.B43 (USB3+)
- net USB1_RX_N: now also J1.B73 (DDI0_PAIR1+), U2.C1 (CH1_OUT+); no longer J1.B38 (USB_4_5_OC#), U2.C3 (CH2_OUT+)
- net USB1_RX_P: now also J1.B74 (DDI0_PAIR1-), U2.C2 (CH1_OUT-); no longer J1.B37 (USB7+_(*)), U2.C4 (CH2_OUT-)
- net USB1_TX_N: now also J1.B76 (DDI0_PAIR2-); no longer J1.B35 (THRM#)
- net USB1_TX_P: now also J1.B77 (DDI0_PAIR4+_(*)); no longer J1.B34 (I2C_DAT)
- net USB1_VBUS: now also J1.B70 (GND(FIXED)), R3.2, R4.2; no longer J1.B41 (GND(FIXED)), J3.1 (VBUS)
- net USB2_DN: now also J1.A108 (VCC_12V), U4.C2 (CH1_OUT-); no longer J1.A3 (GBE0_MDI3+), U4.C1 (CH1_OUT+)
- net USB2_DP: now also J1.A109 (VCC_12V), U4.C1 (CH1_OUT+); no longer J1.A2 (GBE0_MDI3-), U4.C2 (CH1_OUT-)
- net USB2_ID1: now also J1.A100 (GND(FIXED)); no longer J1.A11 (GND(FIXED))
- net USB2_OC: now also J1.A96 (TPM_PP_(*)); no longer J1.A15 (SUS_S3#)
- net USB2_PWR_EN: now also J1.A97 (TYPE10#); no longer J1.A14 (GBE0_CTREF_(*))
- net USB2_RX_N: now also J1.A102 (SER1_RX_(**)); no longer J1.A9 (GBE0_MDI1-)
- net USB2_RX_P: now also J1.A103 (LID#); no longer J1.A8 (GBE0_LINK#)
- net USB2_TX_N: now also J1.A105 (VCC_12V); no longer J1.A6 (GBE0_MDI2-)
- net USB2_TX_P: now also J1.A106 (VCC_12V); no longer J1.A5 (GBE0_LINK1000#)
- net USB2_VBUS: now also J1.A99 (SER0_RX_(**)), R13.1, U6.4; no longer J1.A12 (GBE0_MDI0-)
- net VBAT: now also J1.A17 (SATA0_TX-); no longer J1.A94 (SPI_CLK_(**))
- net AP_N: now reaches C?.2, U3.14 (TX_AP-)
- net D1_N: now reaches J3.2 (D-)
- net D1_N: now also U2.A4 (CH2_IN-); no longer U2.A1 (CH1_IN+)
- net D1_P: now reaches J3.3 (D+)
- net D1_P: now also U2.A3 (CH2_IN+); no longer U2.A2 (CH1_IN-)
- net U2TX1_N: now reaches J7.A3 (TX1-), U4.A5 (CH3_IN+)
- net U2TX1_P: now reaches J7.A2 (TX1+), U4.A6 (CH3_IN-)
- net _TXC2_N: now reaches C?.1, U4.C5 (CH3_OUT+)
- net _TXC2_N: now also C?.2, U4.C6 (CH3_OUT-)
- net U2D_P: now reaches J7.A7 (D-), J7.B7 (D-), U4.A1 (CH1_IN+)
- net U2D_N: now reaches J7.A6 (D+), J7.B6 (D+), U4.A2 (CH1_IN-)
- net at C?.1: now also H4.1; no longer H3.1
- net TXC2_N: now reaches C?.1, U3.11 (TX_CON_2-)
- net AP_P: now reaches C?.1, U3.15 (TX_AP+)
- net U2RX2_N: now reaches J7.A10 (RX2-)
- net U2RX2_N: now also U5.A2 (CH1_IN-); no longer U5.A1 (CH1_IN+)
- net U2RX2_P: now reaches J7.A11 (RX2+)
- net U2RX2_P: now also U5.A1 (CH1_IN+); no longer U5.A2 (CH1_IN-)
- net RXC_P: now reaches U3.2 (RX_CON_1+), U5.C1 (CH1_OUT+)
- net RXC_N: now reaches U3.3 (RX_CON_1-), U5.C2 (CH1_OUT-)
- net C_VBUS: now reaches J7.A4 (VBUS), J7.A9 (VBUS), J7.B4 (VBUS), J7.B9 (VBUS)
- net C_VBUS: now also C18.1, C19.1, D12.1 (A1), R17.2
- net U1RX1_P: now reaches J7.B10 (RX1-), U4.A3 (CH2_IN+)
- net U1RX1_N: now reaches J7.B11 (RX1+), U4.A4 (CH2_IN-)
- net U2TX2_N: now reaches U5.A4 (CH2_IN-)
- net U2TX2_N: now also J7.B3 (TX2-); no longer J7.B2 (TX2+)
- net U2TX2_P: now reaches U5.A3 (CH2_IN+)
- net U2TX2_P: now also J7.B2 (TX2+); no longer J7.B3 (TX2-)
- net HEAC_P: now reaches J10.14 (UTILITY)
- net HEAC_P: now also U7.A5 (CH3_IN+)
- net HDMI_5V: now reaches J10.18 (+5V)
- net HDMI_5V: now also D13.1 (K), R20.1
- net TXC2_P: now reaches C?.2, U3.12 (TX_CON_2+)
- net HOST_PCIE1_CLK_N: now reaches J1.A66 (GND)
- net HOST_PCIE1_CLK_N: now also J10.1 (Pin_1)
- net HOST_PCIE2_CLK_N: now reaches J1.A69 (PCIE_TX0-)
- net HOST_PCIE2_CLK_N: now also J11.7 (Pin_7)
- net RX1_N: now reaches J3.5 (SSRX-)
- net RX1_N: now also U2.A1 (CH1_IN+); no longer U2.A3 (CH2_IN+)
- net RX1_P: now reaches J3.6 (SSRX+)
- net RX1_P: now also U2.A2 (CH1_IN-); no longer U2.A4 (CH2_IN-)
- net TX1_N: now reaches J3.8 (SSTX-), U2.A5 (CH3_IN+)
- net TX1_P: now reaches J3.9 (SSTX+), U2.A6 (CH3_IN-)
- net R_AP_N: now reaches C?.2, U3.17 (RX_AP-)
- net R_AP_P: now reaches C?.1, U3.18 (RX_AP+)
- net TXC1_P: now reaches C?.2, U3.6 (TX_CON_1+)
- net TXC1_N: now reaches C?.1, U3.7 (TX_CON_1-)
- net RX_C2_N: now reaches U3.8 (RX_CON_2-), U5.C4 (CH2_OUT-)
- net RX_C2_P: now reaches U3.9 (RX_CON_2+), U5.C3 (CH2_OUT+)
- net _TXC1_P: now reaches C?.1, U4.C3 (CH2_OUT+)
- net _TXC1_N: now reaches C?.2, U4.C4 (CH2_OUT-)
- removed net VIN_ACDC: C4.1, D1.2 (A2), J1.A104 (VCC_12V), J1.A105 (VCC_12V), J1.A106 (VCC_12V), J1.A107 (VCC_12V), J1.A108 (VCC_12V), J1.A109 (VCC_12V), J1.B104 (VCC_12V), J1.B105 (VCC_12V), J1.B106 (VCC_12V), J1.B107 (VCC_12V), J1.B108 (VCC_12V), J1.B109 (VCC_12V), J2.3 (Pin_3), J2.4 (Pin_4)
- new net: D13.2 (A), R20.2, TH1.2
- new net: FB1.1, U1.C2 (VBUS1), U1.D1 (VBUS2), U1.D2 (VBUS3)
- new net: R17.1, R18.2, U6.3 (+)
- new net: R1.1, U1.A1 (EN)
- new net: R15.1, R16.2, U6.1 (-)
- new net: D1.1 (K), U1.A2 (#FLT)
- new net: R2.2, U1.A3 (IL)
- new net HC_N: J10.12 (CK-), U7.A2 (CH1_IN-)
- new net HC_P: J10.10 (CK+), U7.A1 (CH1_IN+)
- new net HEAC_N: J10.19 (HPD), R21.1, U7.A6 (CH3_IN-)
- new net HOST_PCIE1_CLK_P: J1.A65 (PCIE_TX1-), J10.2 (Pin_2)
- new net HOST_PCIE2_CLK_P: J1.A68 (PCIE_TX0+), J11.8 (Pin_8)
- new net HSCL: J10.15 (SCL), U7.A4 (CH2_IN-)
- new net HSDA: J10.16 (SDA), U7.A3 (CH2_IN+)
- new net HTX0_N: J10.9 (D0-), U8.A6 (CH3_IN-)
- new net HTX0_P: J10.7 (D0+), U8.A5 (CH3_IN+)
- new net HTX1_N: J10.6 (D1-), U8.A4 (CH2_IN-)
- new net HTX1_P: J10.4 (D1+), U8.A3 (CH2_IN+)
- new net HTX2_N: J10.3 (D2-), U8.A2 (CH1_IN-)
- new net HTX2_P: J10.1 (D2+), U8.A1 (CH1_IN+)
- new net U1_VBUS: C6.1, C7.1, D4.1 (K), FB1.2, J3.1 (VBUS)
- new net VIN: C4.1, D1.2 (A2), J1.A2 (GBE0_MDI3-), J1.A3 (GBE0_MDI3+), J1.A4 (GBE0_LINK100#), J1.A5 (GBE0_LINK1000#), J1.A6 (GBE0_MDI2-), J1.A7 (GBE0_MDI2+), J1.B2 (GBE0_ACT#), J1.B3 (SPI0_NCS0), J1.B4 (SPI0_IO0), J1.B5 (SPI0_IO1), J1.B6 (SPI0_IO2), J1.B7 (SPI0_IO3), J2.3 (Pin_3), J2.4 (Pin_4)
Other:
- note added: "IOS"
- note added: "USB 3.0 HOST."
- note removed: "USB 3.0"
- moved on the sheet: C?, D11, FB10, FB11, FB9, H1, H3, J1, J10, J3, J4, J5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

Commit message: Regular Update.
Parts:
- removed C? (x4): 220nF, Capacitor_SMD:C_0603_1608Metric, symbol awg1000:CAP_UNPOL
- removed H2, H3 (x2): MountingHole_Pad, MountingHole:MountingHole_2.7mm_M2.5_DIN965_Pad_TopBottom, symbol Mechanical:MountingHole_Pad
- removed J14: Bus_M.2_Socket_E, symbol Connector:Bus_M.2_Socket_E
- removed R85: 49.9, Resistor_SMD:R_0402_1005Metric_Pad0.72x0.64mm_HandSolder, symbol awg1000:R
- added H4, H5, H6: MountingHole_Pad, MountingHole:MountingHole_2.7mm_M2.5_DIN965_Pad_TopBottom, symbol Mechanical:MountingHole_Pad
- SW1: footprint (none) -> Button_Switch_THT:SW_PUSH_1P1T_6x3.5mm_H4.3_APEM_MJTP1243
- renumbered C19 to C14, C18 to C15, C20 to C16, C21 to C17, C7 to C2, C6 to C3, D1 to D10, D10 to D3, D9 to D4, D8 to D5, D7 to D6, D6 to D7, D5 to D8, D4 to D9, FB1 to FB2, H4 to H8, J7 to J10, J3 to J4, J8 to J5, J5 to J7, J11 to J8, J10 to J9, R19 to R14, R20 to R19, R21 to R20, R3 to R7, R4 to R8
Connections:
- net RST_SW is gone; now on net SYS_NRST: SW1.2
- no-connect marks 24 -> 29
