File: 03_TestingBaseboard/Baseboard.kicad_pcb (KiCad board)
At the start: 4 copper layers, 122.5 x 102.5 mm, 36 parts, among them J1 3-1827253-6, J10 B4P-VH(LF)(SN), J11 B4P-VH(LF)(SN), J12 USB_C_Receptacle, J13 Conn_02x05_Odd_Even, J14 Conn_02x05_Odd_Even, J2 Conn_02x05_Odd_Even, J3 HDMI_A, J4 USB3_A, J5 RJ45_RB1-125B8G1A, J6 Micro_SD_Card_Det, J7 Conn_02x05_Odd_Even, J8 Conn_02x05_Odd_Even, U1 PCMF3USB3S, U3 PCMF3USB3S, U4 PCMF3USB3S

Commit message: Update.
Parts:
- removed the C1 at (96.7, 57.2)
- removed the J13 at (93.7, 142.7)
- removed J14: Conn_02x05_Odd_Even, Connector_PinHeader_1.00mm:PinHeader_2x05_P1.00mm_Vertical
- added C10: 220nF, Capacitor_SMD:C_0402_1005Metric, F.Cu at (114.0, 138.7)
- added C11: 220nF, Capacitor_SMD:C_0402_1005Metric, F.Cu at (114.0, 140.7)
- added C12: 220nF, Capacitor_SMD:C_0603_1608Metric, B.Cu at (117.3, 141.2)
- added C13: 220nF, Capacitor_SMD:C_0603_1608Metric, B.Cu at (117.3, 142.7)
- added C14: 220nF, Capacitor_SMD:C_0402_1005Metric, F.Cu at (123.9, 137.7)
- added C15: 220nF, Capacitor_SMD:C_0402_1005Metric, F.Cu at (121.9, 137.7)
- added C16: 220nF, Capacitor_SMD:C_0402_1005Metric, F.Cu at (122.9, 137.7)
- added C17: 220nF, Capacitor_SMD:C_0402_1005Metric, F.Cu at (120.9, 137.7)
- added C18: 10uF, Capacitor_SMD:C_1206_3216Metric, F.Cu at (136.7, 147.4)
- added C19: 220nF, Capacitor_SMD:C_0603_1608Metric, F.Cu at (138.8, 147.4)
- added C20: 220nF, Capacitor_SMD:C_0603_1608Metric, F.Cu at (147.9, 86.2)
- added C21: 10uF, Capacitor_SMD:C_1206_3216Metric, F.Cu at (145.9, 87.1)
- added C6: 10uF, Capacitor_SMD:C_1206_3216Metric, F.Cu at (154.7, 108.8)
- added C7: 220nF, Capacitor_SMD:C_0603_1608Metric, F.Cu at (154.8, 106.8)
- added C8: 220nF, Capacitor_SMD:C_0402_1005Metric, F.Cu at (114.0, 139.6)
- added C9: 220nF, Capacitor_SMD:C_0402_1005Metric, F.Cu at (114.0, 141.7)
- added D1: SD0603S040S0R2, Diode_SMD:D_SOD-323, F.Cu at (159.7, 110.2)
- added D10: ESD9B3.3ST5G, Diode_SMD:D_SOD-923, F.Cu at (62.9, 108.3)
- added D12: SM6T24A, Diode_SMD:D_SMB, F.Cu at (133.0, 147.1)
- added D13: SD0603S040S0R2, Diode_SMD:D_SOD-323, F.Cu at (150.4, 83.9)
- added D4: ESD5Zxx, Diode_SMD:D_SOD-523, F.Cu at (154.7, 105.3)
- added D5: ESD9B3.3ST5G, Diode_SMD:D_SOD-923, F.Cu at (62.2, 116.0)
- added D6: ESD9B3.3ST5G, Diode_SMD:D_SOD-923, F.Cu at (62.9, 114.9)
- added D7: ESD9B3.3ST5G, Diode_SMD:D_SOD-923, F.Cu at (62.2, 113.8)
- added D8: ESD9B3.3ST5G, Diode_SMD:D_SOD-923, F.Cu at (62.2, 111.6)
- added D9: ESD9B3.3ST5G, Diode_SMD:D_SOD-923, F.Cu at (62.2, 109.4)
- added FB1: FerriteBead_Small, Inductor_SMD:L_0402_1005Metric, F.Cu at (159.6, 105.5)
- added H5: MountingHole_Pad, MountingHole:MountingHole_2.7mm_M2.5_DIN965_Pad_TopBottom, F.Cu at (56.2, 84.7)
- added H6: MountingHole_Pad, MountingHole:MountingHole_2.7mm_M2.5_DIN965_Pad_TopBottom, F.Cu at (132.2, 131.7)
- added H8: MountingHole_Pad, MountingHole:MountingHole_2.7mm_M2.5_DIN965_Pad_TopBottom, F.Cu at (56.2, 131.7)
- added J10: Conn_01x09_Pin, Connector_PinSocket_1.00mm:PinSocket_1x09_P1.00mm_Vertical, F.Cu at (86.6, 149.4)
- added J11: Conn_01x09_Pin, Connector_PinSocket_1.00mm:PinSocket_1x09_P1.00mm_Vertical, F.Cu at (93.1, 149.4)
- added R1: 10K, Resistor_SMD:R_0402_1005Metric, F.Cu at (160.9, 108.3)
- added R10: 49.9, Resistor_SMD:R_0402_1005Metric, F.Cu at (116.4, 137.7)
- added R11: 49.9, Resistor_SMD:R_0402_1005Metric, F.Cu at (118.5, 143.3)
- added R12: 49.9, Resistor_SMD:R_0402_1005Metric, F.Cu at (115.4, 142.6)
- added R13: 49.9, Resistor_SMD:R_0402_1005Metric_Pad0.72x0.64mm_HandSolder, F.Cu at (147.4, 147.1)
- added R15: 49.9, Resistor_SMD:R_0402_1005Metric_Pad0.72x0.64mm_HandSolder, F.Cu at (144.2, 144.9)
- added R16: 49.9, Resistor_SMD:R_0402_1005Metric_Pad0.72x0.64mm_HandSolder, F.Cu at (142.0, 146.6)
- added R17: 49.9, Resistor_SMD:R_0402_1005Metric_Pad0.72x0.64mm_HandSolder, F.Cu at (145.6, 149.5)
- added R18: 49.9, Resistor_SMD:R_0402_1005Metric_Pad0.72x0.64mm_HandSolder, F.Cu at (143.3, 149.5)
- added R19: 49.9, Resistor_SMD:R_0402_1005Metric_Pad0.72x0.64mm_HandSolder, F.Cu at (123.1, 81.8)
- added R2: 24.3K, Resistor_SMD:R_0402_1005Metric, F.Cu at (158.6, 108.7)
- added R20: 49.9, Resistor_SMD:R_0402_1005Metric_Pad0.72x0.64mm_HandSolder, F.Cu at (150.4, 85.4)
- added R21: 1M, Resistor_SMD:R_0402_1005Metric_Pad0.72x0.64mm_HandSolder, F.Cu at (154.6, 85.5)
- added R3: 24.3K, Resistor_SMD:R_0402_1005Metric, F.Cu at (162.0, 109.5)
- added R4: 24.3K, Resistor_SMD:R_0402_1005Metric, F.Cu at (163.0, 109.5)
- added R5: 49.9, Resistor_SMD:R_0402_1005Metric, F.Cu at (116.4, 142.6)
- added R6: 49.9, Resistor_SMD:R_0402_1005Metric, F.Cu at (118.5, 142.3)
- added R7: 49.9, Resistor_SMD:R_0402_1005Metric, F.Cu at (115.4, 137.7)
- added R8: 49.9, Resistor_SMD:R_0402_1005Metric, F.Cu at (118.5, 137.4)
- added R9: 49.9, Resistor_SMD:R_0402_1005Metric, F.Cu at (118.5, 138.3)
- added TH1: Thermistor_PTC_US, Fuse:Fuse_0603_1608Metric_Pad1.05x0.95mm_HandSolder, F.Cu at (147.0, 83.9)
- added U1: NX5P3090, SBC:WLCSP12_1.65X1.35, F.Cu at (159.6, 107.2)
- added U3: PTN36043ABX, SBC:DHX2QFN18, F.Cu at (117.1, 140.1)
- added U6: LM397, Package_TO_SOT_SMD:SOT-23-5, F.Cu at (144.7, 147.2)
- added U7: PCMF3USB3S, Package_CSP:Nexperia_WLCSP-15_6-3-6_2.37x1.17mm_Layout6x3_P0.4mm, F.Cu at (150.4, 80.5)
- added U8: PCMF3USB3S, Package_CSP:Nexperia_WLCSP-15_6-3-6_2.37x1.17mm_Layout6x3_P0.4mm, F.Cu at (150.4, 76.0)
- J8: value Conn_02x05_Odd_Even -> Conn_01x15_Pin; footprint Connector_PinHeader_1.00mm:PinHeader_2x05_P1.00mm_Vertical -> Connector_PinSocket_1.00mm:PinSocket_1x15_P1.00mm_Vertical
- moved H2 142.1 mm to (-4.49, 74.3)
- moved H1 131.1 mm to (-4.49, 68.0)
- moved C2 104.2 mm to (136.9, 131.7)
- moved J4 103.7 mm to (51.7, 113.2), turned to -90 degrees
- moved C5 87.9 mm to (51.3, 131.8), turned to 180 degrees
- moved J1 83.8 mm to (53.7, 150.4), turned to 90 degrees
- moved H4 82.7 mm to (132.2, 84.7)
- moved D2 82.2 mm to (62.3, 144.6)
- moved FB3 76.6 mm to (150.5, 139.4), turned to 180 degrees
- moved H3 74.4 mm to (-4.49, 80.5)
- moved J8 69.3 mm to (142.8, 102.5)
- moved C4 68.4 mm to (136.9, 85.6)
- moved J7 66.5 mm to (125.0, 148.0)
- moved U4 66.0 mm to (122.7, 140.9), turned to 180 degrees
- moved U5 66.0 mm to (127.2, 140.9), turned to 180 degrees
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- renumbered C17 to C1, C18 to C2, C21 to C3, C19 to C4, C20 to C5, D1 to D2, D2 to D3, FB5 to FB2, FB4 to FB3, FB3 to FB4, H3 to H7, J10 to J1, J1 to J12, J3 to J13, J11 to J2, J4 to J3, J6 to J4, J2 to J5, J7 to J6, J12 to J7, J5 to J9, R9 to R14, U1 to U2, U3 to U4, U4 to U5
Connections:
- net Net-(J12-RX1+) renamed /BASEBOARD/U1RX1_N
- net Net-(J12-RX1-) renamed /BASEBOARD/U1RX1_P
- net Net-(J12-TX1+) renamed /BASEBOARD/U2TX1_P
- net Net-(J12-TX1-) renamed /BASEBOARD/U2TX1_N
- net Net-(J12-VBUS-PadA4) renamed /BASEBOARD/C_VBUS
- net Net-(J4-SSTX+) renamed /BASEBOARD/TX1_P
- net Net-(J4-SSTX-) renamed /BASEBOARD/TX1_N
- net Net-(U3A-CH1_IN+) renamed /BASEBOARD/U2D_P
- net Net-(U3A-CH1_IN-) renamed /BASEBOARD/U2D_N
- C1 pad 1: Net-(C17-Pad1) -> Net-(C1-Pad1)
- C2 pad 1: Net-(C18-Pad1) -> Net-(C2-Pad1)
- C3 pad 1: VIN_ACDC -> VIN
- C4 pad 1: Net-(C19-Pad1) -> Net-(C4-Pad1)
- C5 pad 1: Net-(C20-Pad1) -> Net-(C5-Pad1)
- D2 pad 2: VIN_ACDC -> VIN
- H1 pad 1: Net-(C17-Pad1) -> unconnected-(H1-Pad1)_0
- H2 pad 1: Net-(C18-Pad1) -> unconnected-(H2-Pad1)_0
- H3 pad 1: Net-(C19-Pad1) -> unconnected-(H3-Pad1)_1
- H4 pad 1: Net-(C20-Pad1) -> Net-(C4-Pad1)
- H7 pad 1: Net-(C19-Pad1) -> unconnected-(H7-Pad1)
- H7 pad 1: Net-(C19-Pad1) -> unconnected-(H7-Pad1)_0 (x2)
- H7 pad 1: Net-(C19-Pad1) -> unconnected-(H7-Pad1)_1
- J1 pad 3: VIN_ACDC -> VIN
- J1 pad 4: VIN_ACDC -> VIN
- J12 pad A100: GND -> USB2_ID1
- J12 pad A102: GND -> USB2_RX_N
- J12 pad A103: GND -> USB2_RX_P
- J12 pad A104: VIN_ACDC -> GND
- J12 pad A105: VIN_ACDC -> USB2_TX_N
- J12 pad A106: VIN_ACDC -> USB2_TX_P
- J12 pad A107: VIN_ACDC -> GND
- J12 pad A108: VIN_ACDC -> USB2_DN
- J12 pad A109: VIN_ACDC -> USB2_DP
- J12 pad A11: USB2_ID1 -> GND
- J12 pad A12: USB2_VBUS -> GND
- J12 pad A14: USB2_PWR_EN -> unconnected-(J12-GBE0_CTREF_(*)-PadA14)
- J12 pad A15: USB2_OC -> SYS_NRST_OUT
- J12 pad A16: GND -> SYS_NRST
- J12 pad A17: UART1_TXD -> VBAT
- J12 pad A18: UART1_RXD -> unconnected-(J12-SUS_S4#-PadA18)
- J12 pad A19: GND -> unconnected-(J12-SATA0_RX+-PadA19)
- J12 pad A2: USB2_DP -> VIN
- J12 pad A20: UART3_TXD -> unconnected-(J12-SATA0_RX--PadA20)
- J12 pad A21: UART3_RXD -> GND
- J12 pad A22: GND -> unconnected-(J12-USB_SSRX0--PadA22)
- J12 pad A23: UART2_RXD -> unconnected-(J12-USB_SSRX0+-PadA23)
- J12 pad A24: UART2_TXD -> unconnected-(J12-SUS_S5#-PadA24)
- J12 pad A25: GND -> unconnected-(J12-USB_SSRX1-_(*)-PadA25)
- J12 pad A26: SPI2_SCLK -> unconnected-(J12-USB_SSRX1+_(*)-PadA26)
- J12 pad A27: SPI2_SSO -> GPIO4
- J12 pad A28: SPI2_MOSI -> GND
- J12 pad A29: SPI2_MISO -> GPIO3
- J12 pad A3: USB2_DN -> VIN
- J12 pad A30: GND -> GPIO0
- J12 pad A31: SPI1_SCLK -> GND
- J12 pad A32: SPI1_SSO -> unconnected-(J12-AC/HDA_BITCLK_(**)-PadA32)
- J12 pad A33: SPI1_MOSI -> GPIO5
- J12 pad A34: SPI1_MISO -> GND
- J12 pad A35: GND -> GPIO6
- J12 pad A36: PCIE2_TXN -> GPIO8
- J12 pad A37: PCIE2_TXP -> GND
- J12 pad A38: GND -> GPIO9
- J12 pad A39: PCIE2_RXN -> GPIO10
- J12 pad A4: GND -> VIN
- J12 pad A40: PCIE2_RXP -> GND
- J12 pad A41: GND -> I2C3_SDA
- J12 pad A42: PCIE2_REF_CLKN -> I2C3_SCL
- J12 pad A43: PCIE2_REF_CLKP -> GND
- J12 pad A44: GND -> I2C2_SCL
- J12 pad A45: PCIE1_REF_CLKN -> I2C2_SDA
- J12 pad A46: PCIE1_REF_CLKP -> GND
- J12 pad A47: GND -> I2C1_SDA
- J12 pad A48: PCIE1_TXP -> I2C1_SCL
- J12 pad A49: PCIE1_TXN -> GND
- J12 pad A5: USB2_TX_P -> VIN
- J12 pad A50: GND -> UART4_TXD
- J12 pad A51: PCIE1_RXP -> UART4_RXD
- J12 pad A52: PCIE1_RXN -> GND
- J12 pad A53: GND -> unconnected-(J12-RSVD-PadA53)
- J12 pad A54: UART4_RXD -> unconnected-(J12-GPI0-PadA54)
- J12 pad A55: UART4_TXD -> GND
- J12 pad A57: I2C1_SCL -> GND
- J12 pad A58: I2C1_SDA -> GND
- J12 pad A59: GND -> PCIE1_RXN
- J12 pad A6: USB2_TX_N -> VIN
- J12 pad A60: I2C2_SDA -> PCIE1_RXP
- J12 pad A61: I2C2_SCL -> GND
- J12 pad A62: GND -> PCIE1_TXN
- J12 pad A63: I2C3_SCL -> PCIE1_TXP
- J12 pad A64: I2C3_SDA -> GND
- J12 pad A65: GND -> HOST_PCIE1_CLK_P
- J12 pad A66: unconnected-(J1-GND-PadA66) -> HOST_PCIE1_CLK_N
- J12 pad A67: unconnected-(J1-GPI2-PadA67) -> GND
- J12 pad A68: GND -> HOST_PCIE2_CLK_P
- J12 pad A69: unconnected-(J1-PCIE_TX0--PadA69) -> HOST_PCIE2_CLK_N
- J12 pad A7: GND -> VIN
- J12 pad A70: unconnected-(J1-GND(FIXED)-PadA70) -> GND
- J12 pad A71: GND -> PCIE2_RXP
- J12 pad A72: GPIO10 -> PCIE2_RXN
- J12 pad A73: GPIO9 -> GND
- J12 pad A74: GND -> PCIE2_TXP
- J12 pad A75: GPIO8 -> PCIE2_TXN
- J12 pad A76: GPIO6 -> GND
- J12 pad A77: GND -> SPI1_MISO
- J12 pad A78: GPIO5 -> SPI1_MOSI
- J12 pad A79: GPIO1 -> SPI1_SSO
- J12 pad A8: USB2_RX_P -> GND
- J12 pad A80: GND -> SPI1_SCLK
- J12 pad A81: GPIO0 -> GND
- J12 pad A82: GPIO3 -> SPI2_MISO
- J12 pad A83: GND -> SPI2_MOSI
- J12 pad A84: GPIO4 -> SPI2_SSO
- J12 pad A85: unconnected-(J1-GPI3-PadA85) -> SPI2_SCLK
- J12 pad A86: unconnected-(J1-RSVD-PadA86) -> GND
- J12 pad A87: unconnected-(J1-eDP_HPD-PadA87) -> UART2_TXD
- J12 pad A88: unconnected-(J1-PCIE_CLK_REF+-PadA88) -> UART2_RXD
- J12 pad A89: unconnected-(J1-PCIE_CLK_REF--PadA89) -> GND
- J12 pad A9: USB2_RX_N -> GND
- J12 pad A90: GND -> UART3_RXD
- J12 pad A91: unconnected-(J1-SPI_POWER-PadA91) -> UART3_TXD
- J12 pad A92: unconnected-(J1-SPI_MISO_(**)-PadA92) -> GND
- J12 pad A93: unconnected-(J1-GPO0-PadA93) -> UART1_RXD
- J12 pad A94: VBAT -> UART1_TXD
- J12 pad A95: SYS_NRST -> GND
- J12 pad A96: SYS_NRST_OUT -> USB2_OC
- J12 pad A97: unconnected-(J1-TYPE10#-PadA97) -> USB2_PWR_EN
- J12 pad A99: GND -> USB2_VBUS
- J12 pad B100: GND -> GBE0_MDI0_N
- J12 pad B102: GND -> GBE0_MDI1_P
- J12 pad B103: GND -> GBE0_MDI1_N
- J12 pad B104: VIN_ACDC -> GND
- J12 pad B105: VIN_ACDC -> GBE0_MDI2_P
- J12 pad B106: VIN_ACDC -> GBE0_MDI2_N
- J12 pad B107: VIN_ACDC -> GND
- J12 pad B108: VIN_ACDC -> GBE0_MDI3_P
- J12 pad B109: VIN_ACDC -> GBE0_MDI3_N
- J12 pad B11: GBE0_MDI0_N -> GND
- J12 pad B12: GBE0_MDI0_P -> GND
- J12 pad B14: /BASEBOARD/LED0 -> GND
- J12 pad B15: /BASEBOARD/LED1 -> SD2_CLK
- J12 pad B16: DSI_D2_N -> SD2_CMD
- J12 pad B17: DSI_D2_P -> SD2_D0
- J12 pad B19: DSI_D0_N -> SD2_D1
- J12 pad B2: GBE0_MDI3_N -> VIN
- J12 pad B20: DSI_D0_P -> SD2_D2
- J12 pad B22: DSI_D1_N -> SD2_D3
- J12 pad B23: DSI_D1_P -> SD2_WP
- J12 pad B25: DSI_D3_N -> SD2_nCD
- J12 pad B26: DSI_D3_P -> SD2_nRST
- J12 pad B28: DSI_CLK_N -> unconnected-(J12-AC/HDA_SDIN2_(*)-PadB28)
- J12 pad B29: DSI_CLK_P -> unconnected-(J12-AC/HDA_SDIN1_(*)-PadB29)
- J12 pad B3: GBE0_MDI3_P -> VIN
- J12 pad B30: GND -> unconnected-(J12-AC/HDA_SDIN0_(**)-PadB30)
- J12 pad B31: USB1_DP -> unconnected-(J12-GND(FIXED)-PadB31)
- J12 pad B32: USB1_DN -> GND
- J12 pad B33: GND -> unconnected-(J12-I2C_CK-PadB33)
- J12 pad B34: USB1_TX_P -> unconnected-(J12-I2C_DAT-PadB34)
- J12 pad B35: USB1_TX_N -> GND
- J12 pad B36: GND -> unconnected-(J12-USB7-_(*)-PadB36)
- J12 pad B37: USB1_RX_P -> unconnected-(J12-USB7+_(*)-PadB37)
- J12 pad B38: USB1_RX_N -> GND
- J12 pad B39: GND -> unconnected-(J12-USB5--PadB39)
- J12 pad B4: GND -> VIN
- J12 pad B40: USB1_OC -> unconnected-(J12-USB5+-PadB40)
- J12 pad B41: USB1_VBUS -> unconnected-(J12-GND(FIXED)-PadB41)
- J12 pad B42: USB1_ID1 -> BOOT_SEL
- J12 pad B43: USB1_PWR_EN -> GND
- J12 pad B44: GND -> HDMI_CEC
- J12 pad B45: HDMI_TX3_N -> HDMI_HDP
- J12 pad B46: HDMI_TX3_P -> GND
- J12 pad B47: GND -> HDMI_SCL
- J12 pad B48: HDMI_TX2_P -> HDMI_SDA
- J12 pad B49: HDMI_TX2_N -> GND
- J12 pad B5: GBE0_MDI2_N -> VIN
- J12 pad B50: GND -> HDMI_AUX_N
- J12 pad B51: HDMI_REFCLK_N -> HDMI_AUX_P
- J12 pad B52: HDMI_REFCLK_P -> GND
- J12 pad B53: GND -> HDMI_TX1_P
- J12 pad B54: HDMI_TX0_P -> HDMI_TX1_N
- J12 pad B55: HDMI_TX0_N -> GND
- J12 pad B56: GND -> HDMI_TX0_N
- J12 pad B57: HDMI_TX1_N -> HDMI_TX0_P
- J12 pad B58: HDMI_TX1_P -> GND
- J12 pad B59: GND -> HDMI_REFCLK_P
- J12 pad B6: GBE0_MDI2_P -> VIN
- J12 pad B60: HDMI_AUX_P -> HDMI_REFCLK_N
- J12 pad B61: HDMI_AUX_N -> GND
- J12 pad B62: GND -> HDMI_TX2_N
- J12 pad B63: HDMI_SDA -> HDMI_TX2_P
- J12 pad B64: HDMI_SCL -> GND
- J12 pad B65: GND -> HDMI_TX3_P
- J12 pad B66: HDMI_HDP -> HDMI_TX3_N
- J12 pad B67: HDMI_CEC -> GND
- J12 pad B68: GND -> USB1_PWR_EN
- J12 pad B69: BOOT_SEL -> USB1_ID1
- J12 pad B7: GND -> VIN
- J12 pad B70: unconnected-(J1-GND(FIXED)-PadB70) -> USB1_VBUS
- J12 pad B71: unconnected-(J1-DDI0_PAIR0+-PadB71) -> USB1_OC
- J12 pad B72: unconnected-(J1-DDI0_PAIR0--PadB72) -> GND
- J12 pad B73: GND -> USB1_RX_N
- J12 pad B74: unconnected-(J1-DDI0_PAIR1--PadB74) -> USB1_RX_P
- J12 pad B75: unconnected-(J1-DDI0_PAIR2+-PadB75) -> GND
- J12 pad B76: GND -> USB1_TX_N
- J12 pad B77: unconnected-(J1-DDI0_PAIR4+_(*)-PadB77) -> USB1_TX_P
- J12 pad B78: unconnected-(J1-DDI0_PAIR4-_(*)-PadB78) -> GND
- J12 pad B79: GND -> USB1_DN
- J12 pad B8: GBE0_MDI1_N -> GND
- J12 pad B80: unconnected-(J1-GND(FIXED)-PadB80) -> USB1_DP
- J12 pad B81: unconnected-(J1-DDI0_PAIR3+-PadB81) -> GND
- J12 pad B82: unconnected-(J1-DDI0_PAIR3--PadB82) -> DSI_CLK_P
- J12 pad B83: unconnected-(J1-eDP/LVDS_BKLT_CTRL-PadB83) -> DSI_CLK_N
- J12 pad B85: SD2_nRST -> DSI_D3_P
- J12 pad B86: SD2_nCD -> DSI_D3_N
- J12 pad B88: SD2_WP -> DSI_D1_P
- J12 pad B89: SD2_D3 -> DSI_D1_N
- J12 pad B9: GBE0_MDI1_P -> GND
- J12 pad B91: SD2_D2 -> DSI_D0_P
- J12 pad B92: SD2_D1 -> DSI_D0_N
- J12 pad B94: SD2_D0 -> DSI_D2_P
- J12 pad B95: SD2_CMD -> DSI_D2_N
- J12 pad B96: SD2_CLK -> /BASEBOARD/LED1
- J12 pad B97: GND -> /BASEBOARD/LED0
- J12 pad B99: GND -> GBE0_MDI0_P
- J13 pad 1: HDMI_TX2_P -> /BASEBOARD/HTX2_P
- J13 pad 10: HDMI_REFCLK_P -> /BASEBOARD/HC_P
- J13 pad 11: unconnected-(J3-CKS-Pad11) -> GND
- J13 pad 12: HDMI_REFCLK_N -> /BASEBOARD/HC_N
- J13 pad 14: unconnected-(J3-UTILITY-Pad14) -> /BASEBOARD/HEAC_P
- J13 pad 15: HDMI_SCL -> /BASEBOARD/HSCL
- J13 pad 16: HDMI_SDA -> /BASEBOARD/HSDA
- J13 pad 17: unconnected-(J3-GND-Pad17) -> GND
- J13 pad 18: unconnected-(J3-+5V-Pad18) -> /BASEBOARD/HDMI_5V
- J13 pad 19: HDMI_HDP -> /BASEBOARD/HEAC_N
- J13 pad 2: unconnected-(J3-D2S-Pad2) -> GND
- J13 pad 3: HDMI_TX2_N -> /BASEBOARD/HTX2_N
- J13 pad 4: HDMI_TX1_P -> /BASEBOARD/HTX1_P
- J13 pad 5: unconnected-(J3-D1S-Pad5) -> GND
- J13 pad 6: HDMI_TX1_N -> /BASEBOARD/HTX1_N
- J13 pad 7: HDMI_TX0_P -> /BASEBOARD/HTX0_P
- J13 pad 8: unconnected-(J3-D0S-Pad8) -> GND
- J13 pad 9: HDMI_TX0_N -> /BASEBOARD/HTX0_N
- J3 pad 1: USB1_VBUS -> /BASEBOARD/U1_VBUS
- J3 pad 2: Net-(J4-D-) -> /BASEBOARD/D1_N
- J3 pad 3: Net-(J4-D+) -> /BASEBOARD/D1_P
- J3 pad 5: Net-(J4-SSRX-) -> /BASEBOARD/RX1_N
- J3 pad 6: Net-(J4-SSRX+) -> /BASEBOARD/RX1_P
- J5 pad 1: UART2_RXD -> UART1_TXD
- J5 pad 10: SPI2_MISO -> UART2_TXD
- J5 pad 2: UART2_TXD -> SPI2_MISO
- J5 pad 3: UART3_RXD -> UART1_RXD
- J5 pad 4: SPI2_SCLK -> SPI2_MOSI
- J5 pad 7: UART1_RXD -> UART3_RXD
- J5 pad 8: SPI2_MOSI -> SPI2_SCLK
- J5 pad 9: UART1_TXD -> UART2_RXD
- J6 pad 10: unconnected-(J7-Pin_10-Pad10) -> SPI1_SCLK
- J6 pad 2: SPI1_SCLK -> unconnected-(J6-Pin_2-Pad2)
- J6 pad 4: SPI1_SSO -> SPI1_MISO
- J6 pad 8: SPI1_MISO -> SPI1_SSO
- J7 pad A10: Net-(J12-RX2-) -> /BASEBOARD/U2RX2_N
- J7 pad A11: Net-(J12-RX2+) -> /BASEBOARD/U2RX2_P
- J7 pad B2: Net-(J12-TX2+) -> /BASEBOARD/U2TX2_P
- J7 pad B3: Net-(J12-TX2-) -> /BASEBOARD/U2TX2_N
- J8 pad 2: unconnected-(J8-Pin_2-Pad2) -> DSI_CLK_P
- J8 pad 3: unconnected-(J8-Pin_3-Pad3) -> DSI_CLK_N
- J8 pad 5: unconnected-(J8-Pin_5-Pad5) -> DSI_D3_P
- J8 pad 6: unconnected-(J8-Pin_6-Pad6) -> DSI_D3_N
- J8 pad 8: unconnected-(J8-Pin_8-Pad8) -> DSI_D1_P
- J8 pad 9: unconnected-(J8-Pin_9-Pad9) -> DSI_D1_N
- U2 pad A1: Net-(J4-D-) -> /BASEBOARD/RX1_N
- U2 pad A2: Net-(J4-D+) -> /BASEBOARD/RX1_P
- U2 pad A3: Net-(J4-SSRX-) -> /BASEBOARD/D1_P
- U2 pad A4: Net-(J4-SSRX+) -> /BASEBOARD/D1_N
- U2 pad C1: USB1_DN -> USB1_RX_N
- U2 pad C2: USB1_DP -> USB1_RX_P
- U2 pad C3: USB1_RX_N -> USB1_DP
- U2 pad C4: USB1_RX_P -> USB1_DN
- U4 pad C1: USB2_DN -> USB2_DP
- U4 pad C2: USB2_DP -> USB2_DN
- U4 pad C3: unconnected-(U3B-CH2_OUT+-PadC3) -> /BASEBOARD/_TXC1_P
- U4 pad C4: unconnected-(U3B-CH2_OUT--PadC4) -> /BASEBOARD/_TXC1_N
- U4 pad C5: unconnected-(U3C-CH3_OUT+-PadC5) -> /BASEBOARD/_TXC2_P
- U4 pad C6: unconnected-(U3C-CH3_OUT--PadC6) -> /BASEBOARD/_TXC2_N
- U5 pad A1: Net-(J12-RX2-) -> /BASEBOARD/U2RX2_P
- U5 pad A2: Net-(J12-RX2+) -> /BASEBOARD/U2RX2_N
- U5 pad A3: Net-(J12-TX2-) -> /BASEBOARD/U2TX2_P
- U5 pad A4: Net-(J12-TX2+) -> /BASEBOARD/U2TX2_N
- U5 pad C1: unconnected-(U4A-CH1_OUT+-PadC1) -> /BASEBOARD/RXC_P
- U5 pad C2: unconnected-(U4A-CH1_OUT--PadC2) -> /BASEBOARD/RXC_N
- U5 pad C3: unconnected-(U4B-CH2_OUT+-PadC3) -> /BASEBOARD/RX_C2_P
- U5 pad C4: unconnected-(U4B-CH2_OUT--PadC4) -> /BASEBOARD/RX_C2_N
Routing:
- net HDMI_CEC: track 0.00 -> 111.6 mm, vias 0 -> 2
- net USB1_VBUS: track 0.00 -> 103.1 mm
- net HDMI_SCL: track 0.00 -> 97.6 mm, vias 0 -> 2
- net HDMI_SDA: track 0.00 -> 93.5 mm
- net HDMI_AUX_N: track 0.00 -> 93.3 mm, vias 0 -> 2
- net HDMI_AUX_P: track 0.00 -> 92.7 mm, vias 0 -> 2
- net HDMI_TX3_P: track 0.00 -> 89.5 mm, vias 0 -> 2
- net HDMI_TX3_N: track 0.00 -> 88.9 mm, vias 0 -> 2
- net GND: track 81.7 -> 167.4 mm, vias 41 -> 144
- net HDMI_HDP: track 0.00 -> 74.3 mm, vias 0 -> 2
- net /BASEBOARD/LED0: track 0.00 -> 61.3 mm
- net GBE0_MDI3_P: track 101.4 -> 40.2 mm, vias 0 -> 1
- net /BASEBOARD/LED1: track 0.00 -> 60.8 mm
- net HDMI_TX2_N: track 39.3 -> 92.2 mm, vias 0 -> 2
- net HDMI_TX2_P: track 39.9 -> 91.6 mm, vias 0 -> 2
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- added copper zone on F.Cu, net +5V
- added copper zone on In2.Cu, net +5V
- added copper zone on F.Cu, net /BASEBOARD/C_VBUS
- added copper zone on In2.Cu, net /BASEBOARD/C_VBUS
- added copper zone on F.Cu, net /BASEBOARD/U1_VBUS
- added copper zone on F.Cu, net GND
- added copper zone on In1.Cu, net GND
- added copper zone on F.Cu, net Net-(U1-VBUS1)
- added copper zone on F.Cu, net VIN
- removed copper zone on F.Cu, net VIN_ACDC

Commit message: Regular Update.
Parts:
- removed the C1 at (61.0, 84.7)
- removed the C2 at (136.9, 131.7)
- removed the C4 at (136.9, 85.6)
- removed the C5 at (51.3, 131.8)
- removed H1: MountingHole_Pad, MountingHole:MountingHole_2.7mm_M2.5_DIN965_Pad_TopBottom
- removed the H2 at (-4.49, 74.3)
- removed the H3 at (-4.49, 80.5)
- removed the H7 at (159.2, 55.9)
- removed the H7 at (46.7, 148.4)
- removed the H7 at (159.2, 148.4)
- removed the H7 at (46.8, 56.1)
- removed the R14 at (54.7, 97.7)
- added SW1: SW_Push, Button_Switch_THT:SW_PUSH_1P1T_6x3.5mm_H4.3_APEM_MJTP1243, F.Cu at (83.2, 147.7)
- moved FB4 83.8 mm to (70.5, 77.8), turned to -90 degrees
- moved J13 83.8 mm to (77.7, 70.7), turned to 180 degrees
- moved U8 75.6 mm to (75.0, 81.4), turned to 0 degrees
- moved U7 70.9 mm to (79.5, 81.4), turned to 0 degrees
- moved R20 70.7 mm to (84.5, 77.2), turned to 0 degrees
- moved R8 68.7 mm to (108.8, 67.3), turned to 0 degrees
- moved D13 67.6 mm to (82.8, 81.4), turned to -90 degrees
- moved R7 67.3 mm to (108.8, 68.3), turned to 0 degrees
- moved R19 66.2 mm to (84.3, 81.4), turned to -90 degrees
- moved R1 65.9 mm to (107.7, 69.4), turned to 180 degrees
- moved FB3 65.7 mm to (129.5, 77.2), turned to -90 degrees
- moved FB2 64.9 mm to (104.9, 70.7), turned to -90 degrees
- moved U1 64.4 mm to (106.5, 70.7), turned to -90 degrees
- moved TH1 64.2 mm to (82.8, 84.8), turned to 90 degrees
- moved D10 63.8 mm to (109.6, 70.6), turned to -90 degrees
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- renumbered C3 to C1, C16 to C10, C17 to C11, C19 to C14, C18 to C15, C20 to C16, C21 to C17, C7 to C2, C6 to C3, C8 to C4, C9 to C5, C10 to C6, C11 to C7, C14 to C8, C15 to C9, D2 to D1, D1 to D10, D3 to D2, D10 to D3, D9 to D4, D8 to D5, D7 to D6, D6 to D7, D5 to D8, D4 to D9, FB2 to FB1, FB1 to FB2, H5 to H2, H6 to H3, H8 to H7, H4 to H8, J7 to J10, J9 to J11, J4 to J3, J3 to J4, J8 to J5, J5 to J7, J11 to J8, J10 to J9, R19 to R14, R20 to R19, R21 to R20, R5 to R3, R6 to R4, R7 to R5, R8 to R6, R3 to R7, R4 to R8
Connections:
- net /BASEBOARD/_TXC2_P renamed Net-(U4C-CH3_OUT+)
- H2 pad 1: Net-(C1-Pad1) -> unconnected-(H2-Pad1)
- H3 pad 1: Net-(C2-Pad1) -> unconnected-(H3-Pad1)
- H7 pad 1: Net-(C5-Pad1) -> unconnected-(H7-Pad1)_1
- H8 pad 1: Net-(C4-Pad1) -> unconnected-(H8-Pad1)_0
- J5 pad 1: unconnected-(J8-Pin_1-Pad1) -> GND
- J5 pad 10: unconnected-(J8-Pin_10-Pad10) -> GND
- J5 pad 13: unconnected-(J8-Pin_13-Pad13) -> GND
- J5 pad 4: unconnected-(J8-Pin_4-Pad4) -> GND
- J5 pad 7: unconnected-(J8-Pin_7-Pad7) -> GND
- J8 pad 3: unconnected-(J11-Pin_3-Pad3) -> GND
- J8 pad 6: unconnected-(J11-Pin_6-Pad6) -> GND
- J8 pad 9: unconnected-(J11-Pin_9-Pad9) -> GND
- J9 pad 3: unconnected-(J10-Pin_3-Pad3) -> GND
- J9 pad 6: unconnected-(J10-Pin_6-Pad6) -> GND
- J9 pad 9: unconnected-(J10-Pin_9-Pad9) -> GND
Routing:
- net HDMI_HDP: track 74.3 -> 17.5 mm, vias 2 -> 0
- net HDMI_REFCLK_P: track 78.3 -> 23.9 mm
- net HDMI_REFCLK_N: track 77.6 -> 23.9 mm
- net HDMI_CEC: track 111.6 -> 64.2 mm
- net HDMI_SCL: track 97.6 -> 53.7 mm
- net HDMI_TX1_P: track 93.0 -> 54.9 mm, vias 2 -> 0
- net HDMI_SDA: track 93.5 -> 55.8 mm, vias 0 -> 2
- net HDMI_TX1_N: track 92.4 -> 54.9 mm, vias 2 -> 0
- net DSI_CLK_P: track 53.1 -> 18.3 mm
- net DSI_CLK_N: track 52.5 -> 18.3 mm
- net HDMI_TX0_N: track 92.2 -> 59.1 mm
- net HDMI_TX0_P: track 92.8 -> 60.4 mm
- net GBE0_MDI3_N: track 36.2 -> 67.6 mm, vias 1 -> 0
- net HDMI_TX3_P: track 89.5 -> 58.2 mm, vias 2 -> 0
- net HDMI_TX3_N: track 88.9 -> 58.2 mm, vias 2 -> 0
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Other:
- board size 122.5 x 102.5 mm -> 97 x 89.2 mm
